File: hdw/USB_Hub/Display.kicad_sch (KiCad schematic)
At the start: 0 parts

Commit message: lots and lots of sch progress
Parts:
- added C?: 10uF, Capacitors_SMD:C_0603, symbol Custom_Library:C_Custom
- added C? (x3): 10uF, Capacitors_SMD:C_0402, symbol Custom_Library:C_Custom
- added C?: 0.1uF, Capacitors_SMD:C_0603, symbol Custom_Library:C_Custom
- added C?: 0.1uF, Capacitors_SMD:C_0402, symbol Custom_Library:C_Custom
- added D?: BAT48JFILM, Diode_SMD:D_SOD-323, symbol Diode:BAT48JFILM
- added DOC1501: 0x3C, symbol Custom Library:I2C_Address
- added DOC?: 0x6B, symbol Custom_Library:I2C_Address
- added U1501: SSD1306, Connector_PinSocket_2.54mm:PinSocket_1x04_P2.54mm_Vertical, symbol Custom Library:SSD1306
- added U?: DS1683, Housings_SOIC:SOIC-8_3.9x4.9mm_Pitch1.27mm, symbol Custom_Library:DS1683
Connections:
- new net: C?.1, C?.1, C?.1, C?.1, D?.1 (K), U?.8 (VCC)
- new net +3.3V: C?.1, C?.1, D?.2 (A), U1501.2 (Vcc), U?.1 (EVENT)
- new net GND: C?.2, C?.2, C?.2, C?.2, C?.2, C?.2, U1501.1 (GND), U?.4 (GND)
- new net I2C_SCL: U1501.3 (SCL), U?.5 (SCL)
- new net I2C_SDA: U1501.4 (SDA), U?.6 (SDA)
- no-connect marks 0 -> 1

Commit message: pulled footprints into layout
Parts:
- C? (x3): footprint Capacitors_SMD:C_0402 -> Capacitors_SMD:C_0603; Digi-Key PN 1276-1451-1-ND -> 1276-1871-1-ND; Voltage 6.3V -> 10V; display_footprint 0402 -> 0603
- C?: footprint Capacitors_SMD:C_0402 -> Capacitors_SMD:C_0603; Digi-Key PN 490-10698-1-ND -> 1276-1935-1-ND; display_footprint 0402 -> 0603
Changed lines of the file:
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@@
       (effects (font (size 1.27 1.27)) (justify left))
     )
-    (property "Footprint" "Capacitors_SMD:C_0402" (at 80.7212 127.508 0)
+    (property "Footprint" "Capacitors_SMD:C_0603" (at 80.7212 127.508 0)
       (effects (font (size 1.27 1.27)) hide)
     )
@@
       (effects (font (size 1.27 1.27)) hide)
     )
-    (property "display_footprint" "0402" (at 75.946 121.158 0)
-      (effects (font (size 1.27 1.27)) (justify right))
-    )
-    (property "Voltage" "6.3V" (at 75.946 123.698 0)
+    (property "display_footprint" "0603" (at 75.946 121.158 0)
+      (effects (font (size 1.27 1.27)) (justify right))
+    )
+    (property "Voltage" "10V" (at 75.946 123.698 0)
       (effects (font (size 1.27 1.27)) (justify right))
     )
@@
       (effects (font (size 1.27 1.27)) (justify right))
     )
-    (property "Digi-Key PN" "1276-1451-1-ND" (at 79.756 123.698 0)
+    (property "Digi-Key PN" "1276-1871-1-ND" (at 79.756 123.698 0)
       (effects (font (size 1.27 1.27)) hide)
     )
@@
       (effects (font (size 1.27 1.27)) (justify left))
     )
-    (property "Footprint" "Capacitors_SMD:C_0402" (at 97.2312 127.508 0)
+    (property "Footprint" "Capacitors_SMD:C_0603" (at 97.2312 127.508 0)
       (effects (font (size 1.27 1.27)) hide)
     )
@@
       (effects (font (size 1.27 1.27)) hide)
     )
-    (property "display_footprint" "0402" (at 92.456 121.158 0)
-      (effects (font (size 1.27 1.27)) (justify right))
-    )
-    (property "Voltage" "6.3V" (at 92.456 123.698 0)
+    (property "display_footprint" "0603" (at 92.456 121.158 0)
+      (effects (font (size 1.27 1.27)) (justify right))
+    )
+    (property "Voltage" "10V" (at 92.456 123.698 0)
       (effects (font (size 1.27 1.27)) (justify right))
     )
@@
       (effects (font (size 1.27 1.27)) (justify right))
     )
-    (property "Digi-Key PN" "1276-1451-1-ND" (at 96.266 123.698 0)
+    (property "Digi-Key PN" "1276-1871-1-ND" (at 96.266 123.698 0)
       (effects (font (size 1.27 1.27)) hide)
     )
@@
       (effects (font (size 1.27 1.27)) (justify left))
     )
-    (property "Footprint" "Capacitors_SMD:C_0402" (at 113.7412 127.508 0)
+    (property "Footprint" "Capacitors_SMD:C_0603" (at 113.7412 127.508 0)
       (effects (font (size 1.27 1.27)) hide)
     )
@@
       (effects (font (size 1.27 1.27)) hide)
     )
-    (property "display_footprint" "0402" (at 108.966 121.158 0)
-      (effects (font (size 1.27 1.27)) (justify right))
-    )
-    (property "Voltage" "6.3V" (at 108.966 123.698 0)
+    (property "display_footprint" "0603" (at 108.966 121.158 0)
+      (effects (font (size 1.27 1.27)) (justify right))
+    )
+    (property "Voltage" "10V" (at 108.966 123.698 0)
       (effects (font (size 1.27 1.27)) (justify right))
     )
@@
       (effects (font (size 1.27 1.27)) (justify right))
     )
-    (property "Digi-Key PN" "1276-1451-1-ND" (at 112.776 123.698 0)
+    (property "Digi-Key PN" "1276-1871-1-ND" (at 112.776 123.698 0)
       (effects (font (size 1.27 1.27)) hide)
     )
@@
       (effects (font (size 1.27 1.27)) (justify left))
     )
-    (property "Footprint" "Capacitors_SMD:C_0402" (at 130.2512 127.508 0)
+    (property "Footprint" "Capacitors_SMD:C_0603" (at 130.2512 127.508 0)
       (effects (font (size 1.27 1.27)) hide)
     )
@@
       (effects (font (size 1.27 1.27)) hide)
     )
-    (property "display_footprint" "0402" (at 125.476 121.158 0)
+    (property "display_footprint" "0603" (at 125.476 121.158 0)
       (effects (font (size 1.27 1.27)) (justify right))
     )
@@
       (effects (font (size 1.27 1.27)) (justify right))
     )
-    (property "Digi-Key PN" "490-10698-1-ND" (at 140.081 110.998 0)
+    (property "Digi-Key PN" "1276-1935-1-ND" (at 140.081 110.998 0)
       (effects (font (size 1.524 1.524)) hide)
     )
