File: hdw/USB_Hub/PIC18F_Core.kicad_sch (KiCad schematic)
At the start: 1 part

Commit message: schematic progress
Other:
- note added: "Switch to TQFP version PIC18F47K40T-I/PTCT-ND"
Changed lines of the file:
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@@
     (stroke (width 0) (type default))
+  )
+  (text "Switch to TQFP version\nPIC18F47K40T-I/PTCT-ND" (at 85.09 39.37 0)
+    (effects (font (face "Courier New") (size 5.08 5.08) (thickness 1.016) bold (color 255 0 0 1)) (justify left bottom))
+  )
+  (global_label "~{DFP0_OC}" (shape input) (at 232.41 63.5 0) (fields_autoplaced)
+    (effects (font (size 1.27 1.27)) (justify left))
+    (property "Intersheetrefs" "${INTERSHEET_REFS}" (at 243.0678 63.5 0)
+      (effects (font (size 1.27 1.27)) (justify left) hide)
+    )
+  )
+  (global_label "~{DFP2_OC}" (shape input) (at 232.41 68.58 0) (fields_autoplaced)
+    (effects (font (size 1.27 1.27)) (justify left))
+    (property "Intersheetrefs" "${INTERSHEET_REFS}" (at 243.0678 68.58 0)
+      (effects (font (size 1.27 1.27)) (justify left) hide)
+    )
+  )
+  (global_label "~{DFP3_OC}" (shape input) (at 232.41 71.12 0) (fields_autoplaced)
+    (effects (font (size 1.27 1.27)) (justify left))
+    (property "Intersheetrefs" "${INTERSHEET_REFS}" (at 243.0678 71.12 0)
+      (effects (font (size 1.27 1.27)) (justify left) hide)
+    )
+  )
+  (global_label "~{DFP1_EN}" (shape output) (at 232.41 53.34 0) (fields_autoplaced)
+    (effects (font (size 1.27 1.27)) (justify left))
+    (property "Intersheetrefs" "${INTERSHEET_REFS}" (at 242.9468 53.34 0)
+      (effects (font (size 1.27 1.27)) (justify left) hide)
+    )
+  )
+  (global_label "~{DFP1_OC}" (shape input) (at 232.41 66.04 0) (fields_autoplaced)
+    (effects (font (size 1.27 1.27)) (justify left))
+    (property "Intersheetrefs" "${INTERSHEET_REFS}" (at 243.0678 66.04 0)
+      (effects (font (size 1.27 1.27)) (justify left) hide)
+    )
+  )
+  (global_label "~{DFP2_EN}" (shape output) (at 232.41 55.88 0) (fields_autoplaced)
+    (effects (font (size 1.27 1.27)) (justify left))
+    (property "Intersheetrefs" "${INTERSHEET_REFS}" (at 242.9468 55.88 0)
+      (effects (font (size 1.27 1.27)) (justify left) hide)
+    )
+  )
+  (global_label "~{DFP3_EN}" (shape output) (at 232.41 58.42 0) (fields_autoplaced)
+    (effects (font (size 1.27 1.27)) (justify left))
+    (property "Intersheetrefs" "${INTERSHEET_REFS}" (at 242.9468 58.42 0)
+      (effects (font (size 1.27 1.27)) (justify left) hide)
+    )
+  )
+  (global_label "~{DFP0_EN}" (shape output) (at 232.41 50.8 0) (fields_autoplaced)
+    (effects (font (size 1.27 1.27)) (justify left))
+    (property "Intersheetrefs" "${INTERSHEET_REFS}" (at 242.9468 50.8 0)
+      (effects (font (size 1.27 1.27)) (justify left) hide)
+    )
   )
   (symbol (lib_id "power:GND") (at 140.97 129.54 0) (unit 1)

Commit message: lots of schematic progress
Connections:
- net +5V renamed +3.3V
Other:
- company: (none) -> Drew Maatman
- title: (none) -> USB Hub
Changed lines of the file:
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@@
 (kicad_sch (version 20230121) (generator eeschema)
   (paper "A")
+  (title_block
+    (title "USB Hub")
+    (date "2023-08-18")
+    (rev "PRELIM")
+    (company "Drew Maatman")
+  )
   (junction (at 140.97 128.27) (diameter 0) (color 0 0 0 0)
   )
@@
     )
   )
+  (global_label "POS5_SOURCE_STATUS" (shape input) (at 222.885 93.98 0) (fields_autoplaced)
+    (effects (font (size 1.27 1.27)) (justify left))
+    (property "Intersheetrefs" "${INTERSHEET_REFS}" (at 246.4241 93.98 0)
+      (effects (font (size 1.27 1.27)) (justify left) hide)
+    )
+  )
   (global_label "~{DFP1_EN}" (shape output) (at 232.41 53.34 0) (fields_autoplaced)
     (effects (font (size 1.27 1.27)) (justify left))
@@
     )
   )
+  (symbol (lib_id "power:+3.3V") (at 140.97 60.96 0) (unit 1)
+    (in_bom yes) (on_board yes) (dnp no)
+    (property "Reference" "#PWR0702" (at 140.97 64.77 0)
+      (effects (font (size 1.27 1.27)) hide)
+    )
+    (property "Value" "+3.3V" (at 140.97 57.404 0)
+      (effects (font (size 1.27 1.27)))
+    )
+    (property "Footprint" "" (at 140.97 60.96 0)
+      (effects (font (size 1.27 1.27)) hide)
+    )
+    (property "Datasheet" "" (at 140.97 60.96 0)
+      (effects (font (size 1.27 1.27)) hide)
+    )
+    (pin "1")
+    (instances
+      (project "USB_Hub"
+        (path "/e85aac8c-404c-45dd-bda3-1057cae83baf/00000000-0000-0000-0000-00005f41a817"
+          (reference "#PWR0702") (unit 1)
+        )
+      )
+    )
+  )
   (symbol (lib_id "power:GND") (at 140.97 129.54 0) (unit 1)
     (in_bom yes) (on_board yes) (dnp no)
@@
         )
       )
-    )
-  )
-  (symbol (lib_id "power:+5V") (at 140.97 60.96 0) (unit 1)
-    (in_bom yes) (on_board yes) (dnp no)
-    (property "Reference" "#PWR0702" (at 140.97 64.77 0)
-      (effects (font (size 1.27 1.27)) hide)
-    )
-    (property "Value" "+5V" (at 140.97 57.404 0)
-      (effects (font (size 1.27 1.27)))
-    )
-    (property "Footprint" "" (at 140.97 60.96 0)
-      (effects (font (size 1.27 1.27)) hide)
-    )
-    (property "Datasheet" "" (at 140.97 60.96 0)
-      (effects (font (size 1.27 1.27)) hide)
-    )
-    (pin "1")
-    (instances
-      (project "USB_Hub"
-        (path "/e85aac8c-404c-45dd-bda3-1057cae83baf/00000000-0000-0000-0000-00005f41a817"
-          (reference "#PWR0702") (unit 1)
-        )
-      )

Commit message: much more schematic progress
Parts:
- removed U?: PIC18(L)F47K40-I_ML, Housings_DFN_QFN:QFN-44-1EP_8x8mm_Pitch0.65mm, symbol Custom Library:PIC18(L)F47K40-I_ML
- added C? (x2): 0.1uF, Capacitors_SMD:C_0603, symbol Custom_Library:C_Custom
- added U?: PIC18(L)F47K40T-I_PT, Housings_QFP:TQFP-44_10x10mm_Pitch0.8mm, symbol Custom Library:PIC18(L)F47K40T-I_PT
Connections:
- net +3.3V: now also C?.1, C?.1, U?.28 (Vdd), U?.7 (Vdd)
- net GND: now also C?.2, C?.2, U?.29 (Vss), U?.6 (Vss)
- new net PIC18F_ICSPCLK: U?.16 (RB6/ICSPCLK)
- new net PIC18F_ICSPDAT: U?.17 (RB7/ICSPDAT)
- new net ~{PIC18F_MCLR}: U?.18 (RE3/~{MCLR}/Vpp)
Other:
- note removed: "Switch to TQFP version PIC18F47K40T-I/PTCT-ND"

Commit message: lots and lots of sch progress
Parts:
- added R? (x3): 10k, Resistors_SMD:R_0603, symbol Custom_Library:R_Custom
- added TP?: TP, Custom Footprints Library:Test_Point, symbol Custom_Library:TP
- gave numbers to parts that had none: 1
Connections:
- net +3.3V: now also R?.1, R?.1
- net CAP_TOUCH_LEFT: now also U1001.19 (RA0)
- net CAP_TOUCH_POWER: now also U1001.21 (RA2)
- net CAP_TOUCH_RIGHT: now also U1001.20 (RA1)
- net Error_LED: now also U1001.23 (RA4)
- net GND: now also R?.2
- net Heartbeat_LED: now also U1001.22 (RA3)
- net I2C_SCL: now also U1001.37 (RC3), R?.2
- net I2C_SDA: now also U1001.42 (RC4), R?.2
- net PGOOD_LED_SHDN: now also U1001.14 (RB4)
- net POS12_PGOOD: now also U1001.9 (RB1)
- net POS3P3_PGOOD: now also U1001.8 (RB0)
- net POS5P_PGOOD: now also U1001.10 (RB2)
- net POS5_SOURCE_STATUS: now also U1001.11 (RB3)
- net Reset_LED: now also U1001.43 (RC5)
- net USB_UART_RX: now also U1001.1 (RC7)
- net USB_UART_TX: now also U1001.44 (RC6)
- net ~{DFP0_EN}: now also U1001.38 (RD0)
- net ~{DFP0_OC}: now also U1001.2 (RD4)
- net ~{DFP1_EN}: now also U1001.39 (RD1)
- net ~{DFP1_OC}: now also U1001.3 (RD5)
- net ~{DFP2_EN}: now also U1001.40 (RD2)
- net ~{DFP2_OC}: now also U1001.4 (RD6)
- net ~{DFP3_EN}: now also U1001.41 (RD3)
- net ~{DFP3_OC}: now also U1001.5 (RD7)
- net ~{HUB_RESET}: now also U1001.24 (RA5)
- net POS5_USB_PGOOD: now reaches U1001.15 (RB5)
- net ~{ETC_Hardstrap}: now reaches U1001.30 (RA7/OSC1/CLKIN)
- net ~{Telemetry_Hardstrap}: now reaches U1001.31 (RA6/OSC2/CLKOUT)
- net HUB_SUSPND: now reaches U1001.32 (SOSCO/RC0)
- net PIC18F_REFCLK0: now reaches U1001.36 (RC2)
- net PIC18F_REFCLK0: now also R?.1, TP?.1 (TP)
- no-connect marks 0 -> 4
Other:
- note added: "CK1PPS"
- note added: "INT0PPS"
- note added: "INT1PPS"
- note added: "INT2PPS"
- note added: "PWM3PPS"
- note added: "RX1PPS"
- note added: "SSP1CLKPPS"
- note added: "SSP1DATPPS"

Commit message: pulled footprints into layout
Parts:
- R? (x3): Digi-Key PN YAG2321CT-ND -> (none)
Changed lines of the file:
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@@
       (effects (font (size 1.27 1.27)) (justify left) hide)
     )
-    (property "Digi-Key PN" "YAG2321CT-ND" (at 233.68 72.39 0)
+    (property "Digi-Key PN" "" (at 233.68 72.39 0)
       (effects (font (size 1.27 1.27)) hide)
     )
@@
       (effects (font (size 1.27 1.27)) (justify left) hide)
     )
-    (property "Digi-Key PN" "YAG2321CT-ND" (at 252.73 72.39 0)
+    (property "Digi-Key PN" "" (at 252.73 72.39 0)
       (effects (font (size 1.27 1.27)) hide)
     )
@@
       (effects (font (size 1.27 1.27)) (justify left) hide)
     )
-    (property "Digi-Key PN" "YAG2321CT-ND" (at 246.38 72.39 0)
-      (effects (font (size 1.27 1.27)) hide)
-    )
+    (property "Digi-Key PN" "" (at 246.38 72.39 0)
+      (effects (font (size 1.27 1.27)) hide)
+    )
