File: hdw/USB_Hub/PIC18F_Programming.kicad_sch (KiCad schematic)
At the start: 0 parts

Commit message: schematic progress
Parts:
- added C? (x2): 0.1uF, Capacitors_SMD:C_0603, symbol Custom_Library:C_Custom
- added D? (x5): PESD3V3L5UY, Package_TO_SOT_SMD:SOT-363_SC-70-6, symbol Power_Protection:PESD3V3L5UY
- added J?: PICKIT4, Custom Footprints Library:PICKIT4_Header, symbol Connector_Generic:Conn_01x08
- added L? (x2): 600R 0.5A, Inductors_SMD:L_0603, symbol Device:Ferrite_Bead
- added Q?: BSS214NW, Package_TO_SOT_SMD:SOT-323_SC-70, symbol Transistor_FET:BSS214NW
- added R? (x2): 10k, Resistors_SMD:R_0603, symbol Custom_Library:R_Custom
- added R? (x2): 10, Resistors_SMD:R_0603, symbol Custom_Library:R_Custom
- added R?: 1k, Resistors_SMD:R_0603, symbol Custom_Library:R_Custom
- added SW?: MRST, Button_Switch_THT:SW_PUSH_6mm, symbol Switch:SW_Push
Connections:
- new net: C?.1, R?.2, R?.2, R?.2
- new net: R?.1, SW?.2
- new net: Q?.1 (G), R?.1, R?.2
- new net: D?.3 (K2), J?.1 (Pin_1), L?.2
- new net: Q?.3 (D), R?.1
- new net: J?.3 (Pin_3), L?.1
- new net +3.3V: C?.1, D?.1 (K1), J?.2 (Pin_2), R?.1, SW?.1
- new net GND: C?.2, C?.2, D?.2 (A), L?.2, Q?.2 (S), R?.2
- new net PIC18F_ICSPCLK: D?.5 (K4), J?.5 (Pin_5)
- new net PIC18F_ICSPDAT: D?.6 (K5), J?.4 (Pin_4)
- new net ~{PIC18F_MCLR}: L?.1, R?.1
- no-connect marks 0 -> 4
Other:
- note added: "+5V?"

Commit message: lots of schematic progress
Other:
- note removed: "+5V?"
- company: (none) -> Drew Maatman
- title: (none) -> USB Hub
Changed lines of the file:
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@@
 (kicad_sch (version 20230121) (generator eeschema)
   (paper "A")
+  (title_block
+    (title "USB Hub")
+    (date "2023-08-18")
+    (rev "PRELIM")
+    (company "Drew Maatman")
+  )
   (junction (at 106.68 137.16) (diameter 0) (color 0 0 0 0)
   )
@@
     (stroke (width 0) (type default))
   )
-  (text "+5V?" (at 100.33 29.21 0)
-    (effects (font (face "Courier New") (size 5.08 5.08) (thickness 1.016) bold (color 255 0 0 1)) (justify left bottom))
-  )
   (global_label "~{PIC18F_MCLR}" (shape passive) (at 147.32 44.45 0) (fields_autoplaced)

Commit message: lots and lots of sch progress
Parts:
- removed D? (x5): PESD3V3L5UY, Package_TO_SOT_SMD:SOT-363_SC-70-6, symbol Power_Protection:PESD3V3L5UY
- added D?: SP0503BAHT, Package_TO_SOT_SMD:SOT-143, symbol Power_Protection:SP0503BAHT
Connections:
- net +3.3V: now also D?.2 (K)
- net GND: now also D?.1 (A)
- net PIC18F_ICSPCLK: now also D?.4 (K)
- net PIC18F_ICSPDAT: now also D?.3 (K)
- no-connect marks 4 -> 3

Commit message: pulled footprints into layout
Parts:
- R? (x2): Digi-Key PN 541-10.0KHCT-ND -> (none)
- R? (x2): Digi-Key PN 541-10.0HCT-ND -> (none)
- R?: Digi-Key PN 541-1.00KHCT-ND -> (none)
Changed lines of the file:
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@@
       (effects (font (size 1.27 1.27)))
     )
-    (property "Digi-Key PN" "541-10.0KHCT-ND" (at 140.335 107.95 0)
+    (property "Digi-Key PN" "" (at 140.335 107.95 0)
       (effects (font (size 1.524 1.524)) hide)
     )
@@
       (effects (font (size 1.27 1.27)))
     )
-    (property "Digi-Key PN" "541-10.0HCT-ND" (at 85.09 129.54 0)
+    (property "Digi-Key PN" "" (at 85.09 129.54 0)
       (effects (font (size 1.524 1.524)) hide)
     )
@@
       (effects (font (size 1.27 1.27)))
     )
-    (property "Digi-Key PN" "541-10.0KHCT-ND" (at 114.3 132.715 0)
+    (property "Digi-Key PN" "" (at 114.3 132.715 0)
       (effects (font (size 1.524 1.524)) hide)
     )
@@
       (effects (font (size 1.27 1.27)))
     )
-    (property "Digi-Key PN" "541-10.0HCT-ND" (at 120.65 116.205 0)
+    (property "Digi-Key PN" "" (at 120.65 116.205 0)
       (effects (font (size 1.524 1.524)) hide)
     )
@@
       (effects (font (size 1.27 1.27)))
     )
-    (property "Digi-Key PN" "541-1.00KHCT-ND" (at 171.45 131.445 0)
+    (property "Digi-Key PN" "" (at 171.45 131.445 0)
       (effects (font (size 1.524 1.524)) hide)
     )
