File: hdw/USB_Hub/POS12_Telemetry.kicad_sch (KiCad schematic)
At the start: 7 parts

Commit message: lots of schematic progress
Other:
- title: Analog Clock -> USB Hub
Changed lines of the file:
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@@
   (paper "A")
   (title_block
-    (title "Analog Clock")
-    (date "2020-08-15")
-    (rev "A")
+    (title "USB Hub")
+    (date "2023-08-18")
+    (rev "PRELIM")
     (company "Drew Maatman")
   )

Commit message: lots and lots of sch progress
Parts:
- DOC301: renamed from DOC?; value FIX ME -> 0x40
- DOC302: renamed from DOC?; value FIX ME -> 0x18
- gave numbers to parts that had none: 5
Connections:
- net GND: now also U301.7 (A0), U301.8 (A1), U302.5 (A2), U302.6 (A1), U302.7 (A0)

Commit message: pulled footprints into layout
Parts:
- C301, C302, C303: Digi-Key PN 399-7845-1-ND -> 1276-1935-1-ND
Changed lines of the file:
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@@
       (effects (font (size 1.27 1.27)) (justify right))
     )
-    (property "Digi-Key PN" "399-7845-1-ND" (at 8.001 226.187 0)
+    (property "Digi-Key PN" "1276-1935-1-ND" (at 8.001 226.187 0)
       (effects (font (size 1.27 1.27)) hide)
     )
@@
       (effects (font (size 1.27 1.27)) (justify right))
     )
-    (property "Digi-Key PN" "399-7845-1-ND" (at 30.226 319.532 0)
+    (property "Digi-Key PN" "1276-1935-1-ND" (at 30.226 319.532 0)
       (effects (font (size 1.27 1.27)) hide)
     )
@@
       (effects (font (size 1.27 1.27)) (justify right))
     )
-    (property "Digi-Key PN" "399-7845-1-ND" (at 30.226 250.952 0)
-      (effects (font (size 1.27 1.27)) hide)
-    )
+    (property "Digi-Key PN" "1276-1935-1-ND" (at 30.226 250.952 0)
+      (effects (font (size 1.27 1.27)) hide)
+    )
