File: hdw/USB_Hub/POS3P3_Telemetry.kicad_sch (KiCad schematic)
At the start: 0 parts

Commit message: much more schematic progress
Parts:
- added C? (x3): 0.1uF, Capacitors_SMD:C_0603, symbol Custom_Library:C_Custom
- added DOC? (x2): FIX ME, symbol Custom_Library:I2C_Address
- added U?: MCP9804, Package_DFN_QFN:DFN-8-1EP_3x2mm_P0.5mm_EP1.3x1.5mm, symbol Sensor_Temperature:MCP9804_DFN
- added U?: INA219BxDCN, Package_TO_SOT_SMD:SOT-23-8, symbol Analog_ADC:INA219BxDCN
Connections:
- new net +3.3V: C?.1, C?.1, U?.4 (VS), U?.8 (V_{DD})
- new net GND: C?.2, C?.2, U?.3 (GND), U?.4 (GND), U?.9 (EP/GND)
- new net I2C_SCL: U?.2 (SCL), U?.5 (SCL)
- new net I2C_SDA: U?.1 (SDA), U?.6 (SDA)
- new net POS3P3_SNS+: C?.1, U?.1 (IN+)
- new net POS3P3_SNS-: C?.2, U?.2 (IN-)
- no-connect marks 0 -> 1
Other:
- note added: "RSHUNT = 0.02 CLSB = 60uA"

Commit message: lots and lots of sch progress
Parts:
- DOC?: value FIX ME -> 0x1A
- DOC?: value FIX ME -> 0x42
Connections:
- net +3.3V: now also U?.6 (A1)
- net GND: now also U?.5 (A2), U?.7 (A0), U?.8 (A1)
- net I2C_SDA: now also U?.7 (A0)
Changed lines of the file:
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@@
   (title_block
     (title "USB Hub")
-    (date "2023-08-18")
+    (date "2023-08-20")
     (rev "PRELIM")
     (company "Drew Maatman")
@@
     )
   )
+  (global_label "I2C_SDA" (shape bidirectional) (at 151.13 52.07 0)
+    (effects (font (size 1.27 1.27)) (justify left))
+    (property "Intersheetrefs" "${INTERSHEET_REFS}" (at 151.13 52.07 0)
+      (effects (font (size 1.27 1.27)) hide)
+    )
+  )
   (global_label "I2C_SDA" (shape bidirectional) (at 151.13 102.87 0)
     (effects (font (size 1.27 1.27)) (justify left))
@@
     )
   )
+  (symbol (lib_id "power:+3.3V") (at 151.13 115.57 270) (mirror x) (unit 1)
+    (in_bom yes) (on_board yes) (dnp no)
+    (property "Reference" "#PWR?" (at 147.32 115.57 0)
+      (effects (font (size 1.27 1.27)) hide)
+    )
+    (property "Value" "+3.3V" (at 154.305 115.57 90)
+      (effects (font (size 1.27 1.27)) (justify left))
+    )
+    (property "Footprint" "" (at 151.13 115.57 0)
+      (effects (font (size 1.27 1.27)) hide)
+    )
+    (property "Datasheet" "" (at 151.13 115.57 0)
+      (effects (font (size 1.27 1.27)) hide)
+    )
+    (pin "1")
+    (instances
+      (project "USB_Hub"
+        (path "/e85aac8c-404c-45dd-bda3-1057cae83baf/00000000-0000-0000-0000-00005f41a7d6"
+          (reference "#PWR?") (unit 1)
+        )
+        (path "/e85aac8c-404c-45dd-bda3-1057cae83baf/b536b902-d925-4d87-a550-76997db32615"
+          (reference "#PWR0711") (unit 1)
+        )
+      )
+    )
+  )
   (symbol (lib_id "power:+3.3V") (at 140.97 67.31 0) (unit 1)
     (in_bom yes) (on_board yes) (dnp no)
@@
         )
         (path "/e85aac8c-404c-45dd-bda3-1057cae83baf/b536b902-d925-4d87-a550-76997db32615"
-          (reference "#PWR02303") (unit 1)
+          (reference "#PWR0703") (unit 1)
         )
       )
@@
         )
         (path "/e85aac8c-404c-45dd-bda3-1057cae83baf/b536b902-d925-4d87-a550-76997db32615"
-          (reference "C?") (unit 1)
+          (reference "C702") (unit 1)
         )
       )
@@
       (effects (font (size 1.524 1.524)) hide)
     )
-    (property "Value" "FIX ME" (at 152.273 136.144 0)
+    (property "Value" "0x1A" (at 152.273 136.144 0)
       (effects (font (size 1.524 1.524)) (justify left))
     )
@@
         )
         (path "/e85aac8c-404c-45dd-bda3-1057cae83baf/b536b902-d925-4d87-a550-76997db32615"
-          (reference "DOC?") (unit 1)
+          (reference "DOC702") (unit 1)
         )
       )
@@
         )
         (path "/e85aac8c-404c-45dd-bda3-1057cae83baf/b536b902-d925-4d87-a550-76997db32615"
-          (reference "C?") (unit 1)
+          (reference "C701") (unit 1)
         )
       )
@@
       (effects (font (size 1.524 1.524)) hide)
     )
-    (property "Value" "FIX ME" (at 152.273 68.072 0)
+    (property "Value" "0x42" (at 152.273 68.072 0)
       (effects (font (size 1.524 1.524)) (justify left))
     )
@@
         )
         (path "/e85aac8c-404c-45dd-bda3-1057cae83baf/b536b902-d925-4d87-a550-76997db32615"
-          (reference "DOC?") (unit 1)
+          (reference "DOC701") (unit 1)
+        )
+      )
+    )
+  )
+  (symbol (lib_id "power:GND") (at 151.13 49.53 90) (unit 1)
+    (in_bom yes) (on_board yes) (dnp no)
+    (property "Reference" "#PWR?" (at 157.48 49.53 0)
+      (effects (font (size 1.27 1.27)) hide)
+    )
+    (property "Value" "GND" (at 154.305 49.53 90)
+      (effects (font (size 1.27 1.27)) (justify right))
+    )
+    (property "Footprint" "" (at 151.13 49.53 0)
+      (effects (font (size 1.27 1.27)) hide)
+    )
+    (property "Datasheet" "" (at 151.13 49.53 0)
+      (effects (font (size 1.27 1.27)) hide)
+    )
+    (pin "1")
+    (instances
+      (project "USB_Hub"
+        (path "/e85aac8c-404c-45dd-bda3-1057cae83baf/00000000-0000-0000-0000-00005f41a7c0"
+          (reference "#PWR?") (unit 1)
+        )
+        (path "/e85aac8c-404c-45dd-bda3-1057cae83baf/b536b902-d925-4d87-a550-76997db32615"
+          (reference "#PWR0709") (unit 1)
         )
       )
@@
         )
         (path "/e85aac8c-404c-45dd-bda3-1057cae83baf/b536b902-d925-4d87-a550-76997db32615"
-          (reference "#PWR02307") (unit 1)
+          (reference "#PWR0707") (unit 1)
         )
       )
@@
         )
         (path "/e85aac8c-404c-45dd-bda3-1057cae83baf/b536b902-d925-4d87-a550-76997db32615"
-          (reference "U?") (unit 1)
+          (reference "U702") (unit 1)
+        )
+      )
+    )
+  )
+  (symbol (lib_id "power:GND") (at 151.13 118.11 90) (unit 1)
+    (in_bom yes) (on_board yes) (dnp no)
+    (property "Reference" "#PWR?" (at 157.48 118.11 0)
+      (effects (font (size 1.27 1.27)) hide)
+    )
+    (property "Value" "GND" (at 154.305 118.11 90)
+      (effects (font (size 1.27 1.27)) (justify right))
+    )
+    (property "Footprint" "" (at 151.13 118.11 0)
+      (effects (font (size 1.27 1.27)) hide)
+    )
+    (property "Datasheet" "" (at 151.13 118.11 0)
+      (effects (font (size 1.27 1.27)) hide)
+    )
+    (pin "1")
+    (instances
+      (project "USB_Hub"
+        (path "/e85aac8c-404c-45dd-bda3-1057cae83baf/00000000-0000-0000-0000-00005f41a7c0"
+          (reference "#PWR?") (unit 1)
+        )
+        (path "/e85aac8c-404c-45dd-bda3-1057cae83baf/b536b902-d925-4d87-a550-76997db32615"
+          (reference "#PWR0712") (unit 1)
         )
       )
@@
         )
         (path "/e85aac8c-404c-45dd-bda3-1057cae83baf/b536b902-d925-4d87-a550-76997db32615"
-          (reference "C?") (unit 1)
+          (reference "C703") (unit 1)
         )
       )
@@
         )
         (path "/e85aac8c-404c-45dd-bda3-1057cae83baf/b536b902-d925-4d87-a550-76997db32615"
-          (reference "#PWR02306") (unit 1)
+          (reference "#PWR0706") (unit 1)
         )
       )
@@
         )
         (path "/e85aac8c-404c-45dd-bda3-1057cae83baf/b536b902-d925-4d87-a550-76997db32615"
-          (reference "#PWR02302") (unit 1)
+          (reference "#PWR0702") (unit 1)
         )
       )
@@
         )
         (path "/e85aac8c-404c-45dd-bda3-1057cae83baf/b536b902-d925-4d87-a550-76997db32615"
-          (reference "#PWR02308") (unit 1)
+          (reference "#PWR0708") (unit 1)
         )
       )
@@
         )
         (path "/e85aac8c-404c-45dd-bda3-1057cae83baf/b536b902-d925-4d87-a550-76997db32615"
-          (reference "#PWR02304") (unit 1)
+          (reference "#PWR0704") (unit 1)
+        )
+      )
+    )
+  )
+  (symbol (lib_id "power:GND") (at 151.13 113.03 90) (unit 1)
+    (in_bom yes) (on_board yes) (dnp no)
+    (property "Reference" "#PWR?" (at 157.48 113.03 0)
+      (effects (font (size 1.27 1.27)) hide)
+    )
+    (property "Value" "GND" (at 154.305 113.03 90)
+      (effects (font (size 1.27 1.27)) (justify right))
+    )
+    (property "Footprint" "" (at 151.13 113.03 0)
+      (effects (font (size 1.27 1.27)) hide)
+    )
+    (property "Datasheet" "" (at 151.13 113.03 0)
+      (effects (font (size 1.27 1.27)) hide)
+    )
+    (pin "1")
+    (instances
+      (project "USB_Hub"
+        (path "/e85aac8c-404c-45dd-bda3-1057cae83baf/00000000-0000-0000-0000-00005f41a7c0"
+          (reference "#PWR?") (unit 1)
+        )
+        (path "/e85aac8c-404c-45dd-bda3-1057cae83baf/b536b902-d925-4d87-a550-76997db32615"
+          (reference "#PWR0710") (unit 1)
         )
       )
@@
         )
         (path "/e85aac8c-404c-45dd-bda3-1057cae83baf/b536b902-d925-4d87-a550-76997db32615"
-          (reference "U?") (unit 1)
+          (reference "U701") (unit 1)
         )
       )
@@
         )
         (path "/e85aac8c-404c-45dd-bda3-1057cae83baf/b536b902-d925-4d87-a550-76997db32615"
-          (reference "#PWR02305") (unit 1)
+          (reference "#PWR0705") (unit 1)
         )
       )
@@
         )
         (path "/e85aac8c-404c-45dd-bda3-1057cae83baf/b536b902-d925-4d87-a550-76997db32615"
-          (reference "#PWR02301") (unit 1)
-        )
-      )
+          (reference "#PWR0701") (unit 1)
+        )
+      )

Commit message: pulled footprints into layout
Parts:
- C? (x3): Digi-Key PN 399-7845-1-ND -> 1276-1935-1-ND
Changed lines of the file:
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@@
       (effects (font (size 1.27 1.27)) (justify right))
     )
-    (property "Digi-Key PN" "399-7845-1-ND" (at 41.656 245.872 0)
+    (property "Digi-Key PN" "1276-1935-1-ND" (at 41.656 245.872 0)
       (effects (font (size 1.27 1.27)) hide)
     )
@@
       (effects (font (size 1.27 1.27)) (justify right))
     )
-    (property "Digi-Key PN" "399-7845-1-ND" (at 19.431 221.107 0)
+    (property "Digi-Key PN" "1276-1935-1-ND" (at 19.431 221.107 0)
       (effects (font (size 1.27 1.27)) hide)
     )
@@
       (effects (font (size 1.27 1.27)) (justify right))
     )
-    (property "Digi-Key PN" "399-7845-1-ND" (at 41.656 314.452 0)
-      (effects (font (size 1.27 1.27)) hide)
-    )
+    (property "Digi-Key PN" "1276-1935-1-ND" (at 41.656 314.452 0)
+      (effects (font (size 1.27 1.27)) hide)
+    )
