File: hdw/USB_Hub/POS5_Telemetry.kicad_sch (KiCad schematic)
At the start: 7 parts

Commit message: schematic progress
Connections:
- net POS12_SNS+ renamed POS5_SNS+
- net POS12_SNS- renamed POS5_SNS-
Changed lines of the file:
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@@
     )
   )
-  (global_label "POS12_SNS+" (shape passive) (at 96.266 45.72 180)
+  (global_label "POS5_SNS+" (shape passive) (at 96.266 45.72 180)
     (effects (font (size 1.27 1.27)) (justify right))
     (property "Intersheetrefs" "${INTERSHEET_REFS}" (at 96.266 45.72 0)
@@
     )
   )
-  (global_label "POS12_SNS-" (shape passive) (at 96.266 57.404 180)
+  (global_label "POS5_SNS-" (shape passive) (at 96.266 57.404 180)
     (effects (font (size 1.27 1.27)) (justify right))
     (property "Intersheetrefs" "${INTERSHEET_REFS}" (at 96.266 57.404 0)

Commit message: lots of schematic progress
Other:
- title: Analog Clock -> USB Hub
Changed lines of the file:
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@@
   (paper "A")
   (title_block
-    (title "Analog Clock")
-    (date "2020-08-15")
-    (rev "A")
+    (title "USB Hub")
+    (date "2023-08-18")
+    (rev "PRELIM")
     (company "Drew Maatman")
   )

Commit message: lots and lots of sch progress
Parts:
- DOC501: renamed from DOC?; value FIX ME -> 0x41
- DOC502: renamed from DOC?; value FIX ME -> 0x19
- gave numbers to parts that had none: 5
Connections:
- net +3.3V: now also U501.7 (A0), U502.7 (A0)
- net GND: now also U501.8 (A1), U502.5 (A2), U502.6 (A1)

Commit message: pulled footprints into layout
Parts:
- C501, C502, C503: Digi-Key PN 399-7845-1-ND -> 1276-1935-1-ND
Changed lines of the file:
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@@
       (effects (font (size 1.27 1.27)) (justify right))
     )
-    (property "Digi-Key PN" "399-7845-1-ND" (at 30.226 319.532 0)
+    (property "Digi-Key PN" "1276-1935-1-ND" (at 30.226 319.532 0)
       (effects (font (size 1.27 1.27)) hide)
     )
@@
       (effects (font (size 1.27 1.27)) (justify right))
     )
-    (property "Digi-Key PN" "399-7845-1-ND" (at 8.001 226.187 0)
+    (property "Digi-Key PN" "1276-1935-1-ND" (at 8.001 226.187 0)
       (effects (font (size 1.27 1.27)) hide)
     )
@@
       (effects (font (size 1.27 1.27)) (justify right))
     )
-    (property "Digi-Key PN" "399-7845-1-ND" (at 30.226 250.952 0)
+    (property "Digi-Key PN" "1276-1935-1-ND" (at 30.226 250.952 0)
       (effects (font (size 1.27 1.27)) hide)
     )
