File: hdw/USB_Hub/Port_Telemetry.kicad_sch (KiCad schematic)
At the start: 16 parts

Commit message: lots and lots of sch progress
Parts:
- added C?: 0.1uF, Capacitors_SMD:C_0603, symbol Custom_Library:C_Custom
- added DOC?: 0x1B, symbol Custom_Library:I2C_Address
- added J?: I2C, Pin_Headers:Pin_Header_Straight_1x03_Pitch2.54mm, symbol Connector_Generic:Conn_01x03
- added J?: USB UART, Pin_Headers:Pin_Header_Straight_1x03_Pitch2.54mm, symbol Connector_Generic:Conn_01x03
- added R? (x2): 10, Resistors_SMD:R_0603, symbol Custom_Library:R_Custom
- added R? (x2): 10k, Resistors_SMD:R_0603, symbol Custom_Library:R_Custom
- added U?: MCP9804, Package_DFN_QFN:DFN-8-1EP_3x2mm_P0.5mm_EP1.3x1.5mm, symbol Sensor_Temperature:MCP9804_DFN
- DOC?: value FIX ME -> 0x43
- DOC?: value FIX ME -> 0x44
- DOC?: value FIX ME -> 0x46
- DOC?: value FIX ME -> 0x45
Connections:
- net +3.3V: now also U?.7 (A0), U?.8 (A1), U?.8 (A1), U?.8 (A1), C?.1, R?.1, R?.1, U?.6 (A1), U?.7 (A0), U?.8 (V_{DD})
- net GND: now also U?.7 (A0), U?.8 (A1), C?.2, J?.3 (Pin_3), J?.3 (Pin_3), R?.2, R?.2, U?.4 (GND), U?.5 (A2), U?.9 (EP/GND)
- net I2C_SCL: now also U?.7 (A0), J?.1 (Pin_1), U?.2 (SCL)
- net I2C_SDA: now also U?.7 (A0), J?.2 (Pin_2), U?.1 (SDA)
- new net USB_UART_RX: J?.2 (Pin_2)
- new net USB_UART_TX: J?.1 (Pin_1)
- new net ~{ETC_Hardstrap}: R?.1, R?.2
- new net ~{Telemetry_Hardstrap}: R?.1, R?.2
- no-connect marks 0 -> 1
Other:
- company: (none) -> Drew Maatman
- title: (none) -> USB Hub
- moved on the sheet: C?, U?

Commit message: pulled footprints into layout
Parts:
- C? (x9): Digi-Key PN 399-7845-1-ND -> 1276-1935-1-ND
- J? (x2): footprint Pin_Headers:Pin_Header_Straight_1x03_Pitch2.54mm -> Connector_PinHeader_2.54mm:PinHeader_1x03_P2.54mm_Vertical
- R? (x2): Digi-Key PN YAG2321CT-ND -> (none)
Changed lines of the file:
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@@
       (effects (font (size 1.27 1.27)) (justify right))
     )
-    (property "Digi-Key PN" "399-7845-1-ND" (at -28.194 273.812 0)
+    (property "Digi-Key PN" "1276-1935-1-ND" (at -28.194 273.812 0)
       (effects (font (size 1.27 1.27)) hide)
     )
@@
       (effects (font (size 1.27 1.27)) (justify left))
     )
-    (property "Digi-Key PN" "YAG2321CT-ND" (at 60.325 148.59 0)
+    (property "Digi-Key PN" "" (at 60.325 148.59 0)
       (effects (font (size 1.524 1.524)) hide)
     )
@@
       (effects (font (size 1.27 1.27)) (justify right))
     )
-    (property "Digi-Key PN" "399-7845-1-ND" (at 73.406 273.812 0)
+    (property "Digi-Key PN" "1276-1935-1-ND" (at 73.406 273.812 0)
       (effects (font (size 1.27 1.27)) hide)
     )
@@
       (effects (font (size 1.27 1.27)) (justify right))
     )
-    (property "Digi-Key PN" "399-7845-1-ND" (at 19.431 361.442 0)
+    (property "Digi-Key PN" "1276-1935-1-ND" (at 19.431 361.442 0)
       (effects (font (size 1.27 1.27)) hide)
     )
@@
       (effects (font (size 1.27 1.27)))
     )
-    (property "Footprint" "Pin_Headers:Pin_Header_Straight_1x03_Pitch2.54mm" (at 38.735 154.94 0)
+    (property "Footprint" "Connector_PinHeader_2.54mm:PinHeader_1x03_P2.54mm_Vertical" (at 38.735 154.94 0)
       (effects (font (size 1.27 1.27)) hide)
     )
@@
       (effects (font (size 1.27 1.27)) (justify right))
     )
-    (property "Digi-Key PN" "399-7845-1-ND" (at 73.406 210.312 0)
+    (property "Digi-Key PN" "1276-1935-1-ND" (at 73.406 210.312 0)
       (effects (font (size 1.27 1.27)) hide)
     )
@@
       (effects (font (size 1.27 1.27)) (justify right))
     )
-    (property "Digi-Key PN" "399-7845-1-ND" (at -5.969 298.577 0)
+    (property "Digi-Key PN" "1276-1935-1-ND" (at -5.969 298.577 0)
       (effects (font (size 1.27 1.27)) hide)
     )
@@
       (effects (font (size 1.27 1.27)))
     )
-    (property "Footprint" "Pin_Headers:Pin_Header_Straight_1x03_Pitch2.54mm" (at 38.735 173.99 0)
+    (property "Footprint" "Connector_PinHeader_2.54mm:PinHeader_1x03_P2.54mm_Vertical" (at 38.735 173.99 0)
       (effects (font (size 1.27 1.27)) hide)
     )
@@
       (effects (font (size 1.27 1.27)) (justify right))
     )
-    (property "Digi-Key PN" "399-7845-1-ND" (at 95.631 298.577 0)
+    (property "Digi-Key PN" "1276-1935-1-ND" (at 95.631 298.577 0)
       (effects (font (size 1.27 1.27)) hide)
     )
@@
       (effects (font (size 1.27 1.27)) (justify left))
     )
-    (property "Digi-Key PN" "YAG2321CT-ND" (at 85.725 148.59 0)
+    (property "Digi-Key PN" "" (at 85.725 148.59 0)
       (effects (font (size 1.524 1.524)) hide)
     )
@@
       (effects (font (size 1.27 1.27)) (justify right))
     )
-    (property "Digi-Key PN" "399-7845-1-ND" (at -5.969 235.077 0)
+    (property "Digi-Key PN" "1276-1935-1-ND" (at -5.969 235.077 0)
       (effects (font (size 1.27 1.27)) hide)
     )
@@
       (effects (font (size 1.27 1.27)) (justify right))
     )
-    (property "Digi-Key PN" "399-7845-1-ND" (at 95.631 235.077 0)
+    (property "Digi-Key PN" "1276-1935-1-ND" (at 95.631 235.077 0)
       (effects (font (size 1.27 1.27)) hide)
     )
@@
       (effects (font (size 1.27 1.27)) (justify right))
     )
-    (property "Digi-Key PN" "399-7845-1-ND" (at -28.194 210.312 0)
-      (effects (font (size 1.27 1.27)) hide)
-    )
+    (property "Digi-Key PN" "1276-1935-1-ND" (at -28.194 210.312 0)
+      (effects (font (size 1.27 1.27)) hide)
+    )
