File: hdw/USB_Hub/Pushbuttons.kicad_sch (KiCad schematic)
At the start: 10 parts

Commit message: lots of schematic progress
Other:
- title: Analog Clock -> USB Hub
Changed lines of the file:
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@@
   (paper "A")
   (title_block
-    (title "Analog Clock")
-    (date "2020-08-15")
-    (rev "A")
+    (title "USB Hub")
+    (date "2023-08-18")
+    (rev "PRELIM")
     (company "Drew Maatman")
   )

Commit message: much more schematic progress
Parts:
- removed C?: 10nF, Capacitors_SMD:C_0603, symbol Custom_Library:C_Custom
- removed C?: 0.1uF, Capacitors_SMD:C_0603, symbol Custom_Library:C_Custom
- removed R?: 499, Resistors_SMD:R_0603, symbol Custom_Library:R_Custom
- removed SW?: Cap_Touch, Custom Footprints Library:Capacitive_Touch_Pad, symbol Custom_Library:Cap_Touch
- removed U?: AT42QT1010-TSHR, TO_SOT_Packages_SMD:SOT-23-6, symbol Sensor_Touch:AT42QT1010-TSHR
- added C? (x2): 10nF, Capacitors_SMD:C_0603, symbol Custom_Library:C_Custom
- added C? (x5): 0.1uF, Capacitors_SMD:C_0603, symbol Custom_Library:C_Custom
- added R? (x3): 10k, Resistors_SMD:R_0402, symbol Custom_Library:R_Custom
- added R? (x2): 499, Resistors_SMD:R_0603, symbol Custom_Library:R_Custom
- added SW? (x2): Cap_Touch, Custom Footprints Library:Capacitive_Touch_Pad, symbol Custom_Library:Cap_Touch
- added U? (x2): AT42QT1010-TSHR, TO_SOT_Packages_SMD:SOT-23-6, symbol Sensor_Touch:AT42QT1010-TSHR
Connections:
- net +3.3V: now also C?.1, C?.1, U?.5 (VDD), U?.5 (VDD), U?.6 (SYNC), U?.6 (SYNC)
- net GND: now also C?.2, C?.2, C?.2, C?.2, C?.2, R?.2, R?.2, R?.2, U?.2 (VSS), U?.2 (VSS)
- net CAP_TOUCH_LEFT: now reaches U?.1 (OUT)
- net CAP_TOUCH_LEFT: now also C?.1, R?.1
- new net: C?.1, U?.4 (SNS) (x2)
- new net: C?.2, R?.2, U?.3 (SNSK) (x2)
- new net: R?.1, SW?.1 (TP) (x2)
- new net CAP_TOUCH_POWER: C?.1, R?.1, U?.1 (OUT)
- new net CAP_TOUCH_RIGHT: C?.1, R?.1, U?.1 (OUT)
Other:
- moved on the sheet: C?, R?, SW?, U?

Commit message: lots and lots of sch progress
Parts:
- gave numbers to parts that had none: 18

Commit message: pulled footprints into layout
Parts:
- C1601, C1602, C1603, C1607, C1608, C1609: Digi-Key PN 399-7845-1-ND -> 1276-1935-1-ND
- R1601, R1602, R1603: Digi-Key PN RMCF0603FT499RCT-ND -> (none)
- R? (x3): Digi-Key PN RMCF0402FT10K0CT-ND -> (none); Wattage 1/16W -> 1/10W; display_footprint 0402 -> 0603
Changed lines of the file:
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@@
       (effects (font (size 1.27 1.27)) hide)
     )
-    (property "Digi-Key PN" "RMCF0603FT499RCT-ND" (at 76.835 49.53 0)
+    (property "Digi-Key PN" "" (at 76.835 49.53 0)
       (effects (font (size 1.524 1.524)) hide)
     )
@@
       (effects (font (size 1.27 1.27)) hide)
     )
-    (property "Digi-Key PN" "399-7845-1-ND" (at 80.01 13.97 0)
+    (property "Digi-Key PN" "1276-1935-1-ND" (at 80.01 13.97 0)
       (effects (font (size 1.524 1.524)) hide)
     )
@@
       (effects (font (size 1.27 1.27)) hide)
     )
-    (property "Digi-Key PN" "399-7845-1-ND" (at 131.445 90.17 0)
+    (property "Digi-Key PN" "1276-1935-1-ND" (at 131.445 90.17 0)
       (effects (font (size 1.524 1.524)) hide)
     )
@@
       (effects (font (size 1.27 1.27)) hide)
     )
-    (property "display_footprint" "0402" (at 159.512 151.638 0)
+    (property "display_footprint" "0603" (at 159.512 151.638 0)
       (effects (font (size 1.27 1.27)) (justify left))
     )
@@
       (effects (font (size 1.27 1.27)) (justify left))
     )
-    (property "Wattage" "1/16W" (at 159.512 155.448 0)
-      (effects (font (size 1.27 1.27)) (justify left))
-    )
-    (property "Digi-Key PN" "RMCF0402FT10K0CT-ND" (at 161.29 153.67 0)
+    (property "Wattage" "1/10W" (at 159.512 155.448 0)
+      (effects (font (size 1.27 1.27)) (justify left))
+    )
+    (property "Digi-Key PN" "" (at 161.29 153.67 0)
       (effects (font (size 1.27 1.27)) hide)
     )
@@
       (effects (font (size 1.27 1.27)) hide)
     )
-    (property "display_footprint" "0402" (at 159.512 100.838 0)
+    (property "display_footprint" "0603" (at 159.512 100.838 0)
       (effects (font (size 1.27 1.27)) (justify left))
     )
@@
       (effects (font (size 1.27 1.27)) (justify left))
     )
-    (property "Wattage" "1/16W" (at 159.512 104.648 0)
-      (effects (font (size 1.27 1.27)) (justify left))
-    )
-    (property "Digi-Key PN" "RMCF0402FT10K0CT-ND" (at 161.29 102.87 0)
+    (property "Wattage" "1/10W" (at 159.512 104.648 0)
+      (effects (font (size 1.27 1.27)) (justify left))
+    )
+    (property "Digi-Key PN" "" (at 161.29 102.87 0)
       (effects (font (size 1.27 1.27)) hide)
     )
@@
       (effects (font (size 1.27 1.27)) hide)
     )
-    (property "Digi-Key PN" "399-7845-1-ND" (at 131.445 140.97 0)
+    (property "Digi-Key PN" "1276-1935-1-ND" (at 131.445 140.97 0)
       (effects (font (size 1.524 1.524)) hide)
     )
@@
       (effects (font (size 1.27 1.27)) hide)
     )
-    (property "Digi-Key PN" "RMCF0603FT499RCT-ND" (at 76.835 151.13 0)
+    (property "Digi-Key PN" "" (at 76.835 151.13 0)
       (effects (font (size 1.524 1.524)) hide)
     )
@@
       (effects (font (size 1.27 1.27)) hide)
     )
-    (property "Digi-Key PN" "399-7845-1-ND" (at 80.01 115.57 0)
+    (property "Digi-Key PN" "1276-1935-1-ND" (at 80.01 115.57 0)
       (effects (font (size 1.524 1.524)) hide)
     )
@@
       (effects (font (size 1.27 1.27)) hide)
     )
-    (property "Digi-Key PN" "RMCF0603FT499RCT-ND" (at 76.835 100.33 0)
+    (property "Digi-Key PN" "" (at 76.835 100.33 0)
       (effects (font (size 1.524 1.524)) hide)
     )
@@
       (effects (font (size 1.27 1.27)) hide)
     )
-    (property "display_footprint" "0402" (at 159.512 50.038 0)
+    (property "display_footprint" "0603" (at 159.512 50.038 0)
       (effects (font (size 1.27 1.27)) (justify left))
     )
@@
       (effects (font (size 1.27 1.27)) (justify left))
     )
-    (property "Wattage" "1/16W" (at 159.512 53.848 0)
-      (effects (font (size 1.27 1.27)) (justify left))
-    )
-    (property "Digi-Key PN" "RMCF0402FT10K0CT-ND" (at 161.29 52.07 0)
+    (property "Wattage" "1/10W" (at 159.512 53.848 0)
+      (effects (font (size 1.27 1.27)) (justify left))
+    )
+    (property "Digi-Key PN" "" (at 161.29 52.07 0)
       (effects (font (size 1.27 1.27)) hide)
     )
@@
       (effects (font (size 1.27 1.27)) hide)
     )
-    (property "Digi-Key PN" "399-7845-1-ND" (at 131.445 39.37 0)
+    (property "Digi-Key PN" "1276-1935-1-ND" (at 131.445 39.37 0)
       (effects (font (size 1.524 1.524)) hide)
     )
@@
       (effects (font (size 1.27 1.27)) hide)
     )
-    (property "Digi-Key PN" "399-7845-1-ND" (at 80.01 64.77 0)
+    (property "Digi-Key PN" "1276-1935-1-ND" (at 80.01 64.77 0)
       (effects (font (size 1.524 1.524)) hide)
     )
