File: hdw/USB_Hub/Status_LEDs.kicad_sch (KiCad schematic)
At the start: 15 parts

Commit message: lots of schematic progress
Other:
- title: Analog Clock -> USB Hub
Changed lines of the file:
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@@
   (paper "A")
   (title_block
-    (title "Analog Clock")
-    (date "2020-08-15")
-    (rev "A")
+    (title "USB Hub")
+    (date "2023-08-18")
+    (rev "PRELIM")
     (company "Drew Maatman")
   )

Commit message: much more schematic progress
Parts:
- removed U? (x3): 74LVC1G06, TO_SOT_Packages_SMD:SOT-353_SC-70-5, symbol Custom_Library:74LVC1G06_Power
- added U? (x3): 74LVC1G97, Package_TO_SOT_SMD:SOT-363_SC-70-6, symbol Custom Library:74LVC1G97_Power_NOT
Connections:
- net +3.3V: now also U?.1 (VCC), U?.1 (VCC), U?.1 (VCC), U?.5 (VCC), U?.5 (VCC), U?.5 (VCC)
- net Error_LED: now also U?.6
- net GND: now also U?.2 (GND), U?.2 (GND), U?.2 (GND), U?.3 (GND), U?.3 (GND), U?.3 (GND)
- net Heartbeat_LED: now also U?.6
- net Reset_LED: now also U?.6
- net at D?.1 (K): now also U?.4 (x3)

Commit message: lots and lots of sch progress
Parts:
- gave numbers to parts that had none: 15

Commit message: pulled footprints into layout
Parts:
- C1301, C1302, C1303: Digi-Key PN 399-7845-1-ND -> 1276-1935-1-ND
- R1301, R1302, R1305: Digi-Key PN YAG2321CT-ND -> (none)
- R1303, R1304, R1306: Digi-Key PN 311-1.00KHRCT-ND -> (none)
- U1301, U1302, U1303: Digi-Key PN (none) -> 296-15582-1-ND
Changed lines of the file:
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@@
       (effects (font (size 1.27 1.27)) hide)
     )
-    (property "Digi-Key PN" "399-7845-1-ND" (at 89.535 40.005 0)
+    (property "Digi-Key PN" "1276-1935-1-ND" (at 89.535 40.005 0)
       (effects (font (size 1.524 1.524)) hide)
     )
@@
       (effects (font (size 1.27 1.27)) (justify left))
     )
-    (property "Digi-Key PN" "311-1.00KHRCT-ND" (at 109.855 45.72 0)
+    (property "Digi-Key PN" "" (at 109.855 45.72 0)
       (effects (font (size 1.524 1.524)) hide)
     )
@@
       (effects (font (size 1.27 1.27)) (justify left))
     )
-    (property "Digi-Key PN" "YAG2321CT-ND" (at 88.9 76.2 0)
+    (property "Digi-Key PN" "" (at 88.9 76.2 0)
       (effects (font (size 1.27 1.27)) hide)
     )
@@
       (effects (font (size 1.27 1.27)) hide)
     )
-    (property "Digi-Key PN" "399-7845-1-ND" (at 140.335 40.005 0)
+    (property "Digi-Key PN" "1276-1935-1-ND" (at 140.335 40.005 0)
       (effects (font (size 1.524 1.524)) hide)
     )
@@
       (effects (font (size 1.27 1.27)) (justify left))
     )
-    (property "Digi-Key PN" "311-1.00KHRCT-ND" (at 160.655 45.72 0)
+    (property "Digi-Key PN" "" (at 160.655 45.72 0)
       (effects (font (size 1.524 1.524)) hide)
     )
@@
       (effects (font (size 1.27 1.27)) (justify left))
     )
-    (property "Digi-Key PN" "YAG2321CT-ND" (at 139.7 64.135 0)
+    (property "Digi-Key PN" "" (at 139.7 64.135 0)
       (effects (font (size 1.27 1.27)) hide)
     )
@@
       (effects (font (size 1.27 1.27)) hide)
     )
-    (property "Digi-Key PN" "399-7845-1-ND" (at 89.535 90.805 0)
+    (property "Digi-Key PN" "1276-1935-1-ND" (at 89.535 90.805 0)
       (effects (font (size 1.524 1.524)) hide)
     )
@@
       (effects (font (size 1.27 1.27)) (justify left))
     )
-    (property "Digi-Key PN" "311-1.00KHRCT-ND" (at 109.855 96.52 0)
+    (property "Digi-Key PN" "" (at 109.855 96.52 0)
       (effects (font (size 1.524 1.524)) hide)
     )
@@
       (effects (font (size 1.27 1.27)) (justify left))
     )
-    (property "Digi-Key PN" "YAG2321CT-ND" (at 88.9 127 0)
+    (property "Digi-Key PN" "" (at 88.9 127 0)
       (effects (font (size 1.27 1.27)) hide)
     )
@@
     )
     (property "Datasheet" "http://www.ti.com/lit/ds/symlink/sn74lvc1g97.pdf" (at 104.14 69.85 0)
+      (effects (font (size 1.27 1.27)) hide)
+    )
+    (property "Digi-Key PN" "296-15582-1-ND" (at 102.87 69.85 0)
       (effects (font (size 1.27 1.27)) hide)
     )
@@
       (effects (font (size 1.27 1.27)) hide)
     )
+    (property "Digi-Key PN" "296-15582-1-ND" (at 102.87 120.65 0)
+      (effects (font (size 1.27 1.27)) hide)
+    )
     (pin "1")
     (pin "2")
@@
       (effects (font (size 1.27 1.27)) hide)
     )
+    (property "Digi-Key PN" "296-15582-1-ND" (at 153.67 69.85 0)
+      (effects (font (size 1.27 1.27)) hide)
+    )
