File: hdw/USB_Hub/USB_UART_Bridge.kicad_sch (KiCad schematic)
At the start: 40 parts

Commit message: schematic progress
Parts:
- removed C? (x2): 47pF, Capacitors_SMD:C_0603, symbol Custom_Library:C_Custom
- removed C? (x9): 0.1uF, Capacitors_SMD:C_0603, symbol Custom_Library:C_Custom
- removed C?: 10uF, Capacitors_SMD:C_0603, symbol Custom_Library:C_Custom
- removed C?: 10uF, Capacitors_SMD:C_0805, symbol Custom_Library:C_Custom
- removed D?: Yellow, LEDs:LED_0603, symbol Device:LED
- removed DOC?: COM_Port_Settings, symbol Custom_Library:COM_Port_Settings
- removed J?: USB_B_Mini, Connectors:USB_Mini-B, symbol Connector:USB_B_Mini
- removed L? (x2): 600R 0.5A, Inductors_SMD:L_0603, symbol Device:Ferrite_Bead
- removed R? (x2): 1k, Resistors_SMD:R_0603, symbol Custom_Library:R_Custom
- removed R? (x2): 27, Resistors_SMD:R_0603, symbol Custom_Library:R_Custom
- removed R?: 6.04k, Resistors_SMD:R_0603, symbol Custom_Library:R_Custom
- removed R?: 40.2k, Resistors_SMD:R_0603, symbol Custom_Library:R_Custom
- removed R?: 487k, Resistors_SMD:R_0603, symbol Custom_Library:R_Custom
- removed R? (x2): 10k, Resistors_SMD:R_0603, symbol Custom_Library:R_Custom
- removed R?: 0.02, Resistors_SMD:R_0612, symbol Custom_Library:R_Custom
- removed R? (x2): 10, Resistors_SMD:R_0603, symbol Custom_Library:R_Custom
- removed R? (x4): 100k, Resistors_SMD:R_0603, symbol Custom_Library:R_Custom
- removed TP?: TP, Custom Footprints Library:Test_Point, symbol Custom_Library:TP
- removed U?: FT234XD, Housings_DFN_QFN:DFN-12-1EP_3x3mm_Pitch0.45mm, symbol Custom_Library:FT234XD
- removed U?: TPD3S014DBVR, TO_SOT_Packages_SMD:SOT-23-6, symbol Custom_Library:TPD3S014DBVR
- removed U?: TLV6700, Package_TO_SOT_SMD:SOT-23-6, symbol Custom_Library:TLV6700
- removed U?: TXB0102DCU, Package_SO:VSSOP-8_2.4x2.1mm_P0.5mm, symbol Logic_LevelTranslator:TXB0102DCU
- removed U?: 74LVC1G17, TO_SOT_Packages_SMD:SOT-353_SC-70-5, symbol Custom_Library:74LVC1G17_Power
- added C? (x3): 10uF, Capacitors_SMD:C_0603, symbol Custom_Library:C_Custom
- added C? (x8): 0.1uF, Capacitors_SMD:C_0603, symbol Custom_Library:C_Custom
- added C? (x2): 47pF, Capacitors_SMD:C_0603, symbol Custom_Library:C_Custom
- added D?: Yellow, LEDs:LED_0603, symbol Device:LED
- added D?: Green, LEDs:LED_0603, symbol Device:LED
- added DOC?: COM_Port_Settings, symbol Custom_Library:COM_Port_Settings
- added J?: USB_B_Mini, Connectors:USB_Mini-B, symbol Connector:USB_B_Mini
- added L? (x2): 600R 0.5A, Inductors_SMD:L_0603, symbol Device:Ferrite_Bead
- added R? (x4): 100k, Resistors_SMD:R_0603, symbol Custom_Library:R_Custom
- added R?: 10k, Resistors_SMD:R_0603, symbol Custom_Library:R_Custom
- added R?: 487k, Resistors_SMD:R_0603, symbol Custom_Library:R_Custom
- added R?: 40.2k, Resistors_SMD:R_0603, symbol Custom_Library:R_Custom
- added R? (x2): 27, Resistors_SMD:R_0603, symbol Custom_Library:R_Custom
- added R?: 6.04k, Resistors_SMD:R_0603, symbol Custom_Library:R_Custom
- added R? (x2): 1k, Resistors_SMD:R_0603, symbol Custom_Library:R_Custom
- added TP?: TP, Custom Footprints Library:Test_Point, symbol Custom_Library:TP
- added U1303: 74LVC1G97, Package_TO_SOT_SMD:SOT-363_SC-70-6, symbol Custom Library:74LVC1G97_Power_NOT
- added U1304: ISO7321C, Package_SO:SOIC-8_3.9x4.9mm_P1.27mm, symbol Isolator:ISO7321C
- added U?: FT234XD, Housings_DFN_QFN:DFN-12-1EP_3x3mm_Pitch0.45mm, symbol Custom_Library:FT234XD
- added U?: TLV6700, Package_TO_SOT_SMD:SOT-23-6, symbol Custom_Library:TLV6700
- added U?: TPD3S014DBVR, TO_SOT_Packages_SMD:SOT-23-6, symbol Custom_Library:TPD3S014DBVR
Connections:
- net +3.3V: now also C?.1, C?.1, R?.1, R?.1, U1304.1 (VCC1)
- net +3.3V_USB: now also C?.1, C?.1, C?.1, C?.1, C?.1, C?.1, R?.1, R?.1, R?.1, R?.1, U1303.1 (VCC), U1303.5 (VCC), U1304.8 (VCC2), U?.3 (3V3OUT), U?.5 (Vs), U?.9 (VCCIO)
- net +5V_USB: now also C?.1, C?.1, C?.1, R?.1, R?.1, TP?.1 (TP), U?.4 (OUT), U?.4 (VCC)
- net BRIDGE_USB+: now also R?.2, U?.12 (USBDP)
- net BRIDGE_USB-: now also R?.2, U?.1 (USBDM)
- net CONN_USB+: now also C?.1, J?.3 (D+), R?.1, U?.6 (D1)
- net CONN_USB-: now also C?.1, J?.2 (D-), R?.1, U?.5 (D2)
- net GND: now also C?.2, C?.2, U1304.4 (GND1)
- net POS5_USB_PGOOD: now also R?.2, U1303.6, U?.1 (OUTA), U?.6 (OUTB)
- net USB_UART_RX: now also R?.2, U1304.2 (OUTA)
- net USB_UART_TX: now also R?.2, U1304.3 (INB)
- net ~{USB_ACTIVE}: now also D?.1 (K), U?.6 (CBUS0)
- new net: D?.1 (K), U1303.4
- new net: R?.1, R?.2, U?.3 (+INA)
- new net: J?.6 (Shield), L?.2
- new net: J?.1 (VBUS), L?.1
- new net: L?.2, U?.1 (EN), U?.3 (IN)
- new net: R?.1, R?.2, U?.4 (-INB)
- new net: D?.2 (A), R?.2 (x2)
- new net GND_USB: C?.2, C?.2, C?.2, C?.2, C?.2, C?.2, C?.2, C?.2, C?.2, C?.2, C?.2, J?.5 (GND), L?.1, R?.2, U1303.2 (GND), U1303.3 (GND), U1304.5 (GND2), U?.13 (GND), U?.2 (GND), U?.2 (GND), U?.5 (GND)
- new net USB_UART_RX_ISO: R?.2, U1304.7 (INA), U?.7 (TXD)
- new net USB_UART_TX_ISO: R?.2, U1304.6 (OUTB), U?.10 (RXD)
Other:
- note added: "Switch to Non-Isolated"
- note removed: "VERIFY BUFFER PINOUT/FOOTPRINT"

Commit message: lots of schematic progress
Other:
- title: Analog Clock -> USB Hub
Changed lines of the file:
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@@
   (paper "A")
   (title_block
-    (title "Analog Clock")
-    (date "2020-08-15")
-    (rev "A")
+    (title "USB Hub")
+    (date "2023-08-18")
+    (rev "PRELIM")
     (company "Drew Maatman")
   )

Commit message: much more schematic progress
Parts:
- removed C? (x3): 10uF, Capacitors_SMD:C_0603, symbol Custom_Library:C_Custom
- removed C? (x8): 0.1uF, Capacitors_SMD:C_0603, symbol Custom_Library:C_Custom
- removed C? (x2): 47pF, Capacitors_SMD:C_0603, symbol Custom_Library:C_Custom
- removed D?: Yellow, LEDs:LED_0603, symbol Device:LED
- removed D?: Green, LEDs:LED_0603, symbol Device:LED
- removed DOC?: COM_Port_Settings, symbol Custom_Library:COM_Port_Settings
- removed J?: USB_B_Mini, Connectors:USB_Mini-B, symbol Connector:USB_B_Mini
- removed L? (x2): 600R 0.5A, Inductors_SMD:L_0603, symbol Device:Ferrite_Bead
- removed R? (x4): 100k, Resistors_SMD:R_0603, symbol Custom_Library:R_Custom
- removed R?: 10k, Resistors_SMD:R_0603, symbol Custom_Library:R_Custom
- removed R?: 487k, Resistors_SMD:R_0603, symbol Custom_Library:R_Custom
- removed R?: 40.2k, Resistors_SMD:R_0603, symbol Custom_Library:R_Custom
- removed R? (x2): 27, Resistors_SMD:R_0603, symbol Custom_Library:R_Custom
- removed R?: 6.04k, Resistors_SMD:R_0603, symbol Custom_Library:R_Custom
- removed R? (x2): 1k, Resistors_SMD:R_0603, symbol Custom_Library:R_Custom
- removed TP?: TP, Custom Footprints Library:Test_Point, symbol Custom_Library:TP
- removed U1303: 74LVC1G97, Package_TO_SOT_SMD:SOT-363_SC-70-6, symbol Custom Library:74LVC1G97_Power_NOT
- removed U1304: ISO7321C, Package_SO:SOIC-8_3.9x4.9mm_P1.27mm, symbol Isolator:ISO7321C
- removed U?: FT234XD, Housings_DFN_QFN:DFN-12-1EP_3x3mm_Pitch0.45mm, symbol Custom_Library:FT234XD
- removed U?: TLV6700, Package_TO_SOT_SMD:SOT-23-6, symbol Custom_Library:TLV6700
- removed U?: TPD3S014DBVR, TO_SOT_Packages_SMD:SOT-23-6, symbol Custom_Library:TPD3S014DBVR
- added C1301, C1302, C1306, C1307, C1310, C1312, C?: 0.1uF, Capacitors_SMD:C_0603, symbol Custom_Library:C_Custom
- added C1309, C1311: 47pF, Capacitors_SMD:C_0603, symbol Custom_Library:C_Custom
- added C?: 10uF, Capacitors_SMD:C_0603, symbol Custom_Library:C_Custom
- added D1301: Yellow, LEDs:LED_0603, symbol Device:LED
- added DOC1301: COM_Port_Settings, symbol Custom_Library:COM_Port_Settings
- added J1301: USB_B_Mini, Connectors:USB_Mini-B, symbol Connector:USB_B_Mini
- added L1301, L1302: 600R 0.5A, Inductors_SMD:L_0603, symbol Device:Ferrite_Bead
- added R1301: 1k, Resistors_SMD:R_0603, symbol Custom_Library:R_Custom
- added R1302: 487k, Resistors_SMD:R_0603, symbol Custom_Library:R_Custom
- added R1303: 6.04k, Resistors_SMD:R_0603, symbol Custom_Library:R_Custom
- added R1304: 40.2k, Resistors_SMD:R_0603, symbol Custom_Library:R_Custom
- added R1305: 10k, Resistors_SMD:R_0603, symbol Custom_Library:R_Custom
- added R1306, R1308, R1314, R1315: 100k, Resistors_SMD:R_0603, symbol Custom_Library:R_Custom
- added R1311, R1312: 27, Resistors_SMD:R_0603, symbol Custom_Library:R_Custom
- added TP?: TP, Custom Footprints Library:Test_Point, symbol Custom_Library:TP
- added U1301: TLV6700, Package_TO_SOT_SMD:SOT-23-6, symbol Custom_Library:TLV6700
- added U1302: FT234XD, Housings_DFN_QFN:DFN-12-1EP_3x3mm_Pitch0.45mm, symbol Custom_Library:FT234XD
- added U1304: TXB0102DCU, Package_SO:VSSOP-8_2.4x2.1mm_P0.5mm, symbol Logic_LevelTranslator:TXB0102DCU
- added U1305: TPD3S014DBVR, TO_SOT_Packages_SMD:SOT-23-6, symbol Custom_Library:TPD3S014DBVR
Connections:
- net +3.3V: now also C1310.1, C?.1, R1305.1, R1306.1, R1308.1, U1301.5 (Vs), U1304.3 (VCCA)
- net +3.3V_USB: now also C1301.1, C1307.1, C1312.1, R1314.1, R1315.1, U1302.3 (3V3OUT), U1302.9 (VCCIO), U1304.7 (VCCB)
- net +5V_USB: now also C1302.1, C1306.1, C?.1, R1301.1, R1302.1, TP?.1 (TP), U1302.4 (VCC), U1305.4 (OUT)
- net BRIDGE_USB+: now also R1311.2, U1302.12 (USBDP)
- net BRIDGE_USB-: now also R1312.2, U1302.1 (USBDM)
- net CONN_USB+: now also C1309.1, J1301.3 (D+), R1311.1, U1305.6 (D1)
- net CONN_USB-: now also C1311.1, J1301.2 (D-), R1312.1, U1305.5 (D2)
- net GND: now also C1301.2, C1302.2, C1306.2, C1307.2, C1309.2, C1310.2, C1311.2, C1312.2, C?.2, C?.2, J1301.5 (GND), L1302.1, R1304.2, U1301.2 (GND), U1302.13 (GND), U1302.5 (GND), U1304.2 (GND), U1305.2 (GND)
- net POS5_USB_PGOOD: now also R1305.2, U1301.1 (OUTA), U1301.6 (OUTB), U1304.6 (OE)
- net USB_UART_RX: now also R1308.2, U1304.5 (A1)
- net USB_UART_TX: now also R1306.2, U1304.4 (A2)
- net ~{USB_ACTIVE}: now also D1301.1 (K), U1302.6 (CBUS0)
- new net: D1301.2 (A), R1301.2
- new net: J1301.6 (Shield), L1302.2
- new net: J1301.1 (VBUS), L1301.1
- new net: L1301.2, U1305.1 (EN), U1305.3 (IN)
- new net: R1303.2, R1304.1, U1301.4 (-INB)
- new net: R1302.2, R1303.1, U1301.3 (+INA)
- new net USB_UART_RX_BUF: R1314.2, U1302.7 (TXD), U1304.8 (B1)
- new net USB_UART_TX_BUF: R1315.2, U1302.10 (RXD), U1304.1 (B2)
Other:
- note removed: "Switch to Non-Isolated"

Commit message: lots and lots of sch progress
Parts:
- removed L1302: 600R 0.5A, Inductors_SMD:L_0603, symbol Device:Ferrite_Bead
- renumbered C1307 to C?, C1301 to C?, C1306 to C?, C1302 to C?, C1310 to C?, C1309 to C?, C1312 to C?, C1311 to C?, D1301 to D?, DOC1301 to DOC?, J1301 to J?, L1301 to L?, R1314 to R?, R1312 to R?, R1301 to R?, R1311 to R?, R1304 to R?, R1303 to R?, R1308 to R?, R1302 to R?, R1305 to R?, R1306 to R?, R1315 to R?, U1305 to U?, U1304 to U?, U1302 to U?, U1301 to U?
Connections:
- net CHASSIS: now reaches J?.6 (Shield)

Commit message: pulled footprints into layout
Parts:
- C? (x7): Digi-Key PN 399-7845-1-ND -> 1276-1935-1-ND
- C?: Digi-Key PN 490-10474-1-ND -> 1276-1871-1-ND
- R? (x4): Digi-Key PN RMCF0603FT100KCT-ND -> (none)
- R? (x2): Digi-Key PN 311-27.0HRCT-ND -> (none)
- R?: Digi-Key PN 311-1.00KHRCT-ND -> (none)
- R?: Digi-Key PN RMCF0603FT40K2CT-ND -> (none)
- R?: Digi-Key PN RMCF0603FT6K04CT-ND -> (none)
- R?: Digi-Key PN 311-487KHRCT-ND -> (none)
- R?: Digi-Key PN YAG2321CT-ND -> (none)
Changed lines of the file:
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@@
       (effects (font (size 1.27 1.27)) (justify right))
     )
-    (property "Digi-Key PN" "399-7845-1-ND" (at 120.015 118.745 0)
+    (property "Digi-Key PN" "1276-1935-1-ND" (at 120.015 118.745 0)
       (effects (font (size 1.524 1.524)) hide)
     )
@@
       (effects (font (size 1.27 1.27)) (justify left))
     )
-    (property "Digi-Key PN" "RMCF0603FT100KCT-ND" (at 154.94 27.94 0)
+    (property "Digi-Key PN" "" (at 154.94 27.94 0)
       (effects (font (size 1.27 1.27)) hide)
     )
@@
       (effects (font (size 1.27 1.27)))
     )
-    (property "Digi-Key PN" "311-27.0HRCT-ND" (at 137.16 125.095 0)
+    (property "Digi-Key PN" "" (at 137.16 125.095 0)
       (effects (font (size 1.524 1.524)) hide)
     )
@@
       (effects (font (size 1.27 1.27)) (justify left))
     )
-    (property "Digi-Key PN" "311-1.00KHRCT-ND" (at 28.575 99.06 0)
+    (property "Digi-Key PN" "" (at 28.575 99.06 0)
       (effects (font (size 1.524 1.524)) hide)
     )
@@
       (effects (font (size 1.27 1.27)))
     )
-    (property "Digi-Key PN" "311-27.0HRCT-ND" (at 137.16 107.315 0)
+    (property "Digi-Key PN" "" (at 137.16 107.315 0)
       (effects (font (size 1.524 1.524)) hide)
     )
@@
       (effects (font (size 1.27 1.27)) (justify right))
     )
-    (property "Digi-Key PN" "399-7845-1-ND" (at 50.165 76.2 0)
+    (property "Digi-Key PN" "1276-1935-1-ND" (at 50.165 76.2 0)
       (effects (font (size 1.524 1.524)) hide)
     )
@@
       (effects (font (size 1.27 1.27)) (justify left))
     )
-    (property "Digi-Key PN" "RMCF0603FT40K2CT-ND" (at 49.53 172.72 0)
+    (property "Digi-Key PN" "" (at 49.53 172.72 0)
       (effects (font (size 1.524 1.524)) hide)
     )
@@
       (effects (font (size 1.27 1.27)) (justify right))
     )
-    (property "Digi-Key PN" "399-7845-1-ND" (at 137.795 80.01 0)
+    (property "Digi-Key PN" "1276-1935-1-ND" (at 137.795 80.01 0)
       (effects (font (size 1.524 1.524)) hide)
     )
@@
       (effects (font (size 1.27 1.27)) (justify left))
     )
-    (property "Digi-Key PN" "RMCF0603FT6K04CT-ND" (at 49.53 160.02 0)
+    (property "Digi-Key PN" "" (at 49.53 160.02 0)
       (effects (font (size 1.524 1.524)) hide)
     )
@@
       (effects (font (size 1.27 1.27)) (justify right))
     )
-    (property "Digi-Key PN" "399-7845-1-ND" (at 67.945 76.2 0)
+    (property "Digi-Key PN" "1276-1935-1-ND" (at 67.945 76.2 0)
       (effects (font (size 1.524 1.524)) hide)
     )
@@
       (effects (font (size 1.27 1.27)) (justify right))
     )
-    (property "Digi-Key PN" "490-10474-1-ND" (at 74.295 88.9 0)
+    (property "Digi-Key PN" "1276-1871-1-ND" (at 74.295 88.9 0)
       (effects (font (size 1.27 1.27)) hide)
     )
@@
       (effects (font (size 1.27 1.27)) hide)
     )
-    (property "Digi-Key PN" "399-7845-1-ND" (at 74.295 175.895 0)
+    (property "Digi-Key PN" "1276-1935-1-ND" (at 74.295 175.895 0)
       (effects (font (size 1.524 1.524)) hide)
     )
@@
       (effects (font (size 1.27 1.27)) (justify left))
     )
-    (property "Digi-Key PN" "RMCF0603FT100KCT-ND" (at 111.125 27.94 0)
+    (property "Digi-Key PN" "" (at 111.125 27.94 0)
       (effects (font (size 1.27 1.27)) hide)
     )
@@
       (effects (font (size 1.27 1.27)) (justify left))
     )
-    (property "Digi-Key PN" "311-487KHRCT-ND" (at 49.53 146.05 0)
+    (property "Digi-Key PN" "" (at 49.53 146.05 0)
       (effects (font (size 1.524 1.524)) hide)
     )
@@
       (effects (font (size 1.27 1.27)) (justify right))
     )
-    (property "Digi-Key PN" "399-7845-1-ND" (at 162.56 38.1 0)
+    (property "Digi-Key PN" "1276-1935-1-ND" (at 162.56 38.1 0)
       (effects (font (size 1.524 1.524)) hide)
     )
@@
       (effects (font (size 1.27 1.27)) (justify right))
     )
-    (property "Digi-Key PN" "399-7845-1-ND" (at 180.34 38.1 0)
+    (property "Digi-Key PN" "1276-1935-1-ND" (at 180.34 38.1 0)
       (effects (font (size 1.524 1.524)) hide)
     )
@@
       (effects (font (size 1.27 1.27)) (justify left))
     )
-    (property "Digi-Key PN" "YAG2321CT-ND" (at 91.44 144.78 0)
+    (property "Digi-Key PN" "" (at 91.44 144.78 0)
       (effects (font (size 1.524 1.524)) hide)
     )
@@
       (effects (font (size 1.27 1.27)) (justify left))
     )
-    (property "Digi-Key PN" "RMCF0603FT100KCT-ND" (at 97.79 27.94 0)
+    (property "Digi-Key PN" "" (at 97.79 27.94 0)
       (effects (font (size 1.27 1.27)) hide)
     )
@@
       (effects (font (size 1.27 1.27)) (justify left))
     )
-    (property "Digi-Key PN" "RMCF0603FT100KCT-ND" (at 168.275 27.94 0)
-      (effects (font (size 1.27 1.27)) hide)
-    )
+    (property "Digi-Key PN" "" (at 168.275 27.94 0)
+      (effects (font (size 1.27 1.27)) hide)
+    )
