File: hdw/USB_Hub/mechanical.kicad_sch (KiCad schematic)
At the start: 12 parts

Commit message: pulled footprints into layout
Parts:
- H? (x4): footprint Mounting_Holes:MountingHole_3mm_Pad_Via -> MountingHole:MountingHole_3mm
Changed lines of the file:
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@@
       (effects (font (size 1.27 1.27)))
     )
-    (property "Footprint" "Mounting_Holes:MountingHole_3mm_Pad_Via" (at 139.7 66.675 0)
+    (property "Footprint" "MountingHole:MountingHole_3mm" (at 139.7 66.675 0)
       (effects (font (size 1.27 1.27)) hide)
     )
@@
       (effects (font (size 1.27 1.27)))
     )
-    (property "Footprint" "Mounting_Holes:MountingHole_3mm_Pad_Via" (at 114.3 66.675 0)
+    (property "Footprint" "MountingHole:MountingHole_3mm" (at 114.3 66.675 0)
       (effects (font (size 1.27 1.27)) hide)
     )
@@
       (effects (font (size 1.27 1.27)))
     )
-    (property "Footprint" "Mounting_Holes:MountingHole_3mm_Pad_Via" (at 114.3 46.355 0)
+    (property "Footprint" "MountingHole:MountingHole_3mm" (at 114.3 46.355 0)
       (effects (font (size 1.27 1.27)) hide)
     )
@@
       (effects (font (size 1.27 1.27)))
     )
-    (property "Footprint" "Mounting_Holes:MountingHole_3mm_Pad_Via" (at 139.7 46.355 0)
-      (effects (font (size 1.27 1.27)) hide)
-    )
+    (property "Footprint" "MountingHole:MountingHole_3mm" (at 139.7 46.355 0)
+      (effects (font (size 1.27 1.27)) hide)
+    )
