File: hdw/USB_Hub/Hub_Controller.kicad_sch (KiCad schematic)
At the start: 25 parts, among them SW901 RESET, U902 TPS3808G33, U903 M93C46-WMN6TP, U904 74LVC1G373, U905 TUSB2046BIRHBT

Commit message: fixed footprints, assigned digikey pns
Parts:
- C? (x2): Digi-Key PN 1276-1871-1-ND -> 399-8153-1-ND
- R902: Digi-Key PN (none) -> 541-1.00KHCT-ND
- R? (x5): footprint Resistors_SMD:R_0402 -> Resistors_SMD:R_0603; Digi-Key PN (none) -> 541-10.0KHCT-ND
- R?: footprint Resistors_SMD:R_0402 -> Resistors_SMD:R_0603; Digi-Key PN (none) -> 541-2982-1-ND
- SW901: footprint (none) -> Button_Switch_THT:SW_PUSH_6mm
- U902: Digi-Key PN (none) -> 296-17195-1-ND
- U903: Digi-Key PN (none) -> 497-5090-1-ND
- U904: footprint (none) -> Package_TO_SOT_SMD:SOT-363_SC-70-6; Digi-Key PN (none) -> 296-18775-1-ND
Changed lines of the file:
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@@
       (effects (font (size 1.27 1.27)) (justify right))
     )
-    (property "Digi-Key PN" "1276-1871-1-ND" (at 237.49 22.86 0)
+    (property "Digi-Key PN" "399-8153-1-ND" (at 237.49 22.86 0)
       (effects (font (size 1.27 1.27)) hide)
     )
@@
       (effects (font (size 1.27 1.27)) (justify left))
     )
-    (property "Footprint" "" (at 27.94 124.46 0)
+    (property "Footprint" "Button_Switch_THT:SW_PUSH_6mm" (at 27.94 124.46 0)
       (effects (font (size 1.27 1.27)) hide)
     )
@@
     )
     (property "Datasheet" "https://www.st.com/resource/en/datasheet/m93c46-w.pdf" (at 64.77 173.355 0)
+      (effects (font (size 1.27 1.27)) hide)
+    )
+    (property "Digi-Key PN" "497-5090-1-ND" (at 64.77 174.625 0)
       (effects (font (size 1.27 1.27)) hide)
     )
@@
       (effects (font (size 1.27 1.27)))
     )
-    (property "Footprint" "Resistors_SMD:R_0402" (at 91.44 113.03 0)
+    (property "Footprint" "Resistors_SMD:R_0603" (at 91.44 113.03 0)
       (effects (font (size 1.27 1.27)) hide)
     )
@@
       (effects (font (size 1.27 1.27)) (justify left))
     )
-    (property "Digi-Key PN" "" (at 91.44 113.03 0)
+    (property "Digi-Key PN" "541-10.0KHCT-ND" (at 91.44 113.03 0)
       (effects (font (size 1.27 1.27)) hide)
     )
@@
       (effects (font (size 1.27 1.27)) hide)
     )
-    (property "Digi-Key PN" "" (at 85.09 167.005 0)
+    (property "Digi-Key PN" "541-1.00KHCT-ND" (at 85.09 167.005 0)
       (effects (font (size 1.27 1.27)) hide)
     )
@@
       (effects (font (size 1.27 1.27)))
     )
-    (property "Footprint" "Resistors_SMD:R_0402" (at 80.01 58.42 0)
+    (property "Footprint" "Resistors_SMD:R_0603" (at 80.01 58.42 0)
       (effects (font (size 1.27 1.27)) hide)
     )
@@
       (effects (font (size 1.27 1.27)))
     )
-    (property "Digi-Key PN" "" (at 69.85 50.8 0)
+    (property "Digi-Key PN" "541-2982-1-ND" (at 69.85 50.8 0)
       (effects (font (size 1.524 1.524)) hide)
     )
@@
       (effects (font (size 1.27 1.27)))
     )
-    (property "Footprint" "Resistors_SMD:R_0402" (at 198.12 151.13 0)
+    (property "Footprint" "Resistors_SMD:R_0603" (at 198.12 151.13 0)
       (effects (font (size 1.27 1.27)) hide)
     )
@@
       (effects (font (size 1.27 1.27)) (justify left))
     )
-    (property "Digi-Key PN" "" (at 198.12 151.13 0)
+    (property "Digi-Key PN" "541-10.0KHCT-ND" (at 198.12 151.13 0)
       (effects (font (size 1.27 1.27)) hide)
     )
@@
       (effects (font (size 1.27 1.27)) (justify right))
     )
-    (property "Digi-Key PN" "1276-1871-1-ND" (at 97.79 40.64 0)
+    (property "Digi-Key PN" "399-8153-1-ND" (at 97.79 40.64 0)
       (effects (font (size 1.27 1.27)) hide)
     )
@@
       (effects (font (size 1.27 1.27)))
     )
-    (property "Footprint" "Resistors_SMD:R_0402" (at 165.1 107.95 0)
+    (property "Footprint" "Resistors_SMD:R_0603" (at 165.1 107.95 0)
       (effects (font (size 1.27 1.27)) hide)
     )
@@
       (effects (font (size 1.27 1.27)) (justify left))
     )
-    (property "Digi-Key PN" "" (at 165.1 107.95 0)
+    (property "Digi-Key PN" "541-10.0KHCT-ND" (at 165.1 107.95 0)
       (effects (font (size 1.27 1.27)) hide)
     )
@@
       (effects (font (size 1.27 1.27)))
     )
-    (property "Footprint" "Resistors_SMD:R_0402" (at 91.44 63.5 0)
+    (property "Footprint" "Resistors_SMD:R_0603" (at 91.44 63.5 0)
       (effects (font (size 1.27 1.27)) hide)
     )
@@
       (effects (font (size 1.27 1.27)) (justify left))
     )
-    (property "Digi-Key PN" "" (at 91.44 63.5 0)
+    (property "Digi-Key PN" "541-10.0KHCT-ND" (at 91.44 63.5 0)
       (effects (font (size 1.27 1.27)) hide)
     )
@@
     )
     (property "Datasheet" "http://www.ti.com/lit/ds/symlink/tps3808.pdf" (at 62.23 118.11 0)
+      (effects (font (size 1.27 1.27)) hide)
+    )
+    (property "Digi-Key PN" "296-17195-1-ND" (at 64.77 118.11 0)
       (effects (font (size 1.27 1.27)) hide)
     )
@@
       (effects (font (size 1.27 1.27)))
     )
-    (property "Footprint" "Resistors_SMD:R_0402" (at 91.44 91.44 0)
+    (property "Footprint" "Resistors_SMD:R_0603" (at 91.44 91.44 0)
       (effects (font (size 1.27 1.27)) hide)
     )
@@
       (effects (font (size 1.27 1.27)) (justify left))
     )
-    (property "Digi-Key PN" "" (at 91.44 91.44 0)
+    (property "Digi-Key PN" "541-10.0KHCT-ND" (at 91.44 91.44 0)
       (effects (font (size 1.27 1.27)) hide)
     )
@@
       (effects (font (size 1.27 1.27)))
     )
-    (property "Footprint" "" (at 166.37 151.13 0)
+    (property "Footprint" "Package_TO_SOT_SMD:SOT-363_SC-70-6" (at 166.37 151.13 0)
       (effects (font (size 1.27 1.27)) hide)
     )
@@
       (effects (font (size 1.27 1.27)) hide)
     )
+    (property "Digi-Key PN" "296-18775-1-ND" (at 166.37 151.13 0)
+      (effects (font (size 1.27 1.27)) hide)
+    )
