File: hdw/USB_Hub/Hub_Controller.kicad_sch (KiCad schematic)
At the start: 25 parts, among them SW901 RESET, U902 TPS3808G33, U903 M93C46-WMN6TP, U904 74LVC1G373, U905 TUSB2046BIRHBT

Commit message: fixed some netlist connectivity issues, finished grouping parts in PCB
Parts:
- L?: footprint Inductors_SMD:L_0402 -> Inductors_SMD:L_0603; Digi-Key PN 490-5441-1-ND -> MH1608-601YCT-ND
Changed lines of the file:
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@@
       (effects (font (size 1.27 1.27)))
     )
-    (property "Footprint" "Inductors_SMD:L_0402" (at 52.07 33.782 90)
+    (property "Footprint" "Inductors_SMD:L_0603" (at 52.07 33.782 90)
       (effects (font (size 1.27 1.27)) hide)
     )
@@
       (effects (font (size 1.27 1.27)) hide)
     )
-    (property "Digi-Key PN" "490-5441-1-ND" (at -26.416 -172.466 0)
+    (property "Digi-Key PN" "MH1608-601YCT-ND" (at -26.416 -172.466 0)
       (effects (font (size 1.27 1.27)) hide)
     )
