File: hdw/USB_Hub/PGOOD_LEDs.kicad_sch (KiCad schematic)
At the start: 12 parts

Commit message: schematic progress
Parts:
- removed C? (x3): 0.1uF, Capacitors_SMD:C_0603, symbol Custom_Library:C_Custom
- removed D? (x3): Green, LEDs:LED_0603, symbol Device:LED
- removed R? (x3): 1k, Resistors_SMD:R_0603, symbol Custom_Library:R_Custom
- removed U? (x3): 74LVC1G06, TO_SOT_Packages_SMD:SOT-353_SC-70-5, symbol Custom_Library:74LVC1G06_Power
- added C1501, C1505: 0.1uF, Capacitors_SMD:C_0603, symbol Custom_Library:C_Custom
- added D1501, D1505: Green, LEDs:LED_0603, symbol Device:LED
- added R1501: 10k, Resistors_SMD:R_0603, symbol Custom_Library:R_Custom
- added R1502, R1506: 1k, Resistors_SMD:R_0603, symbol Custom_Library:R_Custom
- added U1501, U1505: 74LVC1G97, Package_TO_SOT_SMD:SOT-363_SC-70-6, symbol Custom_Library:74LVC1G97_Power_NAND_INV
Connections:
- net +3.3V: now also C1501.1, C1505.1, R1502.1, R1506.1, U1501.1 (VCC), U1501.5 (VCC), U1505.1 (VCC), U1505.5 (VCC)
- net GND: now also C1501.2, C1505.2, R1501.2, U1501.2 (GND), U1505.2 (GND)
- net POS12_PGOOD: now also U1501.6
- net POS3P3_PGOOD: now also U1505.6
- new net: D1501.1 (K), U1501.4
- new net: D1501.2 (A), R1502.2
- new net: D1505.1 (K), U1505.4
- new net: D1505.2 (A), R1506.2
- new net PGOOD_LED_SHDN: R1501.1, U1501.3, U1505.3
Other:
- note removed: "SWITCH TO AND GATE WITH ENABLE"

Commit message: lots of schematic progress
Other:
- title: Analog Clock -> USB Hub
Changed lines of the file:
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@@
   (paper "A")
   (title_block
-    (title "Analog Clock")
-    (date "2020-08-15")
-    (rev "A")
+    (title "USB Hub")
+    (date "2023-08-18")
+    (rev "PRELIM")
     (company "Drew Maatman")
   )

Commit message: much more schematic progress
Parts:
- removed R1501: 10k, Resistors_SMD:R_0603, symbol Custom_Library:R_Custom
- added C1505 (x2): 0.1uF, Capacitors_SMD:C_0603, symbol Custom_Library:C_Custom
- added D1505 (x2): Green, LEDs:LED_0603, symbol Device:LED
- added R1506 (x2): 1k, Resistors_SMD:R_0603, symbol Custom_Library:R_Custom
- added U1505 (x2): 74LVC1G97, Package_TO_SOT_SMD:SOT-363_SC-70-6, symbol Custom_Library:74LVC1G97_Power_NAND_INV
Connections:
- net +3.3V: now also C1505.1, C1505.1, R1506.1, R1506.1, U1505.1 (VCC), U1505.1 (VCC), U1505.5 (VCC), U1505.5 (VCC)
- net GND: now also C1505.2, C1505.2, U1505.2 (GND), U1505.2 (GND)
- net PGOOD_LED_SHDN: now also U1505.3, U1505.3
- new net: D1505.1 (K), U1505.4 (x2)
- new net: D1505.2 (A), R1506.2 (x2)
- new net POS5_PGOOD: U1505.6
- new net POS5_USB_PGOOD: U1505.6
Other:
- moved on the sheet: C1501, C1505, D1501, D1505, R1502, R1506, U1501, U1505

Commit message: lots and lots of sch progress
Parts:
- added C?: 0.1uF, Capacitors_SMD:C_0603, symbol Custom_Library:C_Custom
- added D?: Green, LEDs:LED_0603, symbol Device:LED
- added R?: 1k, Resistors_SMD:R_0603, symbol Custom_Library:R_Custom
- added U?: 74LVC1G97, Package_TO_SOT_SMD:SOT-363_SC-70-6, symbol Custom_Library:74LVC1G97_Power_NAND_INV
- renumbered C1505 to C?, C1501 to C?, D1501 to D?, D1505 to D?, R1506 to R?, R1502 to R?, U1505 to U?, U1501 to U?
Connections:
- net +3.3V: now also C?.1, R?.1, U?.1 (VCC), U?.5 (VCC)
- net GND: now also C?.2, U?.2 (GND)
- net PGOOD_LED_SHDN: now also U?.3
- net POS5_PGOOD renamed POS5P_PGOOD
- new net: D?.1 (K), U?.4
- new net: D?.2 (A), R?.2
- new net POS5_SOURCE_STATUS: U?.6

Commit message: pulled footprints into layout
Parts:
- R? (x5): Digi-Key PN 541-1.00KHCT-ND -> (none)
Changed lines of the file:
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@@
       (effects (font (size 1.27 1.27)) (justify left))
     )
-    (property "Digi-Key PN" "541-1.00KHCT-ND" (at 227.965 38.1 0)
+    (property "Digi-Key PN" "" (at 227.965 38.1 0)
       (effects (font (size 1.524 1.524)) hide)
     )
@@
       (effects (font (size 1.27 1.27)) (justify left))
     )
-    (property "Digi-Key PN" "541-1.00KHCT-ND" (at 177.165 38.1 0)
+    (property "Digi-Key PN" "" (at 177.165 38.1 0)
       (effects (font (size 1.524 1.524)) hide)
     )
@@
       (effects (font (size 1.27 1.27)) (justify left))
     )
-    (property "Digi-Key PN" "541-1.00KHCT-ND" (at 75.565 38.1 0)
+    (property "Digi-Key PN" "" (at 75.565 38.1 0)
       (effects (font (size 1.524 1.524)) hide)
     )
@@
       (effects (font (size 1.27 1.27)) (justify left))
     )
-    (property "Digi-Key PN" "541-1.00KHCT-ND" (at 126.365 38.1 0)
+    (property "Digi-Key PN" "" (at 126.365 38.1 0)
       (effects (font (size 1.524 1.524)) hide)
     )
@@
       (effects (font (size 1.27 1.27)) (justify left))
     )
-    (property "Digi-Key PN" "541-1.00KHCT-ND" (at 75.565 76.2 0)
+    (property "Digi-Key PN" "" (at 75.565 76.2 0)
       (effects (font (size 1.524 1.524)) hide)
     )

Commit message: big restructuring, removed microcontroller and all telemtry
Parts:
- removed U? (x5): 74LVC1G97, Package_TO_SOT_SMD:SOT-363_SC-70-6, symbol Custom_Library:74LVC1G97_Power_NAND_INV
- added R?: 10k, Resistors_SMD:R_0402, symbol Custom_Library:R_Custom
- added U601, U602, U603, U604, U605: 74LVC1G97, Package_TO_SOT_SMD:SOT-363_SC-70-6, symbol Custom Library:74LVC1G97_Power_NOT
Connections:
- net +3.3V: now also U604.1 (VCC), U604.5 (VCC); no longer C?.1, C?.1, C?.1, C?.1, R?.1, R?.1, R?.1, R?.1
- net GND: now also U601.2 (GND), U601.3 (GND), U602.2 (GND), U602.3 (GND), U603.2 (GND), U603.3 (GND), U604.2 (GND), U604.3 (GND), U605.2 (GND), U605.3 (GND)
- net POS12_PGOOD: now also U601.6
- net POS3P3_PGOOD: now also U604.6
- net POS5P_PGOOD: now also U603.6
- net POS5_SOURCE_STATUS: now also U602.6
- net at D?.1 (K): now also U601.4
- net at D?.1 (K): now also U604.4
- net at D?.1 (K): now also U602.4
- net at D?.1 (K): now also U603.4
- net at D?.1 (K): now also U605.4
- new net: R?.2, U605.6
- new net +5V: C?.1, C?.1, R?.1, R?.1, U601.1 (VCC), U601.5 (VCC), U602.1 (VCC), U602.5 (VCC)
- new net +5VP: C?.1, R?.1, U603.1 (VCC), U603.5 (VCC)
- new net VBUS: C?.1, R?.1, R?.1, U605.1 (VCC), U605.5 (VCC)
Other:
- moved on the sheet: C?, D?, R?

Commit message: fixed footprints, assigned digikey pns
Parts:
- R? (x5): Digi-Key PN (none) -> 541-1.00KHCT-ND
- R?: footprint Resistors_SMD:R_0402 -> Resistors_SMD:R_0603; Digi-Key PN (none) -> 541-10.0KHCT-ND
- U601, U602, U603, U604, U605: Digi-Key PN (none) -> 1727-1772-1-ND
Changed lines of the file:
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@@
+      (effects (font (size 1.27 1.27)) hide)
+    )
+    (property "Digi-Key PN" "1727-1772-1-ND" (at 120.65 62.23 0)
       (effects (font (size 1.27 1.27)) hide)
     )
@@
       (effects (font (size 1.27 1.27)) (justify left))
     )
-    (property "Digi-Key PN" "" (at 228.6 38.1 0)
+    (property "Digi-Key PN" "541-1.00KHCT-ND" (at 228.6 38.1 0)
       (effects (font (size 1.524 1.524)) hide)
     )
@@
       (effects (font (size 1.27 1.27)) (justify left))
     )
-    (property "Digi-Key PN" "" (at 177.8 38.1 0)
+    (property "Digi-Key PN" "541-1.00KHCT-ND" (at 177.8 38.1 0)
       (effects (font (size 1.524 1.524)) hide)
     )
@@
     )
     (property "Datasheet" "http://www.ti.com/lit/ds/symlink/sn74lvc1g97.pdf" (at 223.52 62.23 0)
+      (effects (font (size 1.27 1.27)) hide)
+    )
+    (property "Digi-Key PN" "1727-1772-1-ND" (at 222.25 62.23 0)
       (effects (font (size 1.27 1.27)) hide)
     )
@@
       (effects (font (size 1.27 1.27)) hide)
     )
+    (property "Digi-Key PN" "1727-1772-1-ND" (at 69.85 62.23 0)
+      (effects (font (size 1.27 1.27)) hide)
+    )
     (pin "1")
     (pin "2")
@@
       (effects (font (size 1.27 1.27)) hide)
     )
+    (property "Digi-Key PN" "1727-1772-1-ND" (at 171.45 62.23 0)
+      (effects (font (size 1.27 1.27)) hide)
+    )
     (pin "1")
     (pin "2")
@@
       (effects (font (size 1.27 1.27)) hide)
     )
+    (property "Digi-Key PN" "1727-1772-1-ND" (at 69.85 100.33 0)
+      (effects (font (size 1.27 1.27)) hide)
+    )
     (pin "1")
     (pin "2")
@@
       (effects (font (size 1.27 1.27)) (justify left))
     )
-    (property "Digi-Key PN" "" (at 76.2 38.1 0)
+    (property "Digi-Key PN" "541-1.00KHCT-ND" (at 76.2 38.1 0)
       (effects (font (size 1.524 1.524)) hide)
     )
@@
       (effects (font (size 1.27 1.27)) (justify left))
     )
-    (property "Digi-Key PN" "" (at 127 38.1 0)
+    (property "Digi-Key PN" "541-1.00KHCT-ND" (at 127 38.1 0)
       (effects (font (size 1.524 1.524)) hide)
     )
@@
       (effects (font (size 1.27 1.27)))
     )
-    (property "Footprint" "Resistors_SMD:R_0402" (at 207.01 55.88 0)
+    (property "Footprint" "Resistors_SMD:R_0603" (at 207.01 55.88 0)
       (effects (font (size 1.27 1.27)) hide)
     )
@@
       (effects (font (size 1.27 1.27)) (justify left))
     )
-    (property "Digi-Key PN" "" (at 207.01 55.88 0)
+    (property "Digi-Key PN" "541-10.0KHCT-ND" (at 207.01 55.88 0)
       (effects (font (size 1.27 1.27)) hide)
     )
@@
       (effects (font (size 1.27 1.27)) (justify left))
     )
-    (property "Digi-Key PN" "" (at 76.2 76.2 0)
+    (property "Digi-Key PN" "541-1.00KHCT-ND" (at 76.2 76.2 0)
       (effects (font (size 1.524 1.524)) hide)
     )
