File: hdw/USB_Hub/POS12_Input.kicad_sch (KiCad schematic)
At the start: 21 parts

Commit message: schematic progress
Parts:
- removed C?: 0.1uF, Capacitors_SMD:C_0603, symbol Custom_Library:C_Custom
- removed C?: 100uF, Capacitors_Tantalum_SMD:CP_Tantalum_Case-X_EIA-7343-43_Reflow, symbol Custom_Library:CP_Tant_Custom
- removed C?: 10nF, Capacitors_SMD:C_0603, symbol Custom_Library:C_Custom
- removed D?: 24V, Diodes_SMD:D_SMA, symbol Device:D_TVS_ALT
- removed J?: +12V IN, Connectors:BARREL_JACK, symbol Connector:Barrel_Jack_Switch
- removed N?: +12V 1A Power Supply, symbol Mechanical:Housing
- removed R?: 1.15k, Resistors_SMD:R_0603, symbol Custom_Library:R_Custom
- removed R?: 51.1k, Resistors_SMD:R_0603, symbol Custom_Library:R_Custom
- removed R? (x2): 5.11k, Resistors_SMD:R_0603, symbol Custom_Library:R_Custom
- removed R? (x2): 10k, Resistors_SMD:R_0603, symbol Custom_Library:R_Custom
- removed R?: 0.02, Resistors_SMD:R_0612, symbol Custom_Library:R_Custom
- removed R? (x2): 10, Resistors_SMD:R_0603, symbol Custom_Library:R_Custom
- removed R?: 13k, Resistors_SMD:R_0603, symbol Custom_Library:R_Custom
- removed R?: R, Resistors_SMD:R_0603, symbol Custom_Library:R_Custom
- removed TP? (x2): TP_Pad, Custom Footprints Library:Test_Point, symbol Custom_Library:TP_Pad
- removed TP?: TP, Pin_Headers:Pin_Header_Angled_1x01_Pitch2.54mm, symbol Custom_Library:TP
- removed U?: TPS26600RHFT, Housings_DFN_QFN:QFN-24-1EP_4x5mm_Pitch0.5mm, symbol Custom_Library:TPS26600RHFT
- added C203: 100uF, Capacitors_Tantalum_SMD:CP_Tantalum_Case-X_EIA-7343-43_Reflow, symbol Custom_Library:CP_Tant_Custom
- added C?: 0.1uF, Capacitors_SMD:C_0402, symbol Custom_Library:C_Custom
- added C?: 10nF, Capacitors_SMD:C_0402, symbol Custom_Library:C_Custom
- added D201: 24V, Diodes_SMD:D_SMA, symbol Device:D_TVS_ALT
- added J201: +12V IN, Connectors:BARREL_JACK, symbol Connector:Barrel_Jack_Switch
- added R? (x2): 100k, Resistors_SMD:R_0402, symbol Custom_Library:R_Custom
- added R? (x9): 10k, Resistors_SMD:R_0402, symbol Custom_Library:R_Custom
- added R? (x3): 0, Resistors_SMD:R_0402, symbol Custom_Library:R_Custom
- added R? (x2): 10, Resistors_SMD:R_0402, symbol Custom_Library:R_Custom
- added R? (x4): 1k, Resistors_SMD:R_0402, symbol Custom_Library:R_Custom
- added R?: 0.02, Resistors_SMD:R_0612, symbol Custom_Library:R_Custom
- added TP201: TP, Pin_Headers:Pin_Header_Angled_1x01_Pitch2.54mm, symbol Custom_Library:TP
- added TP202, TP203: TP, Custom Footprints Library:Test_Point, symbol Custom_Library:TP_Pad
- added U201: TPS26600RHFT, Housings_DFN_QFN:QFN-24-1EP_4x5mm_Pitch0.5mm, symbol Custom_Library:TPS26600RHFT
Connections:
- net +12V: now also C203.1, R?.1, R?.2, R?.2, R?.2, R?.2, R?.2, TP203.1 (TP)
- net +12Vin: now also C?.1, D201.1 (A1), J201.1, R?.1, R?.1, R?.1, TP202.1 (TP), U201.8 (IN), U201.9 (IN)
- net GND: now also C203.2, C?.2, D201.2 (A2), J201.2, J201.3, R?.2, R?.2, TP201.1 (TP), U201.17 (GND)
- net POS12_PGOOD: now also R?.1, R?.1, R?.2, U201.22 (~{FLT})
- net POS12_SNS+: now also R?.1
- net POS12_SNS-: now also R?.1
- new net: R?.1, R?.2, R?.2, U201.10 (UVLO)
- new net: R?.2, U201.14 (~{SHDN})
- new net: R?.1, R?.2 (x3)
- new net: R?.1, R?.1, R?.2, U201.12 (OVP)
- new net: C?.2, R?.2, R?.2, R?.2, R?.2, R?.2, U201.15 (RTN), U201.25 (RTN_PAD)
- new net: R?.1, R?.1, R?.1, R?.1, R?.2, U201.23 (OUT), U201.24 (OUT)
- new net: R?.1, U201.18 (IMON)
- new net: R?.1, R?.1, U201.19 (ILIM)
- new net: C?.1, U201.20 (dVdT)
Other:
- note added: "Switch to fewer components, more BOM line items"
- note added: "UVLO threshold set to 11.12V OVLO threshold set to 13.33V MODE set to Circuit Breaker with Auto-Retry Output Current Limit set to 1.2A Output ramp rate = 12.5V/ms"
- note removed: "UVLO threshold set to 10.8V OVLO threshold set to 13.2V MODE set to Circuit Breaker with Auto-Retry Output Current Limit set to TBD A"

Commit message: lots of schematic progress
Parts:
- removed R? (x2): 100k, Resistors_SMD:R_0402, symbol Custom_Library:R_Custom
- removed R? (x5): 10k, Resistors_SMD:R_0402, symbol Custom_Library:R_Custom
- removed R? (x3): 0, Resistors_SMD:R_0402, symbol Custom_Library:R_Custom
- removed R? (x3): 1k, Resistors_SMD:R_0402, symbol Custom_Library:R_Custom
- added R? (x2): 4.99k, Resistors_SMD:R_0402, symbol Custom_Library:R_Custom
- added R?: 13k, Resistors_SMD:R_0402, symbol Custom_Library:R_Custom
- added R?: 49.9k, Resistors_SMD:R_0402, symbol Custom_Library:R_Custom
- C?: footprint Capacitors_SMD:C_0402 -> Capacitors_SMD:C_0603; Digi-Key PN 490-10698-1-ND -> 1276-1935-1-ND; display_footprint 0402 -> 0603
- C?: footprint Capacitors_SMD:C_0402 -> Capacitors_SMD:C_0603; Digi-Key PN 399-3066-1-ND -> 399-7842-1-ND; display_footprint 0402 -> 0603
- R?: value 1k -> 1.15k; Digi-Key PN RMCF0402FT1K00CT-ND -> (none)
- R?: Configuration Telemetry -> (none)
Connections:
- net +12V: now also R?.1
- net +12Vin: now also R?.1
- net GND: now also R?.2
- net POS12_PGOOD: now also R?.1, R?.2
- net at R?.1, U201.10 (UVLO): now also R?.2
- net at R?.2, U201.12 (OVP): now also R?.1
- net at C?.2, R?.2, R?.2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: now also R?.2
Other:
- note added: "UVLO threshold set to ~10.8V OVLO threshold set to ~13.2V MODE set to Circuit Breaker with Auto-Retry Output Current Limit set to 1.2A Output ramp rate = 12.5V/ms"
- note removed: "UVLO threshold set to 11.12V OVLO threshold set to 13.33V MODE set to Circuit Breaker with Auto-Retry Output Current Limit set to 1.2A Output ramp rate = 12.5V/ms"
- title: Analog Clock -> USB Hub
- moved on the sheet: TP203

Commit message: much more schematic progress
Parts:
- removed C203: 100uF, Capacitors_Tantalum_SMD:CP_Tantalum_Case-X_EIA-7343-43_Reflow, symbol Custom_Library:CP_Tant_Custom
- removed C?: 0.1uF, Capacitors_SMD:C_0603, symbol Custom_Library:C_Custom
- removed C?: 10nF, Capacitors_SMD:C_0603, symbol Custom_Library:C_Custom
- removed R? (x2): 4.99k, Resistors_SMD:R_0402, symbol Custom_Library:R_Custom
- removed R? (x4): 10k, Resistors_SMD:R_0402, symbol Custom_Library:R_Custom
- removed R? (x2): 10, Resistors_SMD:R_0402, symbol Custom_Library:R_Custom
- removed R?: 1.15k, Resistors_SMD:R_0402, symbol Custom_Library:R_Custom
- removed R?: 0.02, Resistors_SMD:R_0612, symbol Custom_Library:R_Custom
- removed R?: 13k, Resistors_SMD:R_0402, symbol Custom_Library:R_Custom
- removed R?: 49.9k, Resistors_SMD:R_0402, symbol Custom_Library:R_Custom
- added C205: 100uF, Capacitors_Tantalum_SMD:CP_Tantalum_Case-X_EIA-7343-43_Reflow, symbol Custom_Library:CP_Tant_Custom
- added C?: 10nF, Capacitors_SMD:C_0603, symbol Custom_Library:C_Custom
- added C?: 0.1uF, Capacitors_SMD:C_0603, symbol Custom_Library:C_Custom
- added N201: +12V 1A Power Supply, symbol Mechanical:Housing
- added R? (x2): 10, Resistors_SMD:R_0603, symbol Custom_Library:R_Custom
- added R? (x3): 10k, Resistors_SMD:R_0603, symbol Custom_Library:R_Custom
- added R?: 1.15k, Resistors_SMD:R_0603, symbol Custom_Library:R_Custom
- added R?: 13k, Resistors_SMD:R_0603, symbol Custom_Library:R_Custom
- added R? (x2): 5.11k, Resistors_SMD:R_0603, symbol Custom_Library:R_Custom
- added R?: 51.1k, Resistors_SMD:R_0603, symbol Custom_Library:R_Custom
- added R?: 0.02, Resistors_SMD:R_0612, symbol Custom_Library:R_Custom
- D201: Configuration DNP -> (none)
- TP202, TP203: value TP -> TP_Pad
Connections:
- net +12V: now also C205.1, R?.1, R?.2, R?.2
- net +12Vin: now also C?.1, R?.1, R?.1
- net GND: now also C205.2, C?.2, R?.2
- net POS12_PGOOD: now also R?.1, R?.2
- net POS12_SNS+: now also R?.1
- net POS12_SNS-: now also R?.1
- net at U201.14 (~{SHDN}): now also R?.2
- net at U201.12 (OVP): now also R?.1, R?.2
- net at U201.15 (RTN), U201.25 (RTN_PAD): now also C?.2, R?.2, R?.2, R?.2
- net at U201.10 (UVLO): now also R?.1, R?.2
- net at U201.18 (IMON): now also R?.1
- net at U201.19 (ILIM): now also R?.1
- net at U201.20 (dVdT): now also C?.1
- net at U201.23 (OUT), U201.24 (OUT): now also R?.1, R?.2
Other:
- note added: "UVLO threshold set to 10.8V OVLO threshold set to 13.2V MODE set to Circuit Breaker with Auto-Retry Output Current Limit set to 1.2A"
- note removed: "Switch to fewer components, more BOM line items"
- note removed: "UVLO threshold set to ~10.8V OVLO threshold set to ~13.2V MODE set to Circuit Breaker with Auto-Retry Output Current Limit set to 1.2A Output ramp rate = 12.5V/ms"

Commit message: lots and lots of sch progress
Parts:
- renumbered C205 to C?, D201 to D?, J201 to J?, N201 to N?, TP203 to TP?, TP202 to TP?, TP201 to TP?, U201 to U?

Commit message: pulled footprints into layout
Parts:
- C?: footprint Capacitors_Tantalum_SMD:CP_Tantalum_Case-X_EIA-7343-43_Reflow -> Capacitor_Tantalum_SMD:CP_EIA-7343-43_Kemet-X
- D?: Configuration (none) -> DNP
- R? (x5): Digi-Key PN YAG2321CT-ND -> (none)
- R?: Digi-Key PN RMCF0603FT1K15CT-ND -> (none)
- R?: Digi-Key PN 311-13.0KHRCT-ND -> (none)
- R? (x2): Digi-Key PN CR0603-FX-5111ELFCT-ND -> (none)
- R?: Digi-Key PN RMCF0603FT51K1TR-ND -> (none)
- TP? (x2): value TP_Pad -> TP
- TP?: footprint Pin_Headers:Pin_Header_Angled_1x01_Pitch2.54mm -> Connector_PinHeader_2.54mm:PinHeader_1x01_P2.54mm_Horizontal
Changed lines of the file:
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@@
       (effects (font (size 1.27 1.27)))
     )
-    (property "Value" "TP_Pad" (at 185.42 44.45 0)
+    (property "Value" "TP" (at 185.42 44.45 0)
       (effects (font (size 1.27 1.27)) hide)
     )
@@
       (effects (font (size 1.27 1.27)) hide)
     )
-    (property "Digi-Key PN" "YAG2321CT-ND" (at 173.355 41.91 0)
+    (property "Digi-Key PN" "" (at 173.355 41.91 0)
       (effects (font (size 1.27 1.27)) hide)
     )
@@
       (effects (font (size 1.27 1.27)) (justify left))
     )
-    (property "Digi-Key PN" "YAG2321CT-ND" (at 111.125 50.8 0)
+    (property "Digi-Key PN" "" (at 111.125 50.8 0)
       (effects (font (size 1.524 1.524)) hide)
     )
@@
       (effects (font (size 1.27 1.27)) (justify left))
     )
-    (property "Digi-Key PN" "RMCF0603FT1K15CT-ND" (at 90.805 72.39 0)
+    (property "Digi-Key PN" "" (at 90.805 72.39 0)
       (effects (font (size 1.524 1.524)) hide)
     )
@@
       (effects (font (size 1.27 1.27)) (justify left))
     )
-    (property "Digi-Key PN" "YAG2321CT-ND" (at 175.895 115.57 0)
+    (property "Digi-Key PN" "" (at 175.895 115.57 0)
       (effects (font (size 1.524 1.524)) hide)
     )
@@
       (effects (font (size 1.27 1.27)) (justify left))
     )
-    (property "Digi-Key PN" "311-13.0KHRCT-ND" (at 170.18 92.71 0)
+    (property "Digi-Key PN" "" (at 170.18 92.71 0)
       (effects (font (size 1.27 1.27)) hide)
     )
@@
       (effects (font (size 1.27 1.27)) (justify left))
     )
-    (property "Digi-Key PN" "CR0603-FX-5111ELFCT-ND" (at 90.805 93.98 0)
+    (property "Digi-Key PN" "" (at 90.805 93.98 0)
       (effects (font (size 1.524 1.524)) hide)
     )
@@
       (effects (font (size 1.27 1.27)) hide)
     )
-    (property "Digi-Key PN" "YAG2321CT-ND" (at 161.29 41.91 0)
+    (property "Digi-Key PN" "" (at 161.29 41.91 0)
       (effects (font (size 1.27 1.27)) hide)
     )
@@
       (effects (font (size 1.27 1.27)) hide)
     )
+    (property "Configuration" "DNP" (at 74.295 59.055 90)
+      (effects (font (size 1.27 1.27)) (justify left))
+    )
     (pin "1")
     (pin "2")
@@
       (effects (font (size 1.27 1.27)) (justify left))
     )
-    (property "Digi-Key PN" "YAG2321CT-ND" (at 196.215 115.57 0)
+    (property "Digi-Key PN" "" (at 196.215 115.57 0)
       (effects (font (size 1.524 1.524)) hide)
     )
@@
       (effects (font (size 1.27 1.27)) (justify left))
     )
-    (property "Digi-Key PN" "RMCF0603FT51K1TR-ND" (at 90.805 50.8 0)
+    (property "Digi-Key PN" "" (at 90.805 50.8 0)
       (effects (font (size 1.524 1.524)) hide)
     )
@@
       (effects (font (size 1.27 1.27)))
     )
-    (property "Value" "TP_Pad" (at 98.425 44.45 0)
+    (property "Value" "TP" (at 98.425 44.45 0)
       (effects (font (size 1.27 1.27)) hide)
     )
@@
       (effects (font (size 1.27 1.27)) (justify left))
     )
-    (property "Footprint" "Capacitors_Tantalum_SMD:CP_Tantalum_Case-X_EIA-7343-43_Reflow" (at 219.4052 59.69 0)
+    (property "Footprint" "Capacitor_Tantalum_SMD:CP_EIA-7343-43_Kemet-X" (at 219.4052 59.69 0)
       (effects (font (size 1.27 1.27)) hide)
     )
@@
       (effects (font (size 1.27 1.27)) (justify left))
     )
-    (property "Digi-Key PN" "CR0603-FX-5111ELFCT-ND" (at 177.8 93.98 0)
+    (property "Digi-Key PN" "" (at 177.8 93.98 0)
       (effects (font (size 1.524 1.524)) hide)
     )
@@
       (effects (font (size 1.27 1.27)) hide)
     )
-    (property "Footprint" "Pin_Headers:Pin_Header_Angled_1x01_Pitch2.54mm" (at 38.1 96.52 0)
+    (property "Footprint" "Connector_PinHeader_2.54mm:PinHeader_1x01_P2.54mm_Horizontal" (at 38.1 96.52 0)
       (effects (font (size 1.524 1.524)) hide)
     )

Commit message: big restructuring, removed microcontroller and all telemtry
Parts:
- removed R? (x2): 10, Resistors_SMD:R_0603, symbol Custom_Library:R_Custom
- removed R?: 0.02, Resistors_SMD:R_0612, symbol Custom_Library:R_Custom
Connections:
- net +12V: now also U?.23 (OUT), U?.24 (OUT)
Other:
- moved on the sheet: C?, J?, R?, TP?, U?

Commit message: fixed footprints, assigned digikey pns
Parts:
- R? (x3): Digi-Key PN (none) -> 541-10.0KHCT-ND
- R?: Digi-Key PN (none) -> 541-1.15KHCT-ND
- R?: Digi-Key PN (none) -> 541-13.0KHCT-ND
- R? (x2): Digi-Key PN (none) -> 541-5.11KHCT-ND
- R?: Digi-Key PN (none) -> 541-3009-1-ND
Changed lines of the file:
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@@
       (effects (font (size 1.27 1.27)) (justify left))
     )
-    (property "Digi-Key PN" "" (at 111.76 50.8 0)
+    (property "Digi-Key PN" "541-10.0KHCT-ND" (at 111.76 50.8 0)
       (effects (font (size 1.524 1.524)) hide)
     )
@@
       (effects (font (size 1.27 1.27)) (justify left))
     )
-    (property "Digi-Key PN" "" (at 91.44 72.39 0)
+    (property "Digi-Key PN" "541-1.15KHCT-ND" (at 91.44 72.39 0)
       (effects (font (size 1.524 1.524)) hide)
     )
@@
       (effects (font (size 1.27 1.27)) (justify left))
     )
-    (property "Digi-Key PN" "" (at 176.53 115.57 0)
+    (property "Digi-Key PN" "541-10.0KHCT-ND" (at 176.53 115.57 0)
       (effects (font (size 1.524 1.524)) hide)
     )
@@
       (effects (font (size 1.27 1.27)) (justify left))
     )
-    (property "Digi-Key PN" "" (at 170.18 92.71 0)
+    (property "Digi-Key PN" "541-13.0KHCT-ND" (at 170.18 92.71 0)
       (effects (font (size 1.27 1.27)) hide)
     )
@@
       (effects (font (size 1.27 1.27)) (justify left))
     )
-    (property "Digi-Key PN" "" (at 91.44 93.98 0)
+    (property "Digi-Key PN" "541-5.11KHCT-ND" (at 91.44 93.98 0)
       (effects (font (size 1.524 1.524)) hide)
     )
@@
       (effects (font (size 1.27 1.27)) (justify left))
     )
-    (property "Digi-Key PN" "" (at 196.85 115.57 0)
+    (property "Digi-Key PN" "541-10.0KHCT-ND" (at 196.85 115.57 0)
       (effects (font (size 1.524 1.524)) hide)
     )
@@
       (effects (font (size 1.27 1.27)) (justify left))
     )
-    (property "Digi-Key PN" "" (at 91.44 50.8 0)
+    (property "Digi-Key PN" "541-3009-1-ND" (at 91.44 50.8 0)
       (effects (font (size 1.524 1.524)) hide)
     )
@@
       (effects (font (size 1.27 1.27)) (justify left))
     )
-    (property "Digi-Key PN" "" (at 177.8 93.98 0)
+    (property "Digi-Key PN" "541-5.11KHCT-ND" (at 177.8 93.98 0)
       (effects (font (size 1.524 1.524)) hide)
     )
