File: hdw/USB_Hub/POS3P3_Power_Supply.kicad_sch (KiCad schematic)
At the start: 23 parts, among them U601 74LVC1G97, U602 TPS62135

Commit message: much more schematic progress
Parts:
- U602: value TPS62135 -> TPS62132
Changed lines of the file:
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@@
       (effects (font (size 1.27 1.27)))
     )
-    (property "Value" "TPS62135" (at 132.715 74.93 0)
+    (property "Value" "TPS62132" (at 132.715 74.93 0)
       (effects (font (size 1.27 1.27)))
     )

Commit message: lots and lots of sch progress
Parts:
- added R?: 10k, Resistors_SMD:R_0402, symbol Custom_Library:R_Custom
- renumbered L601 to L?, U601 to U?, U602 to U?
Connections:
- net +5V: now also R?.1
- net POS3P3_RUN: now also R?.2
Other:
- note added: "DOUBLE CHECK POS3P3_RUN VOLTAGE LEVEL TOLERANCE"

Commit message: pulled footprints into layout
Parts:
- R? (x4): Digi-Key PN RMCF0402FT10K0CT-ND -> (none); Wattage 1/16W -> 1/10W; display_footprint 0402 -> 0603
- R?: Digi-Key PN RMCF0402ZT0R00CT-ND -> (none); Wattage 1/16W -> 1/10W; display_footprint 0402 -> 0603
- R? (x2): Digi-Key PN RMCF0402FT10R0CT-ND -> (none); Wattage 1/16W -> 1/10W; display_footprint 0402 -> 0603
- U?: footprint Package_DFN_QFN:QFN-16-1EP_3x3mm_P0.5mm_EP1.8x1.8mm -> Package_DFN_QFN:QFN-16-1EP_3x3mm_P0.5mm_EP1.75x1.75mm
Changed lines of the file:
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@@
       (effects (font (size 1.27 1.27)) hide)
     )
-    (property "display_footprint" "0402" (at 40.005 93.218 0)
+    (property "display_footprint" "0603" (at 40.005 93.218 0)
       (effects (font (size 1.27 1.27)) (justify left))
     )
@@
       (effects (font (size 1.27 1.27)) (justify left))
     )
-    (property "Wattage" "1/16W" (at 39.751 97.282 0)
-      (effects (font (size 1.27 1.27)) (justify left))
-    )
-    (property "Digi-Key PN" "RMCF0402FT10K0CT-ND" (at 34.925 85.09 0)
+    (property "Wattage" "1/10W" (at 39.751 97.282 0)
+      (effects (font (size 1.27 1.27)) (justify left))
+    )
+    (property "Digi-Key PN" "" (at 34.925 85.09 0)
       (effects (font (size 1.524 1.524)) hide)
     )
@@
       (effects (font (size 1.27 1.27)) hide)
     )
-    (property "display_footprint" "0402" (at 187.325 98.044 0)
+    (property "display_footprint" "0603" (at 187.325 98.044 0)
       (effects (font (size 1.27 1.27)) (justify right))
     )
@@
       (effects (font (size 1.27 1.27)) (justify right))
     )
-    (property "Wattage" "1/16W" (at 187.325 102.87 0)
-      (effects (font (size 1.27 1.27)) (justify right))
-    )
-    (property "Digi-Key PN" "RMCF0402ZT0R00CT-ND" (at 184.785 100.33 0)
+    (property "Wattage" "1/10W" (at 187.325 102.87 0)
+      (effects (font (size 1.27 1.27)) (justify right))
+    )
+    (property "Digi-Key PN" "" (at 184.785 100.33 0)
       (effects (font (size 1.27 1.27)) hide)
     )
@@
       (effects (font (size 1.27 1.27)) hide)
     )
-    (property "display_footprint" "0402" (at 92.075 53.848 0)
+    (property "display_footprint" "0603" (at 92.075 53.848 0)
       (effects (font (size 1.27 1.27)) (justify left))
     )
@@
       (effects (font (size 1.27 1.27)) (justify left))
     )
-    (property "Wattage" "1/16W" (at 92.329 57.912 0)
-      (effects (font (size 1.27 1.27)) (justify left))
-    )
-    (property "Digi-Key PN" "RMCF0402FT10K0CT-ND" (at 97.155 45.72 0)
+    (property "Wattage" "1/10W" (at 92.329 57.912 0)
+      (effects (font (size 1.27 1.27)) (justify left))
+    )
+    (property "Digi-Key PN" "" (at 97.155 45.72 0)
       (effects (font (size 1.524 1.524)) hide)
     )
@@
       (effects (font (size 1.27 1.27)) hide)
     )
-    (property "display_footprint" "0402" (at 191.135 48.26 90)
+    (property "display_footprint" "0603" (at 191.135 48.26 90)
       (effects (font (size 1.27 1.27)) hide)
     )
@@
       (effects (font (size 1.27 1.27)) hide)
     )
-    (property "Wattage" "1/16W" (at 186.055 48.26 90)
-      (effects (font (size 1.27 1.27)) hide)
-    )
-    (property "Digi-Key PN" "RMCF0402FT10R0CT-ND" (at 193.675 48.26 0)
+    (property "Wattage" "1/10W" (at 186.055 48.26 90)
+      (effects (font (size 1.27 1.27)) hide)
+    )
+    (property "Digi-Key PN" "" (at 193.675 48.26 0)
       (effects (font (size 1.27 1.27)) hide)
     )
@@
       (effects (font (size 1.27 1.27)) hide)
     )
-    (property "display_footprint" "0402" (at 69.215 74.168 0)
+    (property "display_footprint" "0603" (at 69.215 74.168 0)
       (effects (font (size 1.27 1.27)) (justify left))
     )
@@
       (effects (font (size 1.27 1.27)) (justify left))
     )
-    (property "Wattage" "1/16W" (at 69.469 78.232 0)
-      (effects (font (size 1.27 1.27)) (justify left))
-    )
-    (property "Digi-Key PN" "RMCF0402FT10K0CT-ND" (at 74.295 66.04 0)
+    (property "Wattage" "1/10W" (at 69.469 78.232 0)
+      (effects (font (size 1.27 1.27)) (justify left))
+    )
+    (property "Digi-Key PN" "" (at 74.295 66.04 0)
       (effects (font (size 1.524 1.524)) hide)
     )
@@
       (effects (font (size 1.27 1.27)) hide)
     )
-    (property "display_footprint" "0402" (at 202.565 48.26 90)
+    (property "display_footprint" "0603" (at 202.565 48.26 90)
       (effects (font (size 1.27 1.27)) hide)
     )
@@
       (effects (font (size 1.27 1.27)) hide)
     )
-    (property "Wattage" "1/16W" (at 197.485 48.26 90)
-      (effects (font (size 1.27 1.27)) hide)
-    )
-    (property "Digi-Key PN" "RMCF0402FT10R0CT-ND" (at 205.105 48.26 0)
+    (property "Wattage" "1/10W" (at 197.485 48.26 90)
+      (effects (font (size 1.27 1.27)) hide)
+    )
+    (property "Digi-Key PN" "" (at 205.105 48.26 0)
       (effects (font (size 1.27 1.27)) hide)
     )
@@
       (effects (font (size 1.27 1.27)))
     )
-    (property "Footprint" "Package_DFN_QFN:QFN-16-1EP_3x3mm_P0.5mm_EP1.8x1.8mm" (at 132.715 74.93 0)
+    (property "Footprint" "Package_DFN_QFN:QFN-16-1EP_3x3mm_P0.5mm_EP1.75x1.75mm" (at 132.715 74.93 0)
       (effects (font (size 1.27 1.27)) hide)
     )
@@
       (effects (font (size 1.27 1.27)) hide)
     )
-    (property "display_footprint" "0402" (at 102.235 151.638 0)
+    (property "display_footprint" "0603" (at 102.235 151.638 0)
       (effects (font (size 1.27 1.27)) (justify left))
     )
@@
       (effects (font (size 1.27 1.27)) (justify left))
     )
-    (property "Wattage" "1/16W" (at 102.489 155.702 0)
-      (effects (font (size 1.27 1.27)) (justify left))
-    )
-    (property "Digi-Key PN" "RMCF0402FT10K0CT-ND" (at 107.315 143.51 0)
+    (property "Wattage" "1/10W" (at 102.489 155.702 0)
+      (effects (font (size 1.27 1.27)) (justify left))
+    )
+    (property "Digi-Key PN" "" (at 107.315 143.51 0)
       (effects (font (size 1.524 1.524)) hide)
     )

Commit message: big restructuring, removed microcontroller and all telemtry
Parts:
- removed C? (x3): 10uF, Capacitors_SMD:C_1206, symbol Custom_Library:C_Custom
- removed C? (x2): 0.1uF, Capacitors_SMD:C_0603, symbol Custom_Library:C_Custom
- removed C?: 10nF, Capacitors_SMD:C_0603, symbol Custom_Library:C_Custom
- removed C?: 10uF, Capacitors_SMD:C_0603, symbol Custom_Library:C_Custom
- removed D?: BAT48JFILM, Diode_SMD:D_SOD-323, symbol Diode:BAT48JFILM
- removed L?: 2.2uH, Inductors_SMD:L_Vishay_IHLP-2020, symbol Custom_Library:L_Custom
- removed Q?: BSS214NW, Package_TO_SOT_SMD:SOT-323_SC-70, symbol Transistor_FET:BSS214NW
- removed Q?: ZXMS6004FFTA, Package_TO_SOT_SMD:SOT-23, symbol Custom_Library:ZXMS6004FFTA
- removed R?: 383k, Resistors_SMD:R_0603, symbol Custom_Library:R_Custom
- removed R? (x4): 10k, Resistors_SMD:R_0402, symbol Custom_Library:R_Custom
- removed R?: 0, Resistors_SMD:R_0402, symbol Custom_Library:R_Custom
- removed R? (x2): 10, Resistors_SMD:R_0402, symbol Custom_Library:R_Custom
- removed R?: 1.21M, Resistors_SMD:R_0603, symbol Custom_Library:R_Custom
- removed R?: 0.02, Resistors_SMD:R_0612, symbol Custom_Library:R_Custom
- removed TP?: TP, Custom Footprints Library:Test_Point, symbol Custom_Library:TP
- removed U?: 74LVC1G97, Package_TO_SOT_SMD:SOT-363_SC-70-6, symbol Custom_Library:74LVC1G97_Power_AND
- removed U?: TPS62132, Package_DFN_QFN:QFN-16-1EP_3x3mm_P0.5mm_EP1.75x1.75mm, symbol Custom_Library:TPS62130
- added C401, C403, C404: 10uF, Capacitors_SMD:C_0402, symbol Custom_Library:C_Custom
- added C402: 0.1uF, Capacitors_SMD:C_0402, symbol Custom_Library:C_Custom
- added R401, R402: 10k, Resistors_SMD:R_0402, symbol Custom_Library:R_Custom
- added R403: 3.57k, Resistors_SMD:R_0402, symbol Custom_Library:R_Custom
- added R404: 1.15k, Resistors_SMD:R_0402, symbol Custom_Library:R_Custom
- added TP401: TP, Custom Footprints Library:Test_Point, symbol Custom_Library:TP
- added U401: TPS7A92, Package_DFN_QFN:Texas_S-PDSO-N10_EP1.2x2mm, symbol Custom_Library:TPS7A91
Connections:
- net +3.3V: now also C403.1, C404.1, R401.1, R403.1, TP401.1 (TP), U401.1 (OUT), U401.2 (OUT)
- net +5V: now also C401.1, R402.1, U401.10 (IN), U401.6 (SS_CTRL), U401.9 (IN)
- net GND: now also C401.2, C402.2, C403.2, C404.2, R404.2, U401.11 (GND), U401.4 (GND)
- new net: R402.2, U401.7 (EN)
- new net: R403.2, R404.1, U401.3 (FB)
- new net: C402.1, U401.8 (NR/SS)
- new net PO3P3_PGOOD: R401.2, U401.5 (PG)
Other:
- note removed: "DOUBLE CHECK POS3P3_RUN VOLTAGE LEVEL TOLERANCE"
- note removed: "Fixed VOUT = +3.3V"

Commit message: fixed footprints, assigned digikey pns
Parts:
- C401, C403, C404: footprint Capacitors_SMD:C_0402 -> Capacitors_SMD:C_0603; Digi-Key PN 490-13211-1-ND -> 399-8153-1-ND; Voltage 6.3V -> 10V; display_footprint 0402 -> 0603
- C402: footprint Capacitors_SMD:C_0402 -> Capacitors_SMD:C_0603; Digi-Key PN 490-10701-1-ND -> 1276-1935-1-ND; display_footprint 0402 -> 0603
- R401, R402: footprint Resistors_SMD:R_0402 -> Resistors_SMD:R_0603; Digi-Key PN RMCF0402FT10K0CT-ND -> 541-10.0KHCT-ND; Wattage 1/16W -> 1/10W; display_footprint 0402 -> 0603
- R403: footprint Resistors_SMD:R_0402 -> Resistors_SMD:R_0603; Digi-Key PN (none) -> 541-3.57KHCT-ND; Wattage 1/16W -> 1/10W; display_footprint 0402 -> 0603
- R404: footprint Resistors_SMD:R_0402 -> Resistors_SMD:R_0603; Digi-Key PN (none) -> 541-1.15KHCT-ND; Wattage 1/16W -> 1/10W; display_footprint 0402 -> 0603
Changed lines of the file:
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@@
       (effects (font (size 1.27 1.27)))
     )
-    (property "Footprint" "Resistors_SMD:R_0402" (at 106.68 73.66 0)
+    (property "Footprint" "Resistors_SMD:R_0603" (at 106.68 73.66 0)
       (effects (font (size 1.27 1.27)) hide)
     )
@@
       (effects (font (size 1.27 1.27)) hide)
     )
-    (property "display_footprint" "0402" (at 109.22 71.628 0)
+    (property "display_footprint" "0603" (at 109.22 71.628 0)
       (effects (font (size 1.27 1.27)) (justify left))
     )
@@
       (effects (font (size 1.27 1.27)) (justify left))
     )
-    (property "Wattage" "1/16W" (at 109.474 75.692 0)
-      (effects (font (size 1.27 1.27)) (justify left))
-    )
-    (property "Digi-Key PN" "RMCF0402FT10K0CT-ND" (at 106.68 73.66 0)
+    (property "Wattage" "1/10W" (at 109.474 75.692 0)
+      (effects (font (size 1.27 1.27)) (justify left))
+    )
+    (property "Digi-Key PN" "541-10.0KHCT-ND" (at 106.68 73.66 0)
       (effects (font (size 1.27 1.27)) hide)
     )
@@
       (effects (font (size 1.016 1.016)))
     )
-    (property "Footprint" "Resistors_SMD:R_0402" (at 189.23 88.9 0)
+    (property "Footprint" "Resistors_SMD:R_0603" (at 189.23 88.9 0)
       (effects (font (size 1.27 1.27)) hide)
     )
@@
       (effects (font (size 1.27 1.27)) hide)
     )
-    (property "display_footprint" "0402" (at 191.77 86.868 0)
+    (property "display_footprint" "0603" (at 191.77 86.868 0)
       (effects (font (size 1.27 1.27)) (justify left))
     )
@@
       (effects (font (size 1.27 1.27)) (justify left))
     )
-    (property "Wattage" "1/16W" (at 192.024 90.932 0)
-      (effects (font (size 1.27 1.27)) (justify left))
-    )
-    (property "Digi-Key PN" "" (at 189.23 88.9 0)
+    (property "Wattage" "1/10W" (at 192.024 90.932 0)
+      (effects (font (size 1.27 1.27)) (justify left))
+    )
+    (property "Digi-Key PN" "541-1.15KHCT-ND" (at 189.23 88.9 0)
       (effects (font (size 1.27 1.27)) hide)
     )
@@
       (effects (font (size 1.27 1.27)) (justify left))
     )
-    (property "Footprint" "Capacitors_SMD:C_0402" (at 116.5352 110.49 0)
+    (property "Footprint" "Capacitors_SMD:C_0603" (at 116.5352 110.49 0)
       (effects (font (size 1.27 1.27)) hide)
     )
@@
       (effects (font (size 1.27 1.27)) hide)
     )
-    (property "display_footprint" "0402" (at 111.76 104.14 0)
+    (property "display_footprint" "0603" (at 111.76 104.14 0)
       (effects (font (size 1.27 1.27)) (justify right))
     )
@@
       (effects (font (size 1.27 1.27)) (justify right))
     )
-    (property "Digi-Key PN" "490-10701-1-ND" (at 126.365 93.98 0)
+    (property "Digi-Key PN" "1276-1935-1-ND" (at 126.365 93.98 0)
       (effects (font (size 1.524 1.524)) hide)
     )
@@
       (effects (font (size 1.27 1.27)) (justify left))
     )
-    (property "Footprint" "Capacitors_SMD:C_0402" (at 168.6052 77.47 0)
+    (property "Footprint" "Capacitors_SMD:C_0603" (at 168.6052 77.47 0)
       (effects (font (size 1.27 1.27)) hide)
     )
@@
       (effects (font (size 1.27 1.27)) hide)
     )
-    (property "display_footprint" "0402" (at 163.83 71.12 0)
-      (effects (font (size 1.27 1.27)) (justify right))
-    )
-    (property "Voltage" "6.3V" (at 163.83 73.66 0)
+    (property "display_footprint" "0603" (at 163.83 71.12 0)
+      (effects (font (size 1.27 1.27)) (justify right))
+    )
+    (property "Voltage" "10V" (at 163.83 73.66 0)
       (effects (font (size 1.27 1.27)) (justify right))
     )
@@
       (effects (font (size 1.27 1.27)) (justify right))
     )
-    (property "Digi-Key PN" "490-13211-1-ND" (at 167.64 73.66 0)
+    (property "Digi-Key PN" "399-8153-1-ND" (at 167.64 73.66 0)
       (effects (font (size 1.27 1.27)) hide)
     )
@@
       (effects (font (size 1.27 1.27)))
     )
-    (property "Footprint" "Resistors_SMD:R_0402" (at 73.66 73.66 0)
+    (property "Footprint" "Resistors_SMD:R_0603" (at 73.66 73.66 0)
       (effects (font (size 1.27 1.27)) hide)
     )
@@
       (effects (font (size 1.27 1.27)) hide)
     )
-    (property "display_footprint" "0402" (at 76.2 71.628 0)
+    (property "display_footprint" "0603" (at 76.2 71.628 0)
       (effects (font (size 1.27 1.27)) (justify left))
     )
@@
       (effects (font (size 1.27 1.27)) (justify left))
     )
-    (property "Wattage" "1/16W" (at 76.454 75.692 0)
-      (effects (font (size 1.27 1.27)) (justify left))
-    )
-    (property "Digi-Key PN" "RMCF0402FT10K0CT-ND" (at 73.66 73.66 0)
+    (property "Wattage" "1/10W" (at 76.454 75.692 0)
+      (effects (font (size 1.27 1.27)) (justify left))
+    )
+    (property "Digi-Key PN" "541-10.0KHCT-ND" (at 73.66 73.66 0)
       (effects (font (size 1.27 1.27)) hide)
     )
@@
       (effects (font (size 1.27 1.27)) (justify left))
     )
-    (property "Footprint" "Capacitors_SMD:C_0402" (at 152.0952 77.47 0)
+    (property "Footprint" "Capacitors_SMD:C_0603" (at 152.0952 77.47 0)
       (effects (font (size 1.27 1.27)) hide)
     )
@@
       (effects (font (size 1.27 1.27)) hide)
     )
-    (property "display_footprint" "0402" (at 147.32 71.12 0)
-      (effects (font (size 1.27 1.27)) (justify right))
-    )
-    (property "Voltage" "6.3V" (at 147.32 73.66 0)
+    (property "display_footprint" "0603" (at 147.32 71.12 0)
+      (effects (font (size 1.27 1.27)) (justify right))
+    )
+    (property "Voltage" "10V" (at 147.32 73.66 0)
       (effects (font (size 1.27 1.27)) (justify right))
     )
@@
       (effects (font (size 1.27 1.27)) (justify right))
     )
-    (property "Digi-Key PN" "490-13211-1-ND" (at 151.13 73.66 0)
+    (property "Digi-Key PN" "399-8153-1-ND" (at 151.13 73.66 0)
       (effects (font (size 1.27 1.27)) hide)
     )
@@
       (effects (font (size 1.016 1.016)))
     )
-    (property "Footprint" "Resistors_SMD:R_0402" (at 189.23 73.66 0)
+    (property "Footprint" "Resistors_SMD:R_0603" (at 189.23 73.66 0)
       (effects (font (size 1.27 1.27)) hide)
     )
@@
       (effects (font (size 1.27 1.27)) hide)
     )
-    (property "display_footprint" "0402" (at 191.77 71.628 0)
+    (property "display_footprint" "0603" (at 191.77 71.628 0)
       (effects (font (size 1.27 1.27)) (justify left))
     )
@@
       (effects (font (size 1.27 1.27)) (justify left))
     )
-    (property "Wattage" "1/16W" (at 192.024 75.692 0)
-      (effects (font (size 1.27 1.27)) (justify left))
-    )
-    (property "Digi-Key PN" "" (at 189.23 73.66 0)
+    (property "Wattage" "1/10W" (at 192.024 75.692 0)
+      (effects (font (size 1.27 1.27)) (justify left))
+    )
+    (property "Digi-Key PN" "541-3.57KHCT-ND" (at 189.23 73.66 0)
       (effects (font (size 1.27 1.27)) hide)
     )
@@
       (effects (font (size 1.27 1.27)) (justify left))
     )
-    (property "Footprint" "Capacitors_SMD:C_0402" (at 94.9452 77.47 0)
+    (property "Footprint" "Capacitors_SMD:C_0603" (at 94.9452 77.47 0)
       (effects (font (size 1.27 1.27)) hide)
     )
@@
       (effects (font (size 1.27 1.27)) hide)
     )
-    (property "display_footprint" "0402" (at 90.17 71.12 0)
-      (effects (font (size 1.27 1.27)) (justify right))
-    )
-    (property "Voltage" "6.3V" (at 90.17 73.66 0)
+    (property "display_footprint" "0603" (at 90.17 71.12 0)
+      (effects (font (size 1.27 1.27)) (justify right))
+    )
+    (property "Voltage" "10V" (at 90.17 73.66 0)
       (effects (font (size 1.27 1.27)) (justify right))
     )
@@
       (effects (font (size 1.27 1.27)) (justify right))
     )
-    (property "Digi-Key PN" "490-13211-1-ND" (at 93.98 73.66 0)
-      (effects (font (size 1.27 1.27)) hide)
-    )
+    (property "Digi-Key PN" "399-8153-1-ND" (at 93.98 73.66 0)
+      (effects (font (size 1.27 1.27)) hide)
+    )

Commit message: pulled in fotprints into layout
Connections:
- net PO3P3_PGOOD renamed POS3P3_PGOOD
Changed lines of the file:
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@@
     (stroke (width 0) (type default))
   )
-  (global_label "PO3P3_PGOOD" (shape output) (at 71.12 82.55 180)
+  (global_label "POS3P3_PGOOD" (shape output) (at 71.12 82.55 180) (fields_autoplaced)
     (effects (font (size 1.27 1.27)) (justify right))
-    (property "Intersheetrefs" "${INTERSHEET_REFS}" (at 71.12 82.55 0)
-      (effects (font (size 1.27 1.27)) hide)
+    (property "Intersheetrefs" "${INTERSHEET_REFS}" (at 53.9308 82.55 0)
+      (effects (font (size 1.27 1.27)) (justify right))
     )
   )
