File: hdw/USB_Hub/USB_Hub.kicad_sch (KiCad schematic)
At the start: 0 parts

Commit message: added new 4 port USB hub controller
Other:
- sheet +5V Power Supply: file POS5_Power_Suply.kicad_sch -> POS5_Power_Supply.kicad_sch
Changed lines of the file:
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@@
       (effects (font (size 1.27 1.27)) (justify left bottom))
     )
-    (property "Sheetfile" "POS5_Power_Suply.kicad_sch" (at 53.34 56.4646 0)
+    (property "Sheetfile" "POS5_Power_Supply.kicad_sch" (at 53.34 56.4646 0)
       (effects (font (size 1.27 1.27)) (justify left top))
     )

Commit message: schematic progress
Other:
- added sheet Power ORing (power_oring.kicad_sch)
Changed lines of the file:
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@@
+    )
+  )
+  (sheet (at 189.23 87.63) (size 12.7 3.81) (fields_autoplaced)
+    (stroke (width 0.1524) (type solid))
+    (fill (color 0 0 0 0.0000))
+    (property "Sheetname" "Power ORing" (at 189.23 86.9184 0)
+      (effects (font (size 1.27 1.27)) (justify left bottom))
+    )
+    (property "Sheetfile" "power_oring.kicad_sch" (at 189.23 92.0246 0)
+      (effects (font (size 1.27 1.27)) (justify left top))
+    )
+    (instances
+      (project "USB_Hub"
+        (path "/e85aac8c-404c-45dd-bda3-1057cae83baf" (page "21"))
+      )
     )
   )

Commit message: lots of schematic progress
Other:
- added sheet +3.3V Power Supply (POS3P3_Power_Supply.kicad_sch)
- added sheet +3.3V Telemetry (POS3P3_Telemetry.kicad_sch)
- added sheet Port Telemetry (Port_Telemetry.kicad_sch)
- company: (none) -> Drew Maatman
- title: (none) -> USB Hub

Commit message: lots and lots of sch progress
Other:
- added sheet Mechanical (mechanical.kicad_sch)
- note added: "01. Table of Contents"
- note added: "02. +12V Input"
- note added: "03. +12V Telemetry"
- note added: "04. +5V Power Supply"
- note added: "05. +5V Telemetry"
- note added: "06. +3.3V Power Supply"
- note added: "07. +3.3V Telemetry"
- note added: "08. Power ORing"
- note added: "09. PIC18F Programming"
- note added: "10. PIC18F Core"
- note added: "11. USB UART Bridge"
- note added: "12. PGOOD LEDs"
- note added: "13. Status LEDs"
- note added: "14. Hub LEDs"
- note added: "15. Display"
- note added: "16. Pushbuttons"
- note added: "17. Hub Controller"
- note added: "18. Downstream Port 0"
- note added: "19. Downstream Port 1"
- note added: "20. Downstream Port 2"
- note added: "21. Downstream Port 3"
- note added: "22. Upstream Port"
- note added: "23. Power Power Control"
- note added: "24. Port Telemetry"
- note added: "25. Mechanical"
- note added: "USB Hub"
- note removed: "Add Mechanical Reorder Sheets"

Commit message: big restructuring, removed microcontroller and all telemtry
Other:
- removed sheet +12V Telemetry
- removed sheet +3.3V Telemetry
- removed sheet +5V Telemetry
- removed sheet Display
- removed sheet PIC18F Core
- removed sheet PIC18F Programming
- removed sheet Port Telemetry
- removed sheet Pushbuttons
- removed sheet Status LEDs
- removed sheet USB UART Bridge
- note added: "03. +5V Power Supply"
- note added: "04. +3.3V Power Supply"
- note added: "05. Power ORing"
- note added: "06. PGOOD LEDs"
- note added: "07. Hub LEDs"
- note added: "08. Mechanical"
- note added: "09. Hub Controller"
- note added: "10. Downstream Port 0"
- note added: "11. Downstream Port 1"
- note added: "12. Downstream Port 2"
- note added: "13. Downstream Port 3"
- note added: "14. Upstream Port"
- note added: "15. Port Power Control"
- note removed: "03. +12V Telemetry"
- note removed: "04. +5V Power Supply"
- note removed: "05. +5V Telemetry"
- note removed: "06. +3.3V Power Supply"
- note removed: "07. +3.3V Telemetry"
- note removed: "08. Power ORing"
- note removed: "09. PIC18F Programming"
- note removed: "10. PIC18F Core"
- note removed: "11. USB UART Bridge"
- note removed: "12. PGOOD LEDs"
- note removed: "13. Status LEDs"
- note removed: "14. Hub LEDs"
- note removed: "15. Display"
- note removed: "16. Pushbuttons"
- note removed: "17. Hub Controller"
- note removed: "18. Downstream Port 0"
- note removed: "19. Downstream Port 1"
- note removed: "20. Downstream Port 2"
- note removed: "21. Downstream Port 3"
- note removed: "22. Upstream Port"
- note removed: "23. Power Power Control"
- note removed: "24. Port Telemetry"
- note removed: "25. Mechanical"

Commit message: pulled in fotprints into layout
Changed lines of the file:
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@@
     (effects (font (size 2.54 2.54) (thickness 0.508) bold) (justify left bottom))
   )
-  (text "08. Mechanical" (at 27.94 97.79 0)
+  (text "08. Mechanical" (at 29.21 97.79 0)
     (effects (font (size 2.54 2.54) (thickness 0.508) bold) (justify left bottom))
   )
