File: hdw/USB_Hub/POS5_Power_Supply.kicad_sch (KiCad schematic)
At the start: 0 parts

Commit message: schematic progress
Parts:
- added C? (x3): 10uF, Capacitors_SMD:C_1206, symbol Custom_Library:C_Custom
- added C? (x2): 0.1uF, Capacitors_SMD:C_0402, symbol Custom_Library:C_Custom
- added C?: 10nF, Capacitors_SMD:C_0402, symbol Custom_Library:C_Custom
- added C?: 10uF, Capacitors_SMD:C_0402, symbol Custom_Library:C_Custom
- added D?: BAT48JFILM, Diode_SMD:D_SOD-323, symbol Diode:BAT48JFILM
- added L601: 2.2uH, Inductors_SMD:L_Vishay_IHLP-2020, symbol Custom_Library:L_Custom
- added Q?: BSS214NW, Package_TO_SOT_SMD:SOT-323_SC-70, symbol Transistor_FET:BSS214NW
- added Q?: ZXMS6004FFTA, Package_TO_SOT_SMD:SOT-23, symbol Custom_Library:ZXMS6004FFTA
- added R?: 180k, Resistors_SMD:R_0402, symbol Custom_Library:R_Custom
- added R?: 953k, Resistors_SMD:R_0402, symbol Custom_Library:R_Custom
- added R? (x2): 10, Resistors_SMD:R_0402, symbol Custom_Library:R_Custom
- added R?: 0.02, Resistors_SMD:R_0612, symbol Custom_Library:R_Custom
- added R? (x3): 10k, Resistors_SMD:R_0402, symbol Custom_Library:R_Custom
- added R?: 0, Resistors_SMD:R_0402, symbol Custom_Library:R_Custom
- added TP?: TP, Custom Footprints Library:Test_Point, symbol Custom_Library:TP
- added U601: 74LVC1G97, Package_TO_SOT_SMD:SOT-363_SC-70-6, symbol Custom_Library:74LVC1G97_Power_AND
- added U602: TPS62133, Package_DFN_QFN:QFN-16-1EP_3x3mm_P0.5mm_EP1.8x1.8mm, symbol Custom_Library:TPS62130
Connections:
- new net: R?.1, R?.1, R?.2, U602.5 (FB)
- new net: C?.1, C?.1, L601.2, R?.1, R?.2
- new net: Q?.1 (G), Q?.3 (D), R?.2
- new net: C?.1, U602.9 (SS/TR)
- new net: L601.1, U602.1 (SW), U602.2 (SW), U602.3 (SW)
- new net: C?.1, D?.1 (K), R?.1
- new net: R?.2, U601.6, U602.4 (PG)
- new net +12V: C?.1, C?.1, U602.10 (AVIN), U602.11 (PVIN), U602.12 (PVIN)
- new net +3.3V: C?.1, D?.2 (A), R?.1, U601.5 (VCC)
- new net +5V: Q?.3 (D), R?.1, R?.2, R?.2, TP?.1 (TP), U602.14 (VOS)
- new net GND: C?.2, C?.2, C?.2, C?.2, C?.2, C?.2, C?.2, Q?.2 (S), Q?.2 (S), R?.2, R?.2, R?.2, U601.1 (GND), U601.2 (GND), U602.15 (PGND), U602.16 (PGND), U602.17 (EP), U602.6 (AGND), U602.7 (FSW), U602.8 (DEF)
- new net POS5_PGOOD: R?.1, U601.4
- new net POS5_RUN: Q?.1 (G), U601.3, U602.13 (EN)
- new net POS5_SNS+: R?.1
- new net POS5_SNS-: R?.1
Other:
- note added: "Fixed VOUT = +5V"

Commit message: lots of schematic progress
Parts:
- removed R? (x2): 10, Resistors_SMD:R_0402, symbol Custom_Library:R_Custom
- removed R?: 0.02, Resistors_SMD:R_0612, symbol Custom_Library:R_Custom
- added R?: 1.37k, Resistors_SMD:R_0603, symbol Custom_Library:R_Custom
- C? (x2): footprint Capacitors_SMD:C_0402 -> Capacitors_SMD:C_0603; Digi-Key PN 490-10698-1-ND -> 1276-1935-1-ND; display_footprint 0402 -> 0603
- C?: footprint Capacitors_SMD:C_0402 -> Capacitors_SMD:C_0603; Digi-Key PN 399-3066-1-ND -> 399-7842-1-ND; display_footprint 0402 -> 0603
- C?: footprint Capacitors_SMD:C_0402 -> Capacitors_SMD:C_0603; Digi-Key PN 1276-1451-1-ND -> 1276-1871-1-ND; Voltage 6.3V -> 10V; display_footprint 0402 -> 0603
- R?: value 10k -> 2.67k; footprint Resistors_SMD:R_0402 -> Resistors_SMD:R_0603; Digi-Key PN RMCF0402FT10K0CT-ND -> (none); Wattage 1/16W -> 1/10W; display_footprint 0402 -> 0603
Connections:
- net +3.3V is gone; now on net +5VP: C?.1, D?.2 (A), R?.1, U601.5 (VCC)
- net +5V is gone; now on net +5VP: Q?.3 (D), R?.1, TP?.1 (TP), U602.14 (VOS)
- net +5VP: now reaches C?.1, C?.1, L601.2
- net POS5_PGOOD: no longer names the net of U601.4
- net POS5_PGOOD: now also R?.2; no longer R?.1
- net POS5_RUN renamed POS5P_RUN
- new net POS5P_PGOOD: R?.1, R?.1
Other:
- company: (none) -> Drew Maatman
- title: (none) -> USB Hub
- moved on the sheet: R?

Commit message: lots and lots of sch progress
Parts:
- added R?: 0, Resistors_SMD:R_0402, symbol Custom_Library:R_Custom
- renumbered L601 to L?, U601 to U?, U602 to U?
Connections:
- net POS5P_RUN: now also R?.2
- new net POS12_PGOOD: R?.1

Commit message: pulled footprints into layout
Parts:
- R?: Digi-Key PN RMCF0402FT180KCT-ND -> (none); Wattage 1/16W -> 1/10W; display_footprint 0402 -> 0603
- R?: Digi-Key PN RMCF0402FT953KCT-ND -> (none); Wattage 1/16W -> 1/10W; display_footprint 0402 -> 0603
- R? (x2): Digi-Key PN RMCF0402ZT0R00CT-ND -> (none); Wattage 1/16W -> 1/10W; display_footprint 0402 -> 0603
- R? (x2): Digi-Key PN RMCF0402FT10K0CT-ND -> (none); Wattage 1/16W -> 1/10W; display_footprint 0402 -> 0603
- U?: footprint Package_DFN_QFN:QFN-16-1EP_3x3mm_P0.5mm_EP1.8x1.8mm -> Package_DFN_QFN:QFN-16-1EP_3x3mm_P0.5mm_EP1.75x1.75mm
Changed lines of the file:
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@@
       (effects (font (size 1.27 1.27)) hide)
     )
-    (property "display_footprint" "0402" (at 219.71 104.648 0)
+    (property "display_footprint" "0603" (at 219.71 104.648 0)
       (effects (font (size 1.27 1.27)) (justify left))
     )
@@
       (effects (font (size 1.27 1.27)) (justify left))
     )
-    (property "Wattage" "1/16W" (at 219.964 108.712 0)
+    (property "Wattage" "1/10W" (at 219.964 108.712 0)
       (effects (font (size 1.27 1.27)) (justify left))
     )
@@
       (effects (font (size 1.27 1.27)))
     )
-    (property "Digi-Key PN" "RMCF0402FT180KCT-ND" (at 217.17 106.68 0)
+    (property "Digi-Key PN" "" (at 217.17 106.68 0)
       (effects (font (size 1.27 1.27)) hide)
     )
@@
       (effects (font (size 1.27 1.27)) hide)
     )
-    (property "display_footprint" "0402" (at 219.71 80.518 0)
+    (property "display_footprint" "0603" (at 219.71 80.518 0)
       (effects (font (size 1.27 1.27)) (justify left))
     )
@@
       (effects (font (size 1.27 1.27)) (justify left))
     )
-    (property "Wattage" "1/16W" (at 219.964 84.582 0)
+    (property "Wattage" "1/10W" (at 219.964 84.582 0)
       (effects (font (size 1.27 1.27)) (justify left))
     )
@@
       (effects (font (size 1.27 1.27)))
     )
-    (property "Digi-Key PN" "RMCF0402FT953KCT-ND" (at 217.17 82.55 0)
+    (property "Digi-Key PN" "" (at 217.17 82.55 0)
       (effects (font (size 1.27 1.27)) hide)
     )
@@
       (effects (font (size 1.27 1.27)) hide)
     )
-    (property "display_footprint" "0402" (at 35.814 170.18 0)
+    (property "display_footprint" "0603" (at 35.814 170.18 0)
       (effects (font (size 1.27 1.27)) (justify right) hide)
     )
@@
       (effects (font (size 1.27 1.27)) (justify right) hide)
     )
-    (property "Wattage" "1/16W" (at 40.64 170.18 0)
+    (property "Wattage" "1/10W" (at 40.64 170.18 0)
       (effects (font (size 1.27 1.27)) (justify right) hide)
     )
-    (property "Digi-Key PN" "RMCF0402ZT0R00CT-ND" (at 38.1 172.72 0)
+    (property "Digi-Key PN" "" (at 38.1 172.72 0)
       (effects (font (size 1.27 1.27)) hide)
     )
@@
       (effects (font (size 1.27 1.27)) hide)
     )
-    (property "display_footprint" "0402" (at 68.58 80.518 0)
+    (property "display_footprint" "0603" (at 68.58 80.518 0)
       (effects (font (size 1.27 1.27)) (justify left))
     )
@@
       (effects (font (size 1.27 1.27)) (justify left))
     )
-    (property "Wattage" "1/16W" (at 68.834 84.582 0)
-      (effects (font (size 1.27 1.27)) (justify left))
-    )
-    (property "Digi-Key PN" "RMCF0402FT10K0CT-ND" (at 73.66 72.39 0)
+    (property "Wattage" "1/10W" (at 68.834 84.582 0)
+      (effects (font (size 1.27 1.27)) (justify left))
+    )
+    (property "Digi-Key PN" "" (at 73.66 72.39 0)
       (effects (font (size 1.524 1.524)) hide)
     )
@@
       (effects (font (size 1.27 1.27)) hide)
     )
-    (property "display_footprint" "0402" (at 101.6 157.988 0)
+    (property "display_footprint" "0603" (at 101.6 157.988 0)
       (effects (font (size 1.27 1.27)) (justify left))
     )
@@
       (effects (font (size 1.27 1.27)) (justify left))
     )
-    (property "Wattage" "1/16W" (at 101.854 162.052 0)
-      (effects (font (size 1.27 1.27)) (justify left))
-    )
-    (property "Digi-Key PN" "RMCF0402FT10K0CT-ND" (at 106.68 149.86 0)
+    (property "Wattage" "1/10W" (at 101.854 162.052 0)
+      (effects (font (size 1.27 1.27)) (justify left))
+    )
+    (property "Digi-Key PN" "" (at 106.68 149.86 0)
       (effects (font (size 1.524 1.524)) hide)
     )
@@
       (effects (font (size 1.27 1.27)) hide)
     )
-    (property "display_footprint" "0402" (at 186.69 104.394 0)
+    (property "display_footprint" "0603" (at 186.69 104.394 0)
       (effects (font (size 1.27 1.27)) (justify right))
     )
@@
       (effects (font (size 1.27 1.27)) (justify right))
     )
-    (property "Wattage" "1/16W" (at 186.69 109.22 0)
-      (effects (font (size 1.27 1.27)) (justify right))
-    )
-    (property "Digi-Key PN" "RMCF0402ZT0R00CT-ND" (at 184.15 106.68 0)
+    (property "Wattage" "1/10W" (at 186.69 109.22 0)
+      (effects (font (size 1.27 1.27)) (justify right))
+    )
+    (property "Digi-Key PN" "" (at 184.15 106.68 0)
       (effects (font (size 1.27 1.27)) hide)
     )
@@
       (effects (font (size 1.27 1.27)))
     )
-    (property "Footprint" "Package_DFN_QFN:QFN-16-1EP_3x3mm_P0.5mm_EP1.8x1.8mm" (at 132.08 81.28 0)
-      (effects (font (size 1.27 1.27)) hide)
-    )
+    (property "Footprint" "Package_DFN_QFN:QFN-16-1EP_3x3mm_P0.5mm_EP1.75x1.75mm" (at 132.08 81.28 0)
+      (effects (font (size 1.27 1.27)) hide)
+    )

Commit message: fixed footprints, assigned digikey pns
Parts:
- C?: Digi-Key PN 1276-1871-1-ND -> 399-8153-1-ND
- R?: footprint Resistors_SMD:R_0402 -> Resistors_SMD:R_0603; Digi-Key PN (none) -> 541-180KHCT-ND
- R?: Digi-Key PN (none) -> 541-1.37KHCT-ND
- R?: footprint Resistors_SMD:R_0402 -> Resistors_SMD:R_0603; Digi-Key PN (none) -> 541-953KHCT-ND
- R? (x2): value 0 -> 10; footprint Resistors_SMD:R_0402 -> Resistors_SMD:R_0603; Digi-Key PN (none) -> 541-2982-1-ND
- R? (x2): footprint Resistors_SMD:R_0402 -> Resistors_SMD:R_0603; Digi-Key PN (none) -> 541-10.0KHCT-ND
- R?: Digi-Key PN (none) -> 541-2.67KHCT-ND
Changed lines of the file:
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@@
       (effects (font (size 1.016 1.016)))
     )
-    (property "Footprint" "Resistors_SMD:R_0402" (at 217.17 106.68 0)
+    (property "Footprint" "Resistors_SMD:R_0603" (at 217.17 106.68 0)
       (effects (font (size 1.27 1.27)) hide)
     )
@@
       (effects (font (size 1.27 1.27)))
     )
-    (property "Digi-Key PN" "" (at 217.17 106.68 0)
+    (property "Digi-Key PN" "541-180KHCT-ND" (at 217.17 106.68 0)
       (effects (font (size 1.27 1.27)) hide)
     )
@@
       (effects (font (size 1.27 1.27)) (justify left) hide)
     )
-    (property "Digi-Key PN" "" (at 33.02 102.87 0)
+    (property "Digi-Key PN" "541-1.37KHCT-ND" (at 33.02 102.87 0)
       (effects (font (size 1.524 1.524)) hide)
     )
@@
       (effects (font (size 1.016 1.016)))
     )
-    (property "Footprint" "Resistors_SMD:R_0402" (at 217.17 82.55 0)
+    (property "Footprint" "Resistors_SMD:R_0603" (at 217.17 82.55 0)
       (effects (font (size 1.27 1.27)) hide)
     )
@@
       (effects (font (size 1.27 1.27)))
     )
-    (property "Digi-Key PN" "" (at 217.17 82.55 0)
+    (property "Digi-Key PN" "541-953KHCT-ND" (at 217.17 82.55 0)
       (effects (font (size 1.27 1.27)) hide)
     )
@@
       (effects (font (size 1.27 1.27)))
     )
-    (property "Value" "0" (at 37.465 172.72 90)
-      (effects (font (size 1.27 1.27)) (justify right))
-    )
-    (property "Footprint" "Resistors_SMD:R_0402" (at 38.1 172.72 0)
+    (property "Value" "10" (at 38.1 172.72 90)
+      (effects (font (size 1.27 1.27)))
+    )
+    (property "Footprint" "Resistors_SMD:R_0603" (at 38.1 172.72 0)
       (effects (font (size 1.27 1.27)) hide)
     )
@@
       (effects (font (size 1.27 1.27)) (justify right) hide)
     )
-    (property "Digi-Key PN" "" (at 38.1 172.72 0)
+    (property "Digi-Key PN" "541-2982-1-ND" (at 38.1 172.72 0)
       (effects (font (size 1.27 1.27)) hide)
     )
@@
       (effects (font (size 1.27 1.27)) (justify right))
     )
-    (property "Digi-Key PN" "1276-1871-1-ND" (at 81.28 160.02 0)
+    (property "Digi-Key PN" "399-8153-1-ND" (at 81.28 160.02 0)
       (effects (font (size 1.27 1.27)) hide)
     )
@@
       (effects (font (size 1.27 1.27)))
     )
-    (property "Footprint" "Resistors_SMD:R_0402" (at 66.04 82.55 0)
+    (property "Footprint" "Resistors_SMD:R_0603" (at 66.04 82.55 0)
       (effects (font (size 1.27 1.27)) hide)
     )
@@
       (effects (font (size 1.27 1.27)) (justify left))
     )
-    (property "Digi-Key PN" "" (at 73.66 72.39 0)
+    (property "Digi-Key PN" "541-10.0KHCT-ND" (at 73.66 72.39 0)
       (effects (font (size 1.524 1.524)) hide)
     )
@@
       (effects (font (size 1.27 1.27)) (justify left))
     )
-    (property "Digi-Key PN" "" (at 27.94 91.44 0)
+    (property "Digi-Key PN" "541-2.67KHCT-ND" (at 27.94 91.44 0)
       (effects (font (size 1.524 1.524)) hide)
     )
@@
       (effects (font (size 1.27 1.27)))
     )
-    (property "Footprint" "Resistors_SMD:R_0402" (at 99.06 160.02 0)
+    (property "Footprint" "Resistors_SMD:R_0603" (at 99.06 160.02 0)
       (effects (font (size 1.27 1.27)) hide)
     )
@@
       (effects (font (size 1.27 1.27)) (justify left))
     )
-    (property "Digi-Key PN" "" (at 106.68 149.86 0)
+    (property "Digi-Key PN" "541-10.0KHCT-ND" (at 106.68 149.86 0)
       (effects (font (size 1.524 1.524)) hide)
     )
@@
       (effects (font (size 1.27 1.27)) (justify left))
     )
-    (property "Value" "0" (at 184.15 106.045 90)
-      (effects (font (size 1.27 1.27)) (justify right))
-    )
-    (property "Footprint" "Resistors_SMD:R_0402" (at 184.15 106.68 0)
+    (property "Value" "10" (at 184.15 106.68 90)
+      (effects (font (size 1.27 1.27)))
+    )
+    (property "Footprint" "Resistors_SMD:R_0603" (at 184.15 106.68 0)
       (effects (font (size 1.27 1.27)) hide)
     )
@@
       (effects (font (size 1.27 1.27)) (justify right))
     )
-    (property "Digi-Key PN" "" (at 184.15 106.68 0)
-      (effects (font (size 1.27 1.27)) hide)
-    )
+    (property "Digi-Key PN" "541-2982-1-ND" (at 184.15 106.68 0)
+      (effects (font (size 1.27 1.27)) hide)
+    )

Commit message: some component placement
Parts:
- added C?: 10uF, Capacitors_SMD:C_1206, symbol Custom_Library:C_Custom
Connections:
- net +12V: now also C?.1
- net GND: now also C?.2
Changed lines of the file:
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@@
   (junction (at 66.04 93.98) (diameter 0) (color 0 0 0 0)
   )
+  (junction (at 85.09 53.34) (diameter 0) (color 0 0 0 0)
+  )
   (junction (at 110.49 53.34) (diameter 0) (color 0 0 0 0)
   )
@@
     (stroke (width 0) (type default))
   )
+  (wire (pts (xy 85.09 53.34) (xy 85.09 58.42))
+    (stroke (width 0) (type default))
+  )
   (wire (pts (xy 144.78 93.98) (xy 184.15 93.98))
     (stroke (width 0) (type default))
@@
     (stroke (width 0) (type default))
   )
+  (wire (pts (xy 85.09 53.34) (xy 110.49 53.34))
+    (stroke (width 0) (type default))
+  )
   (wire (pts (xy 119.38 53.34) (xy 110.49 53.34))
     (stroke (width 0) (type default))
@@
     (stroke (width 0) (type default))
   )
-  (wire (pts (xy 66.04 53.34) (xy 110.49 53.34))
+  (wire (pts (xy 66.04 53.34) (xy 85.09 53.34))
     (stroke (width 0) (type default))
   )
@@
     )
   )
+  (symbol (lib_id "Custom_Library:C_Custom") (at 85.09 62.23 0) (unit 1)
+    (in_bom yes) (on_board yes) (dnp no)
+    (property "Reference" "C?" (at 85.725 59.69 0)
+      (effects (font (size 1.27 1.27)) (justify left))
+    )
+    (property "Value" "10uF" (at 85.725 64.77 0)
+      (effects (font (size 1.27 1.27)) (justify left))
+    )
+    (property "Footprint" "Capacitors_SMD:C_1206" (at 86.0552 66.04 0)
+      (effects (font (size 1.27 1.27)) hide)
+    )
+    (property "Datasheet" "" (at 85.725 59.69 0)
+      (effects (font (size 1.27 1.27)) hide)
+    )
+    (property "display_footprint" "1206" (at 81.28 59.69 0)
+      (effects (font (size 1.27 1.27)) (justify right))
+    )
+    (property "Voltage" "25V" (at 81.28 62.23 0)
+      (effects (font (size 1.27 1.27)) (justify right))
+    )
+    (property "Dielectric" "X5R" (at 81.28 64.77 0)
+      (effects (font (size 1.27 1.27)) (justify right))
+    )
+    (property "Digi-Key PN" "399-8153-1-ND" (at 95.885 49.53 0)
+      (effects (font (size 1.524 1.524)) hide)
+    )
+    (pin "1")
+    (pin "2")
+    (instances
+      (project "LED_Panel_Controller"
+        (path "/9a153a92-537f-48f9-b716-589877e287a5/00000000-0000-0000-0000-00005e0dc082"
+          (reference "C?") (unit 1)
+        )
+        (path "/9a153a92-537f-48f9-b716-589877e287a5/00000000-0000-0000-0000-00005eae2d8a"
+          (reference "C?") (unit 1)
+        )
+        (path "/9a153a92-537f-48f9-b716-589877e287a5/00000000-0000-0000-0000-00005cb7718d"
+          (reference "C?") (unit 1)
+        )
+        (path "/9a153a92-537f-48f9-b716-589877e287a5/00000000-0000-0000-0000-00005f581ba3"
+          (reference "C?") (unit 1)
+        )
+        (path "/9a153a92-537f-48f9-b716-589877e287a5/00000000-0000-0000-0000-00005e0f263a"
+          (reference "C?") (unit 1)
+        )
+      )
+      (project "USB_Hub"
+        (path "/e85aac8c-404c-45dd-bda3-1057cae83baf/00000000-0000-0000-0000-00005f41a7c7"
+          (reference "C308") (unit 1)
+        )
+      )
+    )
+  )
   (symbol (lib_id "power:+5VP") (at 118.11 161.29 0) (unit 1)
     (in_bom yes) (on_board yes) (dnp no)
@@
         )
       )
+    )
+  )
+  (symbol (lib_id "power:GND") (at 85.09 66.04 0) (unit 1)
+    (in_bom yes) (on_board yes) (dnp no)
+    (property "Reference" "#PWR?" (at 85.09 72.39 0)
+      (effects (font (size 1.27 1.27)) hide)
+    )
+    (property "Value" "GND" (at 85.09 69.85 0)
+      (effects (font (size 1.27 1.27)))
+    )
+    (property "Footprint" "" (at 85.09 66.04 0)
+      (effects (font (size 1.27 1.27)) hide)
+    )
+    (property "Datasheet" "" (at 85.09 66.04 0)
+      (effects (font (size 1.27 1.27)) hide)
+    )
+    (pin "1")
+    (instances
+      (project "LED_Panel_Controller"
+        (path "/9a153a92-537f-48f9-b716-589877e287a5/00000000-0000-0000-0000-00005e0dc082"
+          (reference "#PWR?") (unit 1)
+        )
+        (path "/9a153a92-537f-48f9-b716-589877e287a5/00000000-0000-0000-0000-00005eae2d8a"
+          (reference "#PWR?") (unit 1)
+        )
+        (path "/9a153a92-537f-48f9-b716-589877e287a5/00000000-0000-0000-0000-00005cb7718d"
+          (reference "#PWR?") (unit 1)
+        )
+        (path "/9a153a92-537f-48f9-b716-589877e287a5/00000000-0000-0000-0000-00005f581ba3"
+          (reference "#PWR?") (unit 1)
+        )
+        (path "/9a153a92-537f-48f9-b716-589877e287a5/00000000-0000-0000-0000-00005e0f263a"
+          (reference "#PWR?") (unit 1)
+        )
+      )
+      (project "USB_Hub"
+        (path "/e85aac8c-404c-45dd-bda3-1057cae83baf/00000000-0000-0000-0000-00005f41a7c7"
+          (reference "#PWR0325") (unit 1)
+        )
+      )
