File: hdw/USB_Hub/Downstream_Port_0.kicad_sch (KiCad schematic)
At the start: 7 parts

Commit message: lots of schematic progress
Other:
- company: (none) -> Drew Maatman
- title: (none) -> USB Hub
Changed lines of the file:
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@@
 (kicad_sch (version 20230121) (generator eeschema)
   (paper "A")
+  (title_block
+    (title "USB Hub")
+    (date "2023-08-18")
+    (rev "PRELIM")
+    (company "Drew Maatman")
+  )
   (junction (at 106.68 83.82) (diameter 0) (color 0 0 0 0)
   )

Commit message: lots and lots of sch progress
Parts:
- gave numbers to parts that had none: 2
Changed lines of the file:
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@@
   (title_block
     (title "USB Hub")
-    (date "2023-08-18")
+    (date "2023-08-20")
     (rev "PRELIM")
     (company "Drew Maatman")
@@
   )
   (wire (pts (xy 88.9 81.28) (xy 121.92 81.28))
+    (stroke (width 0) (type default))
+  )
+  (wire (pts (xy 185.42 74.93) (xy 185.42 76.2))
     (stroke (width 0) (type default))
   )
@@
   (symbol (lib_id "Connector:USB_A") (at 205.74 81.28 0) (mirror y) (unit 1)
     (in_bom yes) (on_board yes) (dnp no)
-    (property "Reference" "J?" (at 210.82 69.85 0)
+    (property "Reference" "J1801" (at 210.82 69.85 0)
       (effects (font (size 1.27 1.27)) (justify left))
     )
@@
       (project "USB_Hub"
         (path "/e85aac8c-404c-45dd-bda3-1057cae83baf/00000000-0000-0000-0000-00005f41b415"
-          (reference "J?") (unit 1)
+          (reference "J1801") (unit 1)
         )
       )
@@
         )
         (path "/e85aac8c-404c-45dd-bda3-1057cae83baf/00000000-0000-0000-0000-00005f41b415"
-          (reference "C?") (unit 1)
+          (reference "C1802") (unit 1)
         )
       )
@@
         )
         (path "/e85aac8c-404c-45dd-bda3-1057cae83baf/00000000-0000-0000-0000-00005f41b415"
-          (reference "R?") (unit 1)
+          (reference "R1802") (unit 1)
         )
       )
@@
         )
         (path "/e85aac8c-404c-45dd-bda3-1057cae83baf/00000000-0000-0000-0000-00005f41b415"
-          (reference "#PWR01505") (unit 1)
+          (reference "#PWR01801") (unit 1)
         )
       )
@@
         )
         (path "/e85aac8c-404c-45dd-bda3-1057cae83baf/00000000-0000-0000-0000-00005f41b415"
-          (reference "C?") (unit 1)
+          (reference "C1803") (unit 1)
         )
       )
@@
   (symbol (lib_id "Power_Protection:SP0503BAHT") (at 157.48 91.44 0) (unit 1)
     (in_bom yes) (on_board yes) (dnp no)
-    (property "Reference" "D?" (at 163.195 88.9 0)
+    (property "Reference" "D1801" (at 163.195 88.9 0)
       (effects (font (size 1.27 1.27)) (justify left))
     )
@@
       (project "USB_Hub"
         (path "/e85aac8c-404c-45dd-bda3-1057cae83baf/00000000-0000-0000-0000-00005f41b415"
-          (reference "D?") (unit 1)
+          (reference "D1801") (unit 1)
+        )
+      )
+    )
+  )
+  (symbol (lib_id "power:PWR_FLAG") (at 185.42 74.93 0) (unit 1)
+    (in_bom yes) (on_board yes) (dnp no)
+    (property "Reference" "#FLG01801" (at 185.42 73.025 0)
+      (effects (font (size 1.27 1.27)) hide)
+    )
+    (property "Value" "PWR_FLAG" (at 185.42 71.12 0)
+      (effects (font (size 1.27 1.27)))
+    )
+    (property "Footprint" "" (at 185.42 74.93 0)
+      (effects (font (size 1.27 1.27)) hide)
+    )
+    (property "Datasheet" "~" (at 185.42 74.93 0)
+      (effects (font (size 1.27 1.27)) hide)
+    )
+    (pin "1")
+    (instances
+      (project "USB_Hub"
+        (path "/e85aac8c-404c-45dd-bda3-1057cae83baf/00000000-0000-0000-0000-00005f41b415"
+          (reference "#FLG01801") (unit 1)
         )
       )
@@
         )
         (path "/e85aac8c-404c-45dd-bda3-1057cae83baf/00000000-0000-0000-0000-00005f41b415"
-          (reference "#PWR01503") (unit 1)
+          (reference "#PWR01803") (unit 1)
         )
       )
@@
         )
         (path "/e85aac8c-404c-45dd-bda3-1057cae83baf/00000000-0000-0000-0000-00005f41b415"
-          (reference "#PWR01501") (unit 1)
+          (reference "#PWR01804") (unit 1)
         )
       )
@@
   (symbol (lib_id "Custom Library:CHASSIS") (at 210.82 96.52 0) (unit 1)
     (in_bom yes) (on_board yes) (dnp no)
-    (property "Reference" "#PWR01506" (at 210.82 101.6 0)
+    (property "Reference" "#PWR01806" (at 210.82 101.6 0)
       (effects (font (size 1.27 1.27)) hide)
     )
@@
       (project "USB_Hub"
         (path "/e85aac8c-404c-45dd-bda3-1057cae83baf/00000000-0000-0000-0000-00005f41b415"
-          (reference "#PWR01506") (unit 1)
+          (reference "#PWR01806") (unit 1)
         )
       )
@@
         )
         (path "/e85aac8c-404c-45dd-bda3-1057cae83baf/00000000-0000-0000-0000-00005f41b415"
-          (reference "#PWR01502") (unit 1)
+          (reference "#PWR01805") (unit 1)
         )
       )
@@
         )
         (path "/e85aac8c-404c-45dd-bda3-1057cae83baf/00000000-0000-0000-0000-00005f41b415"
-          (reference "#PWR01504") (unit 1)
+          (reference "#PWR01802") (unit 1)
         )
       )
@@
         )
         (path "/e85aac8c-404c-45dd-bda3-1057cae83baf/00000000-0000-0000-0000-00005f41b415"
-          (reference "C?") (unit 1)
+          (reference "C1801") (unit 1)
         )
       )
@@
         )
         (path "/e85aac8c-404c-45dd-bda3-1057cae83baf/00000000-0000-0000-0000-00005f41b415"
-          (reference "R?") (unit 1)
-        )
-      )
+          (reference "R1801") (unit 1)
+        )
+      )

Commit message: pulled footprints into layout
Parts:
- C?: footprint Capacitors_Tantalum_SMD:CP_Tantalum_Case-X_EIA-7343-43_Reflow -> Capacitor_Tantalum_SMD:CP_EIA-7343-43_Kemet-X
- J1801: footprint (none) -> Connector_USB:USB_A_Molex_67643_Horizontal
- R? (x2): Digi-Key PN 311-27.0HRCT-ND -> (none)
Changed lines of the file:
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@@
       (effects (font (size 1.27 1.27)) (justify left))
     )
-    (property "Footprint" "" (at 201.93 82.55 0)
+    (property "Footprint" "Connector_USB:USB_A_Molex_67643_Horizontal" (at 201.93 82.55 0)
       (effects (font (size 1.27 1.27)) hide)
     )
@@
       (effects (font (size 1.27 1.27)) hide)
     )
-    (property "Digi-Key PN" "311-27.0HRCT-ND" (at 135.89 91.44 0)
+    (property "Digi-Key PN" "" (at 135.89 91.44 0)
       (effects (font (size 1.524 1.524)) hide)
     )
@@
       (effects (font (size 1.27 1.27)) (justify left))
     )
-    (property "Footprint" "Capacitors_Tantalum_SMD:CP_Tantalum_Case-X_EIA-7343-43_Reflow" (at 186.3852 96.52 0)
+    (property "Footprint" "Capacitor_Tantalum_SMD:CP_EIA-7343-43_Kemet-X" (at 186.3852 96.52 0)
       (effects (font (size 1.27 1.27)) hide)
     )
@@
       (effects (font (size 1.27 1.27)) hide)
     )
-    (property "Digi-Key PN" "311-27.0HRCT-ND" (at 135.89 73.66 0)
+    (property "Digi-Key PN" "" (at 135.89 73.66 0)
       (effects (font (size 1.524 1.524)) hide)
     )

Commit message: big restructuring, removed microcontroller and all telemtry
Parts:
- gave numbers to parts that had none: 4
- renumbered D1801 to D1001, J1801 to J1001
Changed lines of the file:
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@@
   (symbol (lib_id "Connector:USB_A") (at 205.74 81.28 0) (mirror y) (unit 1)
     (in_bom yes) (on_board yes) (dnp no)
-    (property "Reference" "J1801" (at 210.82 69.85 0)
+    (property "Reference" "J1001" (at 210.82 69.85 0)
       (effects (font (size 1.27 1.27)) (justify left))
     )
@@
       (project "USB_Hub"
         (path "/e85aac8c-404c-45dd-bda3-1057cae83baf/00000000-0000-0000-0000-00005f41b415"
-          (reference "J1801") (unit 1)
+          (reference "J1001") (unit 1)
         )
       )
@@
     (instances
       (project "USB_Hub"
-        (path "/e85aac8c-404c-45dd-bda3-1057cae83baf/00000000-0000-0000-0000-00005f41a830"
-          (reference "C?") (unit 1)
-        )
-        (path "/e85aac8c-404c-45dd-bda3-1057cae83baf/00000000-0000-0000-0000-00005f41b415"
-          (reference "C1802") (unit 1)
+        (path "/e85aac8c-404c-45dd-bda3-1057cae83baf/00000000-0000-0000-0000-00005f41b415"
+          (reference "C1002") (unit 1)
         )
       )
@@
     (instances
       (project "USB_Hub"
-        (path "/e85aac8c-404c-45dd-bda3-1057cae83baf/00000000-0000-0000-0000-00005f41a830"
-          (reference "R?") (unit 1)
-        )
-        (path "/e85aac8c-404c-45dd-bda3-1057cae83baf/00000000-0000-0000-0000-00005f41b415"
-          (reference "R1802") (unit 1)
+        (path "/e85aac8c-404c-45dd-bda3-1057cae83baf/00000000-0000-0000-0000-00005f41b415"
+          (reference "R1002") (unit 1)
         )
       )
@@
     (instances
       (project "USB_Hub"
-        (path "/e85aac8c-404c-45dd-bda3-1057cae83baf/00000000-0000-0000-0000-00005f41a830"
-          (reference "#PWR?") (unit 1)
-        )
-        (path "/e85aac8c-404c-45dd-bda3-1057cae83baf/00000000-0000-0000-0000-00005f41b415"
-          (reference "#PWR01801") (unit 1)
+        (path "/e85aac8c-404c-45dd-bda3-1057cae83baf/00000000-0000-0000-0000-00005f41b415"
+          (reference "#PWR01001") (unit 1)
         )
       )
@@
         )
         (path "/e85aac8c-404c-45dd-bda3-1057cae83baf/00000000-0000-0000-0000-00005f41b415"
-          (reference "C1803") (unit 1)
+          (reference "C1003") (unit 1)
         )
       )
@@
   (symbol (lib_id "Power_Protection:SP0503BAHT") (at 157.48 91.44 0) (unit 1)
     (in_bom yes) (on_board yes) (dnp no)
-    (property "Reference" "D1801" (at 163.195 88.9 0)
+    (property "Reference" "D1001" (at 163.195 88.9 0)
       (effects (font (size 1.27 1.27)) (justify left))
     )
@@
       (project "USB_Hub"
         (path "/e85aac8c-404c-45dd-bda3-1057cae83baf/00000000-0000-0000-0000-00005f41b415"
-          (reference "D1801") (unit 1)
+          (reference "D1001") (unit 1)
         )
       )
@@
   (symbol (lib_id "power:PWR_FLAG") (at 185.42 74.93 0) (unit 1)
     (in_bom yes) (on_board yes) (dnp no)
-    (property "Reference" "#FLG01801" (at 185.42 73.025 0)
+    (property "Reference" "#FLG01001" (at 185.42 73.025 0)
       (effects (font (size 1.27 1.27)) hide)
     )
@@
       (project "USB_Hub"
         (path "/e85aac8c-404c-45dd-bda3-1057cae83baf/00000000-0000-0000-0000-00005f41b415"
-          (reference "#FLG01801") (unit 1)
+          (reference "#FLG01001") (unit 1)
         )
       )
@@
         )
         (path "/e85aac8c-404c-45dd-bda3-1057cae83baf/00000000-0000-0000-0000-00005f41b415"
-          (reference "#PWR01803") (unit 1)
+          (reference "#PWR01003") (unit 1)
         )
       )
@@
         )
         (path "/e85aac8c-404c-45dd-bda3-1057cae83baf/00000000-0000-0000-0000-00005f41b415"
-          (reference "#PWR01804") (unit 1)
+          (reference "#PWR01004") (unit 1)
         )
       )
@@
   (symbol (lib_id "Custom Library:CHASSIS") (at 210.82 96.52 0) (unit 1)
     (in_bom yes) (on_board yes) (dnp no)
-    (property "Reference" "#PWR01806" (at 210.82 101.6 0)
+    (property "Reference" "#PWR01006" (at 210.82 101.6 0)
       (effects (font (size 1.27 1.27)) hide)
     )
@@
       (project "USB_Hub"
         (path "/e85aac8c-404c-45dd-bda3-1057cae83baf/00000000-0000-0000-0000-00005f41b415"
-          (reference "#PWR01806") (unit 1)
+          (reference "#PWR01006") (unit 1)
         )
       )
@@
         )
         (path "/e85aac8c-404c-45dd-bda3-1057cae83baf/00000000-0000-0000-0000-00005f41b415"
-          (reference "#PWR01805") (unit 1)
+          (reference "#PWR01005") (unit 1)
         )
       )
@@
     (instances
       (project "USB_Hub"
-        (path "/e85aac8c-404c-45dd-bda3-1057cae83baf/00000000-0000-0000-0000-00005f41a830"
-          (reference "#PWR?") (unit 1)
-        )
-        (path "/e85aac8c-404c-45dd-bda3-1057cae83baf/00000000-0000-0000-0000-00005f41b415"
-          (reference "#PWR01802") (unit 1)
+        (path "/e85aac8c-404c-45dd-bda3-1057cae83baf/00000000-0000-0000-0000-00005f41b415"
+          (reference "#PWR01002") (unit 1)
         )
       )
@@
     (instances
       (project "USB_Hub"
-        (path "/e85aac8c-404c-45dd-bda3-1057cae83baf/00000000-0000-0000-0000-00005f41a830"
-          (reference "C?") (unit 1)
-        )
-        (path "/e85aac8c-404c-45dd-bda3-1057cae83baf/00000000-0000-0000-0000-00005f41b415"
-          (reference "C1801") (unit 1)
+        (path "/e85aac8c-404c-45dd-bda3-1057cae83baf/00000000-0000-0000-0000-00005f41b415"
+          (reference "C1001") (unit 1)
         )
       )
@@
     (instances
       (project "USB_Hub"
-        (path "/e85aac8c-404c-45dd-bda3-1057cae83baf/00000000-0000-0000-0000-00005f41a830"
-          (reference "R?") (unit 1)
-        )
-        (path "/e85aac8c-404c-45dd-bda3-1057cae83baf/00000000-0000-0000-0000-00005f41b415"
-          (reference "R1801") (unit 1)
-        )
-      )
+        (path "/e85aac8c-404c-45dd-bda3-1057cae83baf/00000000-0000-0000-0000-00005f41b415"
+          (reference "R1001") (unit 1)
+        )
+      )

Commit message: fixed footprints, assigned digikey pns
Parts:
- C1001, C1002: Digi-Key PN (none) -> 1292-1501-1-ND
- D1001: Digi-Key PN (none) -> F2715CT-ND
- J1001: footprint Connector_USB:USB_A_Molex_67643_Horizontal -> Connector_USB:USB_A_Wuerth_614004134726_Horizontal; Digi-Key PN (none) -> 732-2731-ND
- R1001, R1002: Digi-Key PN (none) -> 541-27.0HCT-ND
Changed lines of the file:
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@@
-    (stroke (width 0) (type default))
-  )
-  (wire (pts (xy 185.42 74.93) (xy 185.42 76.2))
     (stroke (width 0) (type default))
   )
@@
       (effects (font (size 1.27 1.27)) (justify left))
     )
-    (property "Footprint" "Connector_USB:USB_A_Molex_67643_Horizontal" (at 201.93 82.55 0)
+    (property "Footprint" "Connector_USB:USB_A_Wuerth_614004134726_Horizontal" (at 201.93 82.55 0)
       (effects (font (size 1.27 1.27)) hide)
     )
     (property "Datasheet" " ~" (at 201.93 82.55 0)
+      (effects (font (size 1.27 1.27)) hide)
+    )
+    (property "Digi-Key PN" "732-2731-ND" (at 205.74 81.28 0)
       (effects (font (size 1.27 1.27)) hide)
     )
@@
       (effects (font (size 1.27 1.27)) (justify right))
     )
-    (property "Digi-Key PN" "" (at 106.68 92.71 0)
+    (property "Digi-Key PN" "1292-1501-1-ND" (at 106.68 92.71 0)
       (effects (font (size 1.27 1.27)) hide)
     )
@@
       (effects (font (size 1.27 1.27)) hide)
     )
-    (property "Digi-Key PN" "" (at 135.89 91.44 0)
+    (property "Digi-Key PN" "541-27.0HCT-ND" (at 135.89 91.44 0)
       (effects (font (size 1.524 1.524)) hide)
     )
@@
       (effects (font (size 1.27 1.27)) hide)
     )
+    (property "Digi-Key PN" "F2715CT-ND" (at 157.48 91.44 0)
+      (effects (font (size 1.27 1.27)) hide)
+    )
     (pin "1")
     (pin "2")
@@
     )
   )
-  (symbol (lib_id "power:PWR_FLAG") (at 185.42 74.93 0) (unit 1)
-    (in_bom yes) (on_board yes) (dnp no)
-    (property "Reference" "#FLG01001" (at 185.42 73.025 0)
-      (effects (font (size 1.27 1.27)) hide)
-    )
-    (property "Value" "PWR_FLAG" (at 185.42 71.12 0)
-      (effects (font (size 1.27 1.27)))
-    )
-    (property "Footprint" "" (at 185.42 74.93 0)
-      (effects (font (size 1.27 1.27)) hide)
-    )
-    (property "Datasheet" "~" (at 185.42 74.93 0)
-      (effects (font (size 1.27 1.27)) hide)
-    )
-    (pin "1")
-    (instances
-      (project "USB_Hub"
-        (path "/e85aac8c-404c-45dd-bda3-1057cae83baf/00000000-0000-0000-0000-00005f41b415"
-          (reference "#FLG01001") (unit 1)
-        )
-      )
-    )
-  )
   (symbol (lib_id "power:GND") (at 157.48 96.52 0) (unit 1)
     (in_bom yes) (on_board yes) (dnp no)
@@
       (effects (font (size 1.27 1.27)) (justify right))
     )
-    (property "Digi-Key PN" "" (at 88.9 92.71 0)
+    (property "Digi-Key PN" "1292-1501-1-ND" (at 88.9 92.71 0)
       (effects (font (size 1.27 1.27)) hide)
     )
@@
       (effects (font (size 1.27 1.27)) hide)
     )
-    (property "Digi-Key PN" "" (at 135.89 73.66 0)
+    (property "Digi-Key PN" "541-27.0HCT-ND" (at 135.89 73.66 0)
       (effects (font (size 1.524 1.524)) hide)
     )

Commit message: fixed some netlist connectivity issues, finished grouping parts in PCB
Connections:
- net DFP0_USB_CONN_D+: now also D1001.4 (K); no longer D1001.3 (K)
- net DFP0_USB_CONN_D-: now also D1001.3 (K); no longer D1001.4 (K)
Changed lines of the file:
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@@
     (company "Drew Maatman")
+  )
+  (junction (at 160.02 81.28) (diameter 0) (color 0 0 0 0)
   )
   (junction (at 106.68 83.82) (diameter 0) (color 0 0 0 0)
@@
   (junction (at 185.42 76.2) (diameter 0) (color 0 0 0 0)
   )
-  (junction (at 160.02 83.82) (diameter 0) (color 0 0 0 0)
-  )
   (junction (at 154.94 76.2) (diameter 0) (color 0 0 0 0)
   )
-  (junction (at 157.48 81.28) (diameter 0) (color 0 0 0 0)
+  (junction (at 157.48 83.82) (diameter 0) (color 0 0 0 0)
   )
-  (wire (pts (xy 129.54 83.82) (xy 160.02 83.82))
+  (wire (pts (xy 129.54 83.82) (xy 157.48 83.82))
+    (stroke (width 0) (type default))
+  )
+  (wire (pts (xy 160.02 81.28) (xy 160.02 86.36))
     (stroke (width 0) (type default))
   )
@@
     (stroke (width 0) (type default))
   )
-  (wire (pts (xy 210.82 96.52) (xy 210.82 95.25))
+  (wire (pts (xy 157.48 83.82) (xy 157.48 86.36))
     (stroke (width 0) (type default))
   )
-  (wire (pts (xy 157.48 81.28) (xy 157.48 86.36))
+  (wire (pts (xy 210.82 96.52) (xy 210.82 95.25))
     (stroke (width 0) (type default))
   )
@@
     (stroke (width 0) (type default))
   )
+  (wire (pts (xy 157.48 83.82) (xy 198.12 83.82))
+    (stroke (width 0) (type default))
+  )
   (wire (pts (xy 76.2 81.28) (xy 88.9 81.28))
     (stroke (width 0) (type default))
   )
   (wire (pts (xy 205.74 95.25) (xy 205.74 91.44))
+    (stroke (width 0) (type default))
+  )
+  (wire (pts (xy 160.02 81.28) (xy 198.12 81.28))
     (stroke (width 0) (type default))
   )
@@
     (stroke (width 0) (type default))
   )
-  (wire (pts (xy 160.02 83.82) (xy 198.12 83.82))
-    (stroke (width 0) (type default))
-  )
   (wire (pts (xy 76.2 83.82) (xy 106.68 83.82))
     (stroke (width 0) (type default))
@@
     (stroke (width 0) (type default))
   )
-  (wire (pts (xy 160.02 83.82) (xy 160.02 86.36))
-    (stroke (width 0) (type default))
-  )
   (wire (pts (xy 154.94 86.36) (xy 154.94 76.2))
     (stroke (width 0) (type default))
   )
-  (wire (pts (xy 157.48 81.28) (xy 198.12 81.28))
-    (stroke (width 0) (type default))
-  )
-  (wire (pts (xy 129.54 81.28) (xy 157.48 81.28))
+  (wire (pts (xy 129.54 81.28) (xy 160.02 81.28))
     (stroke (width 0) (type default))
   )
@@
     (effects (font (size 1.27 1.27)) (justify right))
     (property "Intersheetrefs" "${INTERSHEET_REFS}" (at 59.5702 83.82 0)
-      (effects (font (size 1.27 1.27)) (justify right) hide)
+      (effects (font (size 1.27 1.27)) (justify right))
     )
   )
@@
     (effects (font (size 1.27 1.27)) (justify right))
     (property "Intersheetrefs" "${INTERSHEET_REFS}" (at 59.5702 81.28 0)
-      (effects (font (size 1.27 1.27)) (justify right) hide)
+      (effects (font (size 1.27 1.27)) (justify right))
     )
   )
@@
     (effects (font (size 1.27 1.27)) (justify right))
     (property "Intersheetrefs" "${INTERSHEET_REFS}" (at 63.2441 76.2 0)
-      (effects (font (size 1.27 1.27)) (justify right) hide)
+      (effects (font (size 1.27 1.27)) (justify right))
     )
   )
