File: hdw/USB_Hub/Downstream_Port_3.kicad_sch (KiCad schematic)
At the start: 7 parts

Commit message: lots of schematic progress
Other:
- company: (none) -> Drew Maatman
- title: (none) -> USB Hub
Changed lines of the file:
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@@
 (kicad_sch (version 20230121) (generator eeschema)
   (paper "A")
+  (title_block
+    (title "USB Hub")
+    (date "2023-08-18")
+    (rev "PRELIM")
+    (company "Drew Maatman")
+  )
   (junction (at 157.48 81.28) (diameter 0) (color 0 0 0 0)
   )

Commit message: lots and lots of sch progress
Changed lines of the file:
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@@
   (title_block
     (title "USB Hub")
-    (date "2023-08-18")
+    (date "2023-08-20")
     (rev "PRELIM")
     (company "Drew Maatman")
@@
   )
   (wire (pts (xy 76.2 81.28) (xy 88.9 81.28))
+    (stroke (width 0) (type default))
+  )
+  (wire (pts (xy 185.42 74.93) (xy 185.42 76.2))
     (stroke (width 0) (type default))
   )
@@
         )
         (path "/e85aac8c-404c-45dd-bda3-1057cae83baf/00000000-0000-0000-0000-00005f41b451"
-          (reference "C?") (unit 1)
+          (reference "C2103") (unit 1)
+        )
+      )
+    )
+  )
+  (symbol (lib_id "power:PWR_FLAG") (at 185.42 74.93 0) (unit 1)
+    (in_bom yes) (on_board yes) (dnp no)
+    (property "Reference" "#FLG?" (at 185.42 73.025 0)
+      (effects (font (size 1.27 1.27)) hide)
+    )
+    (property "Value" "PWR_FLAG" (at 185.42 71.12 0)
+      (effects (font (size 1.27 1.27)))
+    )
+    (property "Footprint" "" (at 185.42 74.93 0)
+      (effects (font (size 1.27 1.27)) hide)
+    )
+    (property "Datasheet" "~" (at 185.42 74.93 0)
+      (effects (font (size 1.27 1.27)) hide)
+    )
+    (pin "1")
+    (instances
+      (project "USB_Hub"
+        (path "/e85aac8c-404c-45dd-bda3-1057cae83baf/00000000-0000-0000-0000-00005f41b415"
+          (reference "#FLG?") (unit 1)
+        )
+        (path "/e85aac8c-404c-45dd-bda3-1057cae83baf/00000000-0000-0000-0000-00005f41b451"
+          (reference "#FLG02101") (unit 1)
         )
       )
@@
         )
         (path "/e85aac8c-404c-45dd-bda3-1057cae83baf/00000000-0000-0000-0000-00005f41b415"
-          (reference "#PWR01502") (unit 1)
-        )
-        (path "/e85aac8c-404c-45dd-bda3-1057cae83baf/00000000-0000-0000-0000-00005f41b451"
-          (reference "#PWR01805") (unit 1)
+          (reference "#PWR?") (unit 1)
+        )
+        (path "/e85aac8c-404c-45dd-bda3-1057cae83baf/00000000-0000-0000-0000-00005f41b451"
+          (reference "#PWR02105") (unit 1)
         )
       )
@@
         )
         (path "/e85aac8c-404c-45dd-bda3-1057cae83baf/00000000-0000-0000-0000-00005f41b415"
-          (reference "#PWR01505") (unit 1)
-        )
-        (path "/e85aac8c-404c-45dd-bda3-1057cae83baf/00000000-0000-0000-0000-00005f41b451"
-          (reference "#PWR01801") (unit 1)
+          (reference "#PWR?") (unit 1)
+        )
+        (path "/e85aac8c-404c-45dd-bda3-1057cae83baf/00000000-0000-0000-0000-00005f41b451"
+          (reference "#PWR02101") (unit 1)
         )
       )
@@
         )
         (path "/e85aac8c-404c-45dd-bda3-1057cae83baf/00000000-0000-0000-0000-00005f41b415"
-          (reference "#PWR01503") (unit 1)
-        )
-        (path "/e85aac8c-404c-45dd-bda3-1057cae83baf/00000000-0000-0000-0000-00005f41b451"
-          (reference "#PWR01803") (unit 1)
+          (reference "#PWR?") (unit 1)
+        )
+        (path "/e85aac8c-404c-45dd-bda3-1057cae83baf/00000000-0000-0000-0000-00005f41b451"
+          (reference "#PWR02103") (unit 1)
         )
       )
@@
         )
         (path "/e85aac8c-404c-45dd-bda3-1057cae83baf/00000000-0000-0000-0000-00005f41b451"
-          (reference "R?") (unit 1)
+          (reference "R2102") (unit 1)
         )
       )
@@
   (symbol (lib_id "Custom Library:CHASSIS") (at 210.82 96.52 0) (unit 1)
     (in_bom yes) (on_board yes) (dnp no)
-    (property "Reference" "#PWR01506" (at 210.82 101.6 0)
+    (property "Reference" "#PWR?" (at 210.82 101.6 0)
       (effects (font (size 1.27 1.27)) hide)
     )
@@
       (project "USB_Hub"
         (path "/e85aac8c-404c-45dd-bda3-1057cae83baf/00000000-0000-0000-0000-00005f41b415"
-          (reference "#PWR01506") (unit 1)
-        )
-        (path "/e85aac8c-404c-45dd-bda3-1057cae83baf/00000000-0000-0000-0000-00005f41b451"
-          (reference "#PWR01806") (unit 1)
+          (reference "#PWR?") (unit 1)
+        )
+        (path "/e85aac8c-404c-45dd-bda3-1057cae83baf/00000000-0000-0000-0000-00005f41b451"
+          (reference "#PWR02106") (unit 1)
         )
       )
@@
         )
         (path "/e85aac8c-404c-45dd-bda3-1057cae83baf/00000000-0000-0000-0000-00005f41b451"
-          (reference "D?") (unit 1)
+          (reference "D2101") (unit 1)
         )
       )
@@
         )
         (path "/e85aac8c-404c-45dd-bda3-1057cae83baf/00000000-0000-0000-0000-00005f41b451"
-          (reference "C?") (unit 1)
+          (reference "C2102") (unit 1)
         )
       )
@@
         )
         (path "/e85aac8c-404c-45dd-bda3-1057cae83baf/00000000-0000-0000-0000-00005f41b451"
-          (reference "C?") (unit 1)
+          (reference "C2101") (unit 1)
         )
       )
@@
         )
         (path "/e85aac8c-404c-45dd-bda3-1057cae83baf/00000000-0000-0000-0000-00005f41b451"
-          (reference "R?") (unit 1)
+          (reference "R2101") (unit 1)
         )
       )
@@
         )
         (path "/e85aac8c-404c-45dd-bda3-1057cae83baf/00000000-0000-0000-0000-00005f41b415"
-          (reference "#PWR01501") (unit 1)
-        )
-        (path "/e85aac8c-404c-45dd-bda3-1057cae83baf/00000000-0000-0000-0000-00005f41b451"
-          (reference "#PWR01804") (unit 1)
+          (reference "#PWR?") (unit 1)
+        )
+        (path "/e85aac8c-404c-45dd-bda3-1057cae83baf/00000000-0000-0000-0000-00005f41b451"
+          (reference "#PWR02104") (unit 1)
         )
       )
@@
         )
         (path "/e85aac8c-404c-45dd-bda3-1057cae83baf/00000000-0000-0000-0000-00005f41b415"
-          (reference "#PWR01504") (unit 1)
-        )
-        (path "/e85aac8c-404c-45dd-bda3-1057cae83baf/00000000-0000-0000-0000-00005f41b451"
-          (reference "#PWR01802") (unit 1)
+          (reference "#PWR?") (unit 1)
+        )
+        (path "/e85aac8c-404c-45dd-bda3-1057cae83baf/00000000-0000-0000-0000-00005f41b451"
+          (reference "#PWR02102") (unit 1)
         )
       )
@@
         )
         (path "/e85aac8c-404c-45dd-bda3-1057cae83baf/00000000-0000-0000-0000-00005f41b451"
-          (reference "J?") (unit 1)
-        )
-      )
+          (reference "J2101") (unit 1)
+        )
+      )

Commit message: pulled footprints into layout
Parts:
- C?: footprint Capacitors_Tantalum_SMD:CP_Tantalum_Case-X_EIA-7343-43_Reflow -> Capacitor_Tantalum_SMD:CP_EIA-7343-43_Kemet-X
- J?: footprint (none) -> Connector_USB:USB_A_Molex_67643_Horizontal
- R? (x2): Digi-Key PN 311-27.0HRCT-ND -> (none)
Changed lines of the file:
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@@
       (effects (font (size 1.27 1.27)) (justify left))
     )
-    (property "Footprint" "Capacitors_Tantalum_SMD:CP_Tantalum_Case-X_EIA-7343-43_Reflow" (at 186.3852 96.52 0)
+    (property "Footprint" "Capacitor_Tantalum_SMD:CP_EIA-7343-43_Kemet-X" (at 186.3852 96.52 0)
       (effects (font (size 1.27 1.27)) hide)
     )
@@
       (effects (font (size 1.27 1.27)) hide)
     )
-    (property "Digi-Key PN" "311-27.0HRCT-ND" (at 135.89 91.44 0)
+    (property "Digi-Key PN" "" (at 135.89 91.44 0)
       (effects (font (size 1.524 1.524)) hide)
     )
@@
       (effects (font (size 1.27 1.27)) hide)
     )
-    (property "Digi-Key PN" "311-27.0HRCT-ND" (at 135.89 73.66 0)
+    (property "Digi-Key PN" "" (at 135.89 73.66 0)
       (effects (font (size 1.524 1.524)) hide)
     )
@@
       (effects (font (size 1.27 1.27)) (justify left))
     )
-    (property "Footprint" "" (at 201.93 82.55 0)
-      (effects (font (size 1.27 1.27)) hide)
-    )
+    (property "Footprint" "Connector_USB:USB_A_Molex_67643_Horizontal" (at 201.93 82.55 0)
+      (effects (font (size 1.27 1.27)) hide)
+    )

Commit message: fixed footprints, assigned digikey pns
Parts:
- C? (x2): Digi-Key PN (none) -> 1292-1501-1-ND
- D?: Digi-Key PN (none) -> F2715CT-ND
- J?: footprint Connector_USB:USB_A_Molex_67643_Horizontal -> Connector_USB:USB_A_Wuerth_614004134726_Horizontal; Digi-Key PN (none) -> 732-2731-ND
- R? (x2): Digi-Key PN (none) -> 541-27.0HCT-ND
Changed lines of the file:
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@@
-    (stroke (width 0) (type default))
-  )
-  (wire (pts (xy 185.42 74.93) (xy 185.42 76.2))
     (stroke (width 0) (type default))
   )
@@
     )
   )
-  (symbol (lib_id "power:PWR_FLAG") (at 185.42 74.93 0) (unit 1)
-    (in_bom yes) (on_board yes) (dnp no)
-    (property "Reference" "#FLG?" (at 185.42 73.025 0)
-      (effects (font (size 1.27 1.27)) hide)
-    )
-    (property "Value" "PWR_FLAG" (at 185.42 71.12 0)
-      (effects (font (size 1.27 1.27)))
-    )
-    (property "Footprint" "" (at 185.42 74.93 0)
-      (effects (font (size 1.27 1.27)) hide)
-    )
-    (property "Datasheet" "~" (at 185.42 74.93 0)
-      (effects (font (size 1.27 1.27)) hide)
-    )
-    (pin "1")
-    (instances
-      (project "USB_Hub"
-        (path "/e85aac8c-404c-45dd-bda3-1057cae83baf/00000000-0000-0000-0000-00005f41b415"
-          (reference "#FLG?") (unit 1)
-        )
-        (path "/e85aac8c-404c-45dd-bda3-1057cae83baf/00000000-0000-0000-0000-00005f41b451"
-          (reference "#FLG01301") (unit 1)
-        )
-      )
-    )
-  )
   (symbol (lib_id "power:GND") (at 203.2 96.52 0) (unit 1)
     (in_bom yes) (on_board yes) (dnp no)
@@
       (effects (font (size 1.27 1.27)) hide)
     )
-    (property "Digi-Key PN" "" (at 135.89 91.44 0)
+    (property "Digi-Key PN" "541-27.0HCT-ND" (at 135.89 91.44 0)
       (effects (font (size 1.524 1.524)) hide)
     )
@@
     )
     (property "Datasheet" "http://www.littelfuse.com/~/media/files/littelfuse/technical%20resources/documents/data%20sheets/sp05xxba.pdf" (at 160.655 88.265 0)
+      (effects (font (size 1.27 1.27)) hide)
+    )
+    (property "Digi-Key PN" "F2715CT-ND" (at 157.48 91.44 0)
       (effects (font (size 1.27 1.27)) hide)
     )
@@
       (effects (font (size 1.27 1.27)) (justify right))
     )
-    (property "Digi-Key PN" "" (at 106.68 92.71 0)
+    (property "Digi-Key PN" "1292-1501-1-ND" (at 106.68 92.71 0)
       (effects (font (size 1.27 1.27)) hide)
     )
@@
       (effects (font (size 1.27 1.27)) (justify right))
     )
-    (property "Digi-Key PN" "" (at 88.9 92.71 0)
+    (property "Digi-Key PN" "1292-1501-1-ND" (at 88.9 92.71 0)
       (effects (font (size 1.27 1.27)) hide)
     )
@@
       (effects (font (size 1.27 1.27)) hide)
     )
-    (property "Digi-Key PN" "" (at 135.89 73.66 0)
+    (property "Digi-Key PN" "541-27.0HCT-ND" (at 135.89 73.66 0)
       (effects (font (size 1.524 1.524)) hide)
     )
@@
       (effects (font (size 1.27 1.27)) (justify left))
     )
-    (property "Footprint" "Connector_USB:USB_A_Molex_67643_Horizontal" (at 201.93 82.55 0)
+    (property "Footprint" "Connector_USB:USB_A_Wuerth_614004134726_Horizontal" (at 201.93 82.55 0)
       (effects (font (size 1.27 1.27)) hide)
     )
@@
       (effects (font (size 1.27 1.27)) hide)
     )
+    (property "Digi-Key PN" "732-2731-ND" (at 205.74 81.28 0)
+      (effects (font (size 1.27 1.27)) hide)
+    )

Commit message: fixed some netlist connectivity issues, finished grouping parts in PCB
Connections:
- net DFP3_USB_CONN_D+: now also D?.4 (K); no longer D?.3 (K)
- net DFP3_USB_CONN_D-: now also D?.3 (K); no longer D?.4 (K)
Changed lines of the file:
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@@
     (company "Drew Maatman")
   )
-  (junction (at 157.48 81.28) (diameter 0) (color 0 0 0 0)
+  (junction (at 157.48 83.82) (diameter 0) (color 0 0 0 0)
   )
   (junction (at 88.9 81.28) (diameter 0) (color 0 0 0 0)
+  )
+  (junction (at 160.02 81.28) (diameter 0) (color 0 0 0 0)
   )
   (junction (at 106.68 83.82) (diameter 0) (color 0 0 0 0)
@@
   (junction (at 185.42 76.2) (diameter 0) (color 0 0 0 0)
   )
-  (junction (at 160.02 83.82) (diameter 0) (color 0 0 0 0)
-  )
   (wire (pts (xy 76.2 81.28) (xy 88.9 81.28))
     (stroke (width 0) (type default))
@@
     (stroke (width 0) (type default))
   )
+  (wire (pts (xy 160.02 81.28) (xy 160.02 86.36))
+    (stroke (width 0) (type default))
+  )
   (wire (pts (xy 203.2 95.25) (xy 205.74 95.25))
     (stroke (width 0) (type default))
   )
-  (wire (pts (xy 129.54 81.28) (xy 157.48 81.28))
-    (stroke (width 0) (type default))
-  )
-  (wire (pts (xy 160.02 83.82) (xy 198.12 83.82))
+  (wire (pts (xy 129.54 83.82) (xy 157.48 83.82))
     (stroke (width 0) (type default))
   )
   (wire (pts (xy 106.68 83.82) (xy 106.68 88.9))
+    (stroke (width 0) (type default))
+  )
+  (wire (pts (xy 160.02 81.28) (xy 198.12 81.28))
     (stroke (width 0) (type default))
   )
@@
     (stroke (width 0) (type default))
   )
-  (wire (pts (xy 129.54 83.82) (xy 160.02 83.82))
-    (stroke (width 0) (type default))
-  )
   (wire (pts (xy 88.9 81.28) (xy 121.92 81.28))
     (stroke (width 0) (type default))
@@
     (stroke (width 0) (type default))
   )
-  (wire (pts (xy 157.48 81.28) (xy 198.12 81.28))
+  (wire (pts (xy 129.54 81.28) (xy 160.02 81.28))
+    (stroke (width 0) (type default))
+  )
+  (wire (pts (xy 157.48 83.82) (xy 198.12 83.82))
     (stroke (width 0) (type default))
   )
@@
     (stroke (width 0) (type default))
   )
-  (wire (pts (xy 160.02 83.82) (xy 160.02 86.36))
-    (stroke (width 0) (type default))
-  )
   (wire (pts (xy 210.82 96.52) (xy 210.82 95.25))
     (stroke (width 0) (type default))
@@
     (stroke (width 0) (type default))
   )
-  (wire (pts (xy 157.48 81.28) (xy 157.48 86.36))
+  (wire (pts (xy 157.48 83.82) (xy 157.48 86.36))
     (stroke (width 0) (type default))
   )
@@
     (effects (font (size 1.27 1.27)) (justify right))
     (property "Intersheetrefs" "${INTERSHEET_REFS}" (at 59.5702 83.82 0)
-      (effects (font (size 1.27 1.27)) (justify right) hide)
+      (effects (font (size 1.27 1.27)) (justify right))
     )
   )
@@
     (effects (font (size 1.27 1.27)) (justify right))
     (property "Intersheetrefs" "${INTERSHEET_REFS}" (at 63.2441 76.2 0)
-      (effects (font (size 1.27 1.27)) (justify right) hide)
+      (effects (font (size 1.27 1.27)) (justify right))
     )
   )
@@
     (effects (font (size 1.27 1.27)) (justify right))
     (property "Intersheetrefs" "${INTERSHEET_REFS}" (at 59.5702 81.28 0)
-      (effects (font (size 1.27 1.27)) (justify right) hide)
+      (effects (font (size 1.27 1.27)) (justify right))
     )
   )
