File: hdw/USB_Hub/Hub_LEDs.kicad_sch (KiCad schematic)
At the start: 0 parts

Commit message: lots of schematic progress
Other:
- company: (none) -> Drew Maatman
- title: (none) -> USB Hub
Changed lines of the file:
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@@
 (kicad_sch (version 20230121) (generator eeschema)
   (paper "A")
+  (title_block
+    (title "USB Hub")
+    (date "2023-08-18")
+    (rev "PRELIM")
+    (company "Drew Maatman")
+  )
 )

Commit message: much more schematic progress
Parts:
- added C1505 (x8), C?: 0.1uF, Capacitors_SMD:C_0603, symbol Custom_Library:C_Custom
- added D1505 (x4): Red, LEDs:LED_0603, symbol Device:LED
- added D1505 (x4): Green, LEDs:LED_0603, symbol Device:LED
- added R1506 (x8): 1k, Resistors_SMD:R_0603, symbol Custom_Library:R_Custom
- added R? (x2): 10k, Resistors_SMD:R_0603, symbol Custom_Library:R_Custom
- added U?: 74LVC1G97, Package_TO_SOT_SMD:SOT-363_SC-70-6, symbol Custom Library:74LVC1G97_Power_NOT
- added U? (x4): 74LVC1G97, Package_TO_SOT_SMD:SOT-363_SC-70-6, symbol Custom Library:74LVC1G97_Power_OR_INV
- added U? (x4): 74LVC1G97, Package_TO_SOT_SMD:SOT-363_SC-70-6, symbol Custom Library:74LVC1G97_Power_NAND_INV
Connections:
- new net: D1505.2 (A), R1506.2 (x8)
- new net: D1505.1 (K), U?.4 (x8)
- new net +3.3V: C1505.1, C1505.1, C1505.1, C1505.1, C1505.1, C1505.1, C1505.1, C1505.1, C?.1, R1506.1, R1506.1, R1506.1, R1506.1, R1506.1, R1506.1, R1506.1, R1506.1, R?.1, U?.1 (VCC), U?.1 (VCC), U?.1 (VCC), U?.1 (VCC), U?.1 (VCC), U?.1 (VCC), U?.1 (VCC), U?.1 (VCC), U?.1 (VCC), U?.5 (VCC), U?.5 (VCC), U?.5 (VCC), U?.5 (VCC), U?.5 (VCC), U?.5 (VCC), U?.5 (VCC), U?.5 (VCC), U?.5 (VCC)
- new net GND: C1505.2, C1505.2, C1505.2, C1505.2, C1505.2, C1505.2, C1505.2, C1505.2, C?.2, R?.2, U?.2 (GND), U?.2 (GND), U?.2 (GND), U?.2 (GND), U?.2 (GND), U?.2 (GND), U?.2 (GND), U?.2 (GND), U?.2 (GND), U?.3 (GND)
- new net PGOOD_LED_SHDN: R?.1, U?.6
- new net ~{DFP0_EN}: U?.3
- new net ~{DFP0_OC}: U?.3
- new net ~{DFP1_EN}: U?.3
- new net ~{DFP1_OC}: U?.3
- new net ~{DFP2_EN}: U?.3
- new net ~{DFP2_OC}: U?.3
- new net ~{DFP3_EN}: U?.3
- new net ~{DFP3_OC}: U?.3
- new net ~{HUB_LED_SHDN}: R?.2, U?.4, U?.6, U?.6, U?.6, U?.6, U?.6, U?.6, U?.6, U?.6
Other:
- note added: "6 3 4 L L H L H H H L L H H H"

Commit message: lots and lots of sch progress
Parts:
- gave numbers to parts that had none: 8
- renumbered C1505 to C?, D1505 to D?, R1506 to R?

Commit message: pulled footprints into layout
Parts:
- C?: Digi-Key PN 399-7845-1-ND -> 1276-1935-1-ND
- D? (x4): Digi-Key PN (none) -> 754-1117-1-ND
- R? (x8): Digi-Key PN 541-1.00KHCT-ND -> (none)
- R? (x2): Digi-Key PN YAG2321CT-ND -> (none)
- U1402, U1403, U1404, U1405, U1406, U1407, U1408, U1409, U?: Digi-Key PN (none) -> 296-15582-1-ND
Changed lines of the file:
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@@
       (effects (font (size 1.27 1.27)) (justify left))
     )
-    (property "Digi-Key PN" "541-1.00KHCT-ND" (at 161.29 133.35 0)
+    (property "Digi-Key PN" "" (at 161.29 133.35 0)
       (effects (font (size 1.524 1.524)) hide)
     )
@@
       (effects (font (size 1.27 1.27)) hide)
     )
+    (property "Digi-Key PN" "296-15582-1-ND" (at 53.34 43.18 0)
+      (effects (font (size 1.27 1.27)) hide)
+    )
     (pin "1")
     (pin "2")
@@
       (effects (font (size 1.27 1.27)) hide)
     )
-    (property "Digi-Key PN" "" (at 392.938 167.894 0)
+    (property "Digi-Key PN" "754-1117-1-ND" (at 392.938 167.894 0)
       (effects (font (size 1.27 1.27)) hide)
     )
@@
       (effects (font (size 1.27 1.27)) hide)
     )
+    (property "Digi-Key PN" "296-15582-1-ND" (at 218.44 157.48 0)
+      (effects (font (size 1.27 1.27)) hide)
+    )
     (pin "1")
     (pin "2")
@@
       (effects (font (size 1.27 1.27)) hide)
     )
+    (property "Digi-Key PN" "296-15582-1-ND" (at 154.94 119.38 0)
+      (effects (font (size 1.27 1.27)) hide)
+    )
     (pin "1")
     (pin "2")
@@
       (effects (font (size 1.27 1.27)) hide)
     )
+    (property "Digi-Key PN" "296-15582-1-ND" (at 154.94 157.48 0)
+      (effects (font (size 1.27 1.27)) hide)
+    )
     (pin "1")
     (pin "2")
@@
       (effects (font (size 1.27 1.27)) hide)
     )
+    (property "Digi-Key PN" "296-15582-1-ND" (at 218.44 81.28 0)
+      (effects (font (size 1.27 1.27)) hide)
+    )
     (pin "1")
     (pin "2")
@@
       (effects (font (size 1.27 1.27)) hide)
     )
-    (property "Digi-Key PN" "399-7845-1-ND" (at 40.005 13.335 0)
+    (property "Digi-Key PN" "1276-1935-1-ND" (at 40.005 13.335 0)
       (effects (font (size 1.524 1.524)) hide)
     )
@@
       (effects (font (size 1.27 1.27)) (justify left))
     )
-    (property "Digi-Key PN" "YAG2321CT-ND" (at 39.37 49.53 0)
+    (property "Digi-Key PN" "" (at 39.37 49.53 0)
       (effects (font (size 1.27 1.27)) hide)
     )
@@
       (effects (font (size 1.27 1.27)) hide)
     )
-    (property "Digi-Key PN" "" (at 392.938 205.994 0)
+    (property "Digi-Key PN" "754-1117-1-ND" (at 392.938 205.994 0)
       (effects (font (size 1.27 1.27)) hide)
     )
@@
       (effects (font (size 1.27 1.27)) hide)
     )
-    (property "Digi-Key PN" "" (at 392.938 244.094 0)
+    (property "Digi-Key PN" "754-1117-1-ND" (at 392.938 244.094 0)
       (effects (font (size 1.27 1.27)) hide)
     )
@@
       (effects (font (size 1.27 1.27)) (justify left))
     )
-    (property "Digi-Key PN" "541-1.00KHCT-ND" (at 224.79 133.35 0)
+    (property "Digi-Key PN" "" (at 224.79 133.35 0)
       (effects (font (size 1.524 1.524)) hide)
     )
@@
       (effects (font (size 1.27 1.27)) (justify left))
     )
-    (property "Digi-Key PN" "541-1.00KHCT-ND" (at 161.29 57.15 0)
+    (property "Digi-Key PN" "" (at 161.29 57.15 0)
       (effects (font (size 1.524 1.524)) hide)
     )
@@
       (effects (font (size 1.27 1.27)) (justify left))
     )
-    (property "Digi-Key PN" "541-1.00KHCT-ND" (at 224.79 95.25 0)
+    (property "Digi-Key PN" "" (at 224.79 95.25 0)
       (effects (font (size 1.524 1.524)) hide)
     )
@@
       (effects (font (size 1.27 1.27)) (justify left))
     )
-    (property "Digi-Key PN" "541-1.00KHCT-ND" (at 161.29 95.25 0)
+    (property "Digi-Key PN" "" (at 161.29 95.25 0)
       (effects (font (size 1.524 1.524)) hide)
     )
@@
       (effects (font (size 1.27 1.27)) hide)
     )
+    (property "Digi-Key PN" "296-15582-1-ND" (at 218.44 119.38 0)
+      (effects (font (size 1.27 1.27)) hide)
+    )
     (pin "1")
     (pin "2")
@@
       (effects (font (size 1.27 1.27)) hide)
     )
+    (property "Digi-Key PN" "296-15582-1-ND" (at 218.44 43.18 0)
+      (effects (font (size 1.27 1.27)) hide)
+    )
     (pin "1")
     (pin "2")
@@
       (effects (font (size 1.27 1.27)) (justify left))
     )
-    (property "Digi-Key PN" "YAG2321CT-ND" (at 72.39 36.83 0)
+    (property "Digi-Key PN" "" (at 72.39 36.83 0)
       (effects (font (size 1.27 1.27)) hide)
     )
@@
       (effects (font (size 1.27 1.27)) hide)
     )
-    (property "Digi-Key PN" "" (at 392.938 282.194 0)
+    (property "Digi-Key PN" "754-1117-1-ND" (at 392.938 282.194 0)
       (effects (font (size 1.27 1.27)) hide)
     )
@@
       (effects (font (size 1.27 1.27)) hide)
     )
+    (property "Digi-Key PN" "296-15582-1-ND" (at 154.94 43.18 0)
+      (effects (font (size 1.27 1.27)) hide)
+    )
     (pin "1")
     (pin "2")
@@
       (effects (font (size 1.27 1.27)) (justify left))
     )
-    (property "Digi-Key PN" "541-1.00KHCT-ND" (at 224.79 57.15 0)
+    (property "Digi-Key PN" "" (at 224.79 57.15 0)
       (effects (font (size 1.524 1.524)) hide)
     )
@@
       (effects (font (size 1.27 1.27)) (justify left))
     )
-    (property "Digi-Key PN" "541-1.00KHCT-ND" (at 224.79 19.05 0)
+    (property "Digi-Key PN" "" (at 224.79 19.05 0)
       (effects (font (size 1.524 1.524)) hide)
     )
@@
       (effects (font (size 1.27 1.27)) hide)
     )
+    (property "Digi-Key PN" "296-15582-1-ND" (at 154.94 81.28 0)
+      (effects (font (size 1.27 1.27)) hide)
+    )
     (pin "1")
     (pin "2")
@@
       (effects (font (size 1.27 1.27)) (justify left))
     )
-    (property "Digi-Key PN" "541-1.00KHCT-ND" (at 161.29 19.05 0)
+    (property "Digi-Key PN" "" (at 161.29 19.05 0)
       (effects (font (size 1.524 1.524)) hide)
     )

Commit message: big restructuring, removed microcontroller and all telemtry
Parts:
- removed C?: 0.1uF, Capacitors_SMD:C_0603, symbol Custom_Library:C_Custom
- removed R? (x2): 10k, Resistors_SMD:R_0603, symbol Custom_Library:R_Custom
- removed U1402, U1403, U1404, U1405: 74LVC1G97, Package_TO_SOT_SMD:SOT-363_SC-70-6, symbol Custom Library:74LVC1G97_Power_NAND_INV
- removed U1406, U1407, U1408, U1409: 74LVC1G97, Package_TO_SOT_SMD:SOT-363_SC-70-6, symbol Custom Library:74LVC1G97_Power_OR_INV
- removed U?: 74LVC1G97, Package_TO_SOT_SMD:SOT-363_SC-70-6, symbol Custom Library:74LVC1G97_Power_NOT
- added C? (x2): 0.1uF, Capacitors_SMD:C_0603, symbol Custom_Library:C_Custom
- added D?: Green, LEDs:LED_0603, symbol Device:LED
- added D?: Red, LEDs:LED_0603, symbol Device:LED
- added R? (x2): 1k, Resistors_SMD:R_0603, symbol Custom_Library:R_Custom
- added U701, U702, U703, U704, U705, U706, U707, U708: 74LVC1G97, Package_TO_SOT_SMD:SOT-363_SC-70-6, symbol Custom Library:74LVC1G97_Power_BUF
- added U? (x2): 74LVC1G97, Package_TO_SOT_SMD:SOT-363_SC-70-6, symbol Custom Library:74LVC1G97_Power_NOT
Connections:
- net GND: now also C?.2, C?.2, U701.2 (GND), U701.3 (GND), U701.6 (GND), U702.2 (GND), U702.3 (GND), U702.6 (GND), U703.2 (GND), U703.3 (GND), U703.6 (GND), U704.2 (GND), U704.3 (GND), U704.6 (GND), U705.2 (GND), U705.3 (GND), U705.6 (GND), U706.2 (GND), U706.3 (GND), U706.6 (GND), U707.2 (GND), U707.3 (GND), U707.6 (GND), U708.2 (GND), U708.3 (GND), U708.6 (GND), U?.2 (GND), U?.2 (GND), U?.3 (GND), U?.3 (GND)
- net ~{DFP0_EN}: now also U701.1
- net ~{DFP0_OC}: now also U705.1
- net ~{DFP1_EN}: now also U702.1
- net ~{DFP1_OC}: now also U706.1
- net ~{DFP2_EN}: now also U703.1
- net ~{DFP2_OC}: now also U707.1
- net ~{DFP3_EN}: now also U704.1
- net ~{DFP3_OC}: now also U708.1
- net at D?.1 (K): now also U705.4
- net at D?.1 (K): now also U701.4
- net at D?.1 (K): now also U708.4
- net at D?.1 (K): now also U703.4
- net at D?.1 (K): now also U704.4
- net at D?.1 (K): now also U706.4
- net at D?.1 (K): now also U707.4
- net at D?.1 (K): now also U702.4
- net +3.3V renamed +5V
- net +5V: now also C?.1, C?.1, R?.1, R?.1, U701.5 (VCC), U702.5 (VCC), U703.5 (VCC), U704.5 (VCC), U705.5 (VCC), U706.5 (VCC), U707.5 (VCC), U708.5 (VCC), U?.1 (VCC), U?.1 (VCC), U?.5 (VCC), U?.5 (VCC)
- new net: D?.1 (K), U?.4 (x2)
- new net: D?.2 (A), R?.2 (x2)
- new net HUB_BUSPWR: U?.6
- new net HUB_SUSPND: U?.6
Other:
- note added: "High when wall wart powering output, low when upstream VBUS powering output. This should not change during operation"
- note removed: "6 3 4 L L H L H H H L L H H H"
- moved on the sheet: C?, D?, R?

Commit message: fixed footprints, assigned digikey pns
Parts:
- R? (x10): Digi-Key PN (none) -> 541-1.00KHCT-ND
- U701, U702, U703, U704, U705, U706, U707, U708, U? (x2): Digi-Key PN (none) -> 1727-1772-1-ND
Changed lines of the file:
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@@
       (effects (font (size 1.27 1.27)) (justify left))
     )
-    (property "Digi-Key PN" "" (at 97.79 134.62 0)
+    (property "Digi-Key PN" "541-1.00KHCT-ND" (at 97.79 134.62 0)
       (effects (font (size 1.524 1.524)) hide)
     )
@@
       (effects (font (size 1.27 1.27)) hide)
     )
+    (property "Digi-Key PN" "1727-1772-1-ND" (at 91.44 120.65 0)
+      (effects (font (size 1.27 1.27)) hide)
+    )
     (pin "1")
     (pin "2")
@@
       (effects (font (size 1.27 1.27)) hide)
     )
+    (property "Digi-Key PN" "1727-1772-1-ND" (at 218.44 82.55 0)
+      (effects (font (size 1.27 1.27)) hide)
+    )
     (pin "1")
     (pin "2")
@@
       (effects (font (size 1.27 1.27)) hide)
     )
+    (property "Digi-Key PN" "1727-1772-1-ND" (at 154.94 82.55 0)
+      (effects (font (size 1.27 1.27)) hide)
+    )
     (pin "1")
     (pin "2")
@@
       (effects (font (size 1.27 1.27)) (justify left))
     )
-    (property "Digi-Key PN" "" (at 224.79 20.32 0)
+    (property "Digi-Key PN" "541-1.00KHCT-ND" (at 224.79 20.32 0)
       (effects (font (size 1.524 1.524)) hide)
     )
@@
       (effects (font (size 1.27 1.27)) hide)
     )
+    (property "Digi-Key PN" "1727-1772-1-ND" (at 154.94 120.65 0)
+      (effects (font (size 1.27 1.27)) hide)
+    )
     (pin "1")
     (pin "2")
@@
       (effects (font (size 1.27 1.27)) hide)
     )
+    (property "Digi-Key PN" "1727-1772-1-ND" (at 91.44 82.55 0)
+      (effects (font (size 1.27 1.27)) hide)
+    )
     (pin "1")
     (pin "2")
@@
       (effects (font (size 1.27 1.27)) hide)
     )
+    (property "Digi-Key PN" "1727-1772-1-ND" (at 91.44 44.45 0)
+      (effects (font (size 1.27 1.27)) hide)
+    )
     (pin "1")
     (pin "2")
@@
       (effects (font (size 1.27 1.27)) (justify left))
     )
-    (property "Digi-Key PN" "" (at 161.29 134.62 0)
+    (property "Digi-Key PN" "541-1.00KHCT-ND" (at 161.29 134.62 0)
       (effects (font (size 1.524 1.524)) hide)
     )
@@
       (effects (font (size 1.27 1.27)) (justify left))
     )
-    (property "Digi-Key PN" "" (at 97.79 58.42 0)
+    (property "Digi-Key PN" "541-1.00KHCT-ND" (at 97.79 58.42 0)
       (effects (font (size 1.524 1.524)) hide)
     )
@@
       (effects (font (size 1.27 1.27)) (justify left))
     )
-    (property "Digi-Key PN" "" (at 161.29 96.52 0)
+    (property "Digi-Key PN" "541-1.00KHCT-ND" (at 161.29 96.52 0)
       (effects (font (size 1.524 1.524)) hide)
     )
@@
       (effects (font (size 1.27 1.27)) (justify left))
     )
-    (property "Digi-Key PN" "" (at 97.79 96.52 0)
+    (property "Digi-Key PN" "541-1.00KHCT-ND" (at 97.79 96.52 0)
       (effects (font (size 1.524 1.524)) hide)
     )
@@
       (effects (font (size 1.27 1.27)) (justify left))
     )
-    (property "Digi-Key PN" "" (at 224.79 58.42 0)
+    (property "Digi-Key PN" "541-1.00KHCT-ND" (at 224.79 58.42 0)
       (effects (font (size 1.524 1.524)) hide)
     )
@@
       (effects (font (size 1.27 1.27)) (justify left))
     )
-    (property "Digi-Key PN" "" (at 161.29 58.42 0)
+    (property "Digi-Key PN" "541-1.00KHCT-ND" (at 161.29 58.42 0)
       (effects (font (size 1.524 1.524)) hide)
     )
@@
       (effects (font (size 1.27 1.27)) hide)
     )
+    (property "Digi-Key PN" "1727-1772-1-ND" (at 154.94 158.75 0)
+      (effects (font (size 1.27 1.27)) hide)
+    )
     (pin "1")
     (pin "2")
@@
       (effects (font (size 1.27 1.27)) hide)
     )
+    (property "Digi-Key PN" "1727-1772-1-ND" (at 91.44 158.75 0)
+      (effects (font (size 1.27 1.27)) hide)
+    )
     (pin "1")
     (pin "2")
@@
       (effects (font (size 1.27 1.27)) hide)
     )
+    (property "Digi-Key PN" "1727-1772-1-ND" (at 154.94 44.45 0)
+      (effects (font (size 1.27 1.27)) hide)
+    )
     (pin "1")
     (pin "2")
@@
       (effects (font (size 1.27 1.27)) (justify left))
     )
-    (property "Digi-Key PN" "" (at 161.29 20.32 0)
+    (property "Digi-Key PN" "541-1.00KHCT-ND" (at 161.29 20.32 0)
       (effects (font (size 1.524 1.524)) hide)
     )
@@
       (effects (font (size 1.27 1.27)) hide)
     )
+    (property "Digi-Key PN" "1727-1772-1-ND" (at 218.44 44.45 0)
+      (effects (font (size 1.27 1.27)) hide)
+    )
     (pin "1")
     (pin "2")
@@
       (effects (font (size 1.27 1.27)) (justify left))
     )
-    (property "Digi-Key PN" "" (at 97.79 20.32 0)
+    (property "Digi-Key PN" "541-1.00KHCT-ND" (at 97.79 20.32 0)
       (effects (font (size 1.524 1.524)) hide)
     )
