File: hdw/USB_Hub/Upstream_Port.kicad_sch (KiCad schematic)
At the start: 0 parts

Commit message: lots of schematic progress
Other:
- company: (none) -> Drew Maatman
- title: (none) -> USB Hub
Changed lines of the file:
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@@
 (kicad_sch (version 20230121) (generator eeschema)
   (paper "A")
+  (title_block
+    (title "USB Hub")
+    (date "2023-08-18")
+    (rev "PRELIM")
+    (company "Drew Maatman")
+  )
+  (symbol (lib_id "power:VBUS") (at 203.2 94.615 0) (unit 1)
+    (in_bom yes) (on_board yes) (dnp no)
+    (property "Reference" "#PWR02012" (at 203.2 98.425 0)
+      (effects (font (size 1.27 1.27)) hide)
+    )
+    (property "Value" "VBUS" (at 203.2 90.805 0)
+      (effects (font (size 1.27 1.27)))
+    )
+    (property "Footprint" "" (at 203.2 94.615 0)
+      (effects (font (size 1.27 1.27)) hide)
+    )
+    (property "Datasheet" "" (at 203.2 94.615 0)
+      (effects (font (size 1.27 1.27)) hide)
+    )
+    (pin "1")
+    (instances
+      (project "USB_Hub"
+        (path "/e85aac8c-404c-45dd-bda3-1057cae83baf/5b35e0c1-9928-450a-ba6b-f2a701eceaac"
+          (reference "#PWR02012") (unit 1)
+        )
+        (path "/e85aac8c-404c-45dd-bda3-1057cae83baf/00000000-0000-0000-0000-00005f41b463"
+          (reference "#PWR02201") (unit 1)
+        )
+      )
+    )
+  )
 )

Commit message: much more schematic progress
Parts:
- added C1306: 0.1uF, Capacitors_SMD:C_0603, symbol Custom_Library:C_Custom
- added C? (x2): 22pF, Capacitors_SMD:C_0603, symbol Custom_Library:C_Custom
- added J1301: USB_B_Mini, Connectors:USB_Mini-B, symbol Connector:USB_B_Mini
- added L1302: 600R 0.5A, Inductors_SMD:L_0603, symbol Device:Ferrite_Bead
- added R1311, R1312: 27, Resistors_SMD:R_0603, symbol Custom_Library:R_Custom
- added TP?: TP, Custom Footprints Library:Test_Point, symbol Custom_Library:TP
- added U1305: TPD3S014DBVR, TO_SOT_Packages_SMD:SOT-23-6, symbol Custom_Library:TPD3S014DBVR
Connections:
- net VBUS: now also C1306.1, TP?.1 (TP), U1305.4 (OUT)
- new net: J1301.1 (VBUS), U1305.1 (EN), U1305.3 (IN)
- new net: J1301.6 (Shield), L1302.2
- new net GND: C1306.2, C?.2, C?.2, J1301.5 (GND), L1302.1, U1305.2 (GND)
- new net UFP_USB_CONN_USB+: C?.1, J1301.3 (D+), R1311.1, U1305.6 (D1)
- new net UFP_USB_CONN_USB-: C?.1, J1301.2 (D-), R1312.1, U1305.5 (D2)
- new net UFP_USB_D+: R1311.2
- new net UFP_USB_D-: R1312.2
- no-connect marks 0 -> 1

Commit message: lots and lots of sch progress
Parts:
- removed L1302: 600R 0.5A, Inductors_SMD:L_0603, symbol Device:Ferrite_Bead
- U?: renamed from U1305; value TPD3S014DBVR -> TPD3S044DBVR; Digi-Key PN 296-38835-1-ND -> 296-38836-1-ND
- renumbered C1306 to C?, J1301 to J?, R1311 to R?, R1312 to R?
Connections:
- net CHASSIS: now reaches J?.6 (Shield)

Commit message: pulled footprints into layout
Parts:
- C?: Digi-Key PN 399-7845-1-ND -> 1276-1935-1-ND
- R? (x2): Digi-Key PN 311-27.0HRCT-ND -> (none)
Changed lines of the file:
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@@
       (effects (font (size 1.27 1.27)))
     )
-    (property "Digi-Key PN" "311-27.0HRCT-ND" (at 154.94 102.235 0)
+    (property "Digi-Key PN" "" (at 154.94 102.235 0)
       (effects (font (size 1.524 1.524)) hide)
     )
@@
       (effects (font (size 1.27 1.27)))
     )
-    (property "Digi-Key PN" "311-27.0HRCT-ND" (at 154.94 120.015 0)
+    (property "Digi-Key PN" "" (at 154.94 120.015 0)
       (effects (font (size 1.524 1.524)) hide)
     )
@@
       (effects (font (size 1.27 1.27)) (justify right))
     )
-    (property "Digi-Key PN" "399-7845-1-ND" (at 154.305 74.93 0)
-      (effects (font (size 1.524 1.524)) hide)
-    )
+    (property "Digi-Key PN" "1276-1935-1-ND" (at 154.305 74.93 0)
+      (effects (font (size 1.524 1.524)) hide)
+    )

Commit message: fixed footprints, assigned digikey pns
Parts:
- C? (x2): Digi-Key PN (none) -> 1292-1501-1-ND
- R? (x2): Digi-Key PN (none) -> 541-27.0HCT-ND
Changed lines of the file:
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@@
       (effects (font (size 1.27 1.27)))
     )
-    (property "Digi-Key PN" "" (at 154.94 102.235 0)
+    (property "Digi-Key PN" "541-27.0HCT-ND" (at 154.94 102.235 0)
       (effects (font (size 1.524 1.524)) hide)
     )
@@
       (effects (font (size 1.27 1.27)) (justify right))
     )
-    (property "Digi-Key PN" "" (at 129.54 120.65 0)
+    (property "Digi-Key PN" "1292-1501-1-ND" (at 129.54 120.65 0)
       (effects (font (size 1.27 1.27)) hide)
     )
@@
       (effects (font (size 1.27 1.27)))
     )
-    (property "Digi-Key PN" "" (at 154.94 120.015 0)
+    (property "Digi-Key PN" "541-27.0HCT-ND" (at 154.94 120.015 0)
       (effects (font (size 1.524 1.524)) hide)
     )
@@
       (effects (font (size 1.27 1.27)) (justify right))
     )
-    (property "Digi-Key PN" "" (at 151.13 120.65 0)
-      (effects (font (size 1.27 1.27)) hide)
-    )
+    (property "Digi-Key PN" "1292-1501-1-ND" (at 151.13 120.65 0)
+      (effects (font (size 1.27 1.27)) hide)
+    )

Commit message: fixed some netlist connectivity issues, finished grouping parts in PCB
Connections:
- net UFP_USB_CONN_USB+: no longer C?.1, U?.6 (D1)
- net UFP_USB_CONN_USB-: no longer C?.1, U?.5 (D2)
- net UFP_USB_D+: now also C?.1, U?.6 (D1)
- net UFP_USB_D-: now also C?.1, U?.5 (D2)
Other:
- moved on the sheet: C?, R?, TP?, U?
