File: hdw/USB_Hub/port_power_control.kicad_sch (KiCad schematic)
At the start: 12 parts

Commit message: lots of schematic progress
Parts:
- added R? (x8): 10, Resistors_SMD:R_0402, symbol Custom_Library:R_Custom
- added R? (x4): 0.02, Resistors_SMD:R_0612, symbol Custom_Library:R_Custom
Connections:
- net DFP0_VBUS: now also R?.2, R?.2; no longer U?.15 (OUT1)
- net DFP1_VBUS: now also R?.2, R?.2; no longer U?.14 (OUT2)
- net DFP2_VBUS: now also R?.2, R?.2; no longer U?.11 (OUT3)
- net DFP3_VBUS: now also R?.2, R?.2; no longer U?.10 (OUT4)
- new net: R?.1, R?.2, U?.10 (OUT4)
- new net: R?.1, R?.2, U?.14 (OUT2)
- new net: R?.1, R?.2, U?.11 (OUT3)
- new net: R?.1, R?.2, U?.15 (OUT1)
- new net DFP0_SNS+: R?.1
- new net DFP0_SNS-: R?.1
- new net DFP1_SNS+: R?.1
- new net DFP1_SNS-: R?.1
- new net DFP2_SNS+: R?.1
- new net DFP2_SNS-: R?.1
- new net DFP3_SNS+: R?.1
- new net DFP3_SNS-: R?.1
Other:
- company: (none) -> Drew Maatman
- title: (none) -> USB Hub
- moved on the sheet: C?, R?, U?A, U?B

Commit message: much more schematic progress
Other:
- moved on the sheet: C?
Changed lines of the file:
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@@
     )
   )
-  (symbol (lib_id "Custom_Library:C_Custom") (at 124.46 106.68 0) (unit 1)
-    (in_bom yes) (on_board yes) (dnp no)
-    (property "Reference" "C?" (at 125.095 104.14 0)
+  (symbol (lib_id "Custom_Library:C_Custom") (at 124.46 101.6 0) (unit 1)
+    (in_bom yes) (on_board yes) (dnp no)
+    (property "Reference" "C?" (at 125.095 99.06 0)
       (effects (font (size 1.27 1.27)) (justify left))
     )
-    (property "Value" "0.1uF" (at 125.095 109.22 0)
+    (property "Value" "0.1uF" (at 125.095 104.14 0)
       (effects (font (size 1.27 1.27)) (justify left))
     )
-    (property "Footprint" "Capacitors_SMD:C_0603" (at 125.4252 110.49 0)
-      (effects (font (size 1.27 1.27)) hide)
-    )
-    (property "Datasheet" "" (at 125.095 104.14 0)
-      (effects (font (size 1.27 1.27)) hide)
-    )
-    (property "display_footprint" "0603" (at 120.65 104.14 0)
+    (property "Footprint" "Capacitors_SMD:C_0603" (at 125.4252 105.41 0)
+      (effects (font (size 1.27 1.27)) hide)
+    )
+    (property "Datasheet" "" (at 125.095 99.06 0)
+      (effects (font (size 1.27 1.27)) hide)
+    )
+    (property "display_footprint" "0603" (at 120.65 99.06 0)
       (effects (font (size 1.27 1.27)) (justify right))
     )
-    (property "Voltage" "50V" (at 120.65 106.68 0)
+    (property "Voltage" "50V" (at 120.65 101.6 0)
       (effects (font (size 1.27 1.27)) (justify right))
     )
-    (property "Dielectric" "X7R" (at 120.65 109.22 0)
+    (property "Dielectric" "X7R" (at 120.65 104.14 0)
       (effects (font (size 1.27 1.27)) (justify right))
     )
-    (property "Digi-Key PN" "399-7845-1-ND" (at 135.255 93.98 0)
+    (property "Digi-Key PN" "399-7845-1-ND" (at 135.255 88.9 0)
       (effects (font (size 1.524 1.524)) hide)
     )
@@
     )
   )
-  (symbol (lib_id "power:+5V") (at 124.46 38.1 0) (unit 1)
-    (in_bom yes) (on_board yes) (dnp no)
-    (property "Reference" "#PWR01906" (at 124.46 41.91 0)
-      (effects (font (size 1.27 1.27)) hide)
-    )
-    (property "Value" "+5V" (at 124.46 34.544 0)
-      (effects (font (size 1.27 1.27)))
-    )
-    (property "Footprint" "" (at 124.46 38.1 0)
-      (effects (font (size 1.27 1.27)) hide)
-    )
-    (property "Datasheet" "" (at 124.46 38.1 0)
+  (symbol (lib_id "power:+5V") (at 124.46 33.02 0) (unit 1)
+    (in_bom yes) (on_board yes) (dnp no)
+    (property "Reference" "#PWR01906" (at 124.46 36.83 0)
+      (effects (font (size 1.27 1.27)) hide)
+    )
+    (property "Value" "+5V" (at 124.46 29.464 0)
+      (effects (font (size 1.27 1.27)))
+    )
+    (property "Footprint" "" (at 124.46 33.02 0)
+      (effects (font (size 1.27 1.27)) hide)
+    )
+    (property "Datasheet" "" (at 124.46 33.02 0)
       (effects (font (size 1.27 1.27)) hide)
     )
@@
     )
   )
-  (symbol (lib_id "power:+5V") (at 124.46 102.87 0) (unit 1)
-    (in_bom yes) (on_board yes) (dnp no)
-    (property "Reference" "#PWR01907" (at 124.46 106.68 0)
-      (effects (font (size 1.27 1.27)) hide)
-    )
-    (property "Value" "+5V" (at 124.46 99.314 0)
-      (effects (font (size 1.27 1.27)))
-    )
-    (property "Footprint" "" (at 124.46 102.87 0)
-      (effects (font (size 1.27 1.27)) hide)
-    )
-    (property "Datasheet" "" (at 124.46 102.87 0)
+  (symbol (lib_id "power:+5V") (at 124.46 97.79 0) (unit 1)
+    (in_bom yes) (on_board yes) (dnp no)
+    (property "Reference" "#PWR01907" (at 124.46 101.6 0)
+      (effects (font (size 1.27 1.27)) hide)
+    )
+    (property "Value" "+5V" (at 124.46 94.234 0)
+      (effects (font (size 1.27 1.27)))
+    )
+    (property "Footprint" "" (at 124.46 97.79 0)
+      (effects (font (size 1.27 1.27)) hide)
+    )
+    (property "Datasheet" "" (at 124.46 97.79 0)
       (effects (font (size 1.27 1.27)) hide)
     )
@@
     )
   )
-  (symbol (lib_id "power:GND") (at 124.46 45.72 0) (unit 1)
-    (in_bom yes) (on_board yes) (dnp no)
-    (property "Reference" "#PWR?" (at 124.46 52.07 0)
-      (effects (font (size 1.27 1.27)) hide)
-    )
-    (property "Value" "GND" (at 124.46 49.53 0)
-      (effects (font (size 1.27 1.27)))
-    )
-    (property "Footprint" "" (at 124.46 45.72 0)
-      (effects (font (size 1.27 1.27)) hide)
-    )
-    (property "Datasheet" "" (at 124.46 45.72 0)
+  (symbol (lib_id "power:GND") (at 124.46 40.64 0) (unit 1)
+    (in_bom yes) (on_board yes) (dnp no)
+    (property "Reference" "#PWR?" (at 124.46 46.99 0)
+      (effects (font (size 1.27 1.27)) hide)
+    )
+    (property "Value" "GND" (at 124.46 44.45 0)
+      (effects (font (size 1.27 1.27)))
+    )
+    (property "Footprint" "" (at 124.46 40.64 0)
+      (effects (font (size 1.27 1.27)) hide)
+    )
+    (property "Datasheet" "" (at 124.46 40.64 0)
       (effects (font (size 1.27 1.27)) hide)
     )
@@
     )
   )
-  (symbol (lib_id "Custom_Library:C_Custom") (at 124.46 41.91 0) (unit 1)
-    (in_bom yes) (on_board yes) (dnp no)
-    (property "Reference" "C?" (at 125.095 39.37 0)
+  (symbol (lib_id "Custom_Library:C_Custom") (at 124.46 36.83 0) (unit 1)
+    (in_bom yes) (on_board yes) (dnp no)
+    (property "Reference" "C?" (at 125.095 34.29 0)
       (effects (font (size 1.27 1.27)) (justify left))
     )
-    (property "Value" "0.1uF" (at 125.095 44.45 0)
+    (property "Value" "0.1uF" (at 125.095 39.37 0)
       (effects (font (size 1.27 1.27)) (justify left))
     )
-    (property "Footprint" "Capacitors_SMD:C_0603" (at 125.4252 45.72 0)
-      (effects (font (size 1.27 1.27)) hide)
-    )
-    (property "Datasheet" "" (at 125.095 39.37 0)
-      (effects (font (size 1.27 1.27)) hide)
-    )
-    (property "display_footprint" "0603" (at 120.65 39.37 0)
+    (property "Footprint" "Capacitors_SMD:C_0603" (at 125.4252 40.64 0)
+      (effects (font (size 1.27 1.27)) hide)
+    )
+    (property "Datasheet" "" (at 125.095 34.29 0)
+      (effects (font (size 1.27 1.27)) hide)
+    )
+    (property "display_footprint" "0603" (at 120.65 34.29 0)
       (effects (font (size 1.27 1.27)) (justify right))
     )
-    (property "Voltage" "50V" (at 120.65 41.91 0)
+    (property "Voltage" "50V" (at 120.65 36.83 0)
       (effects (font (size 1.27 1.27)) (justify right))
     )
-    (property "Dielectric" "X7R" (at 120.65 44.45 0)
+    (property "Dielectric" "X7R" (at 120.65 39.37 0)
       (effects (font (size 1.27 1.27)) (justify right))
     )
-    (property "Digi-Key PN" "399-7845-1-ND" (at 135.255 29.21 0)
+    (property "Digi-Key PN" "399-7845-1-ND" (at 135.255 24.13 0)
       (effects (font (size 1.524 1.524)) hide)
     )
@@
     )
   )
-  (symbol (lib_id "power:GND") (at 124.46 110.49 0) (unit 1)
-    (in_bom yes) (on_board yes) (dnp no)
-    (property "Reference" "#PWR?" (at 124.46 116.84 0)
-      (effects (font (size 1.27 1.27)) hide)
-    )
-    (property "Value" "GND" (at 124.46 114.3 0)
-      (effects (font (size 1.27 1.27)))
-    )
-    (property "Footprint" "" (at 124.46 110.49 0)
-      (effects (font (size 1.27 1.27)) hide)
-    )
-    (property "Datasheet" "" (at 124.46 110.49 0)
-      (effects (font (size 1.27 1.27)) hide)
-    )
+  (symbol (lib_id "power:GND") (at 124.46 105.41 0) (unit 1)
+    (in_bom yes) (on_board yes) (dnp no)
+    (property "Reference" "#PWR?" (at 124.46 111.76 0)
+      (effects (font (size 1.27 1.27)) hide)
+    )
+    (property "Value" "GND" (at 124.46 109.22 0)
+      (effects (font (size 1.27 1.27)))
+    )
+    (property "Footprint" "" (at 124.46 105.41 0)
+      (effects (font (size 1.27 1.27)) hide)
+    )
+    (property "Datasheet" "" (at 124.46 105.41 0)
+      (effects (font (size 1.27 1.27)) hide)
+    )

Commit message: lots and lots of sch progress
Parts:
- gave numbers to parts that had none: 1

Commit message: pulled footprints into layout
Parts:
- C? (x2): Digi-Key PN 399-7845-1-ND -> 1276-1935-1-ND
- R? (x8): Digi-Key PN PN -> (none)
- R? (x8): Digi-Key PN RMCF0402FT10R0CT-ND -> (none); Wattage 1/16W -> 1/10W; display_footprint 0402 -> 0603
Changed lines of the file:
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@@
       (effects (font (size 1.27 1.27)) (justify left) hide)
     )
-    (property "Digi-Key PN" "PN" (at 86.36 105.41 0)
+    (property "Digi-Key PN" "" (at 86.36 105.41 0)
       (effects (font (size 1.524 1.524)) hide)
     )
@@
       (effects (font (size 1.27 1.27)) (justify left) hide)
     )
-    (property "Digi-Key PN" "PN" (at 93.98 105.41 0)
+    (property "Digi-Key PN" "" (at 93.98 105.41 0)
       (effects (font (size 1.524 1.524)) hide)
     )
@@
       (effects (font (size 1.27 1.27)) (justify left) hide)
     )
-    (property "Digi-Key PN" "PN" (at 78.74 105.41 0)
+    (property "Digi-Key PN" "" (at 78.74 105.41 0)
       (effects (font (size 1.524 1.524)) hide)
     )
@@
       (effects (font (size 1.27 1.27)) (justify right))
     )
-    (property "Digi-Key PN" "399-7845-1-ND" (at 135.255 88.9 0)
+    (property "Digi-Key PN" "1276-1935-1-ND" (at 135.255 88.9 0)
       (effects (font (size 1.524 1.524)) hide)
     )
@@
       (effects (font (size 1.27 1.27)) hide)
     )
-    (property "display_footprint" "0402" (at 161.29 118.11 90)
+    (property "display_footprint" "0603" (at 161.29 118.11 90)
       (effects (font (size 1.27 1.27)) hide)
     )
@@
       (effects (font (size 1.27 1.27)) hide)
     )
-    (property "Wattage" "1/16W" (at 156.21 118.11 90)
-      (effects (font (size 1.27 1.27)) hide)
-    )
-    (property "Digi-Key PN" "RMCF0402FT10R0CT-ND" (at 163.83 118.11 0)
+    (property "Wattage" "1/10W" (at 156.21 118.11 90)
+      (effects (font (size 1.27 1.27)) hide)
+    )
+    (property "Digi-Key PN" "" (at 163.83 118.11 0)
       (effects (font (size 1.27 1.27)) hide)
     )
@@
       (effects (font (size 1.27 1.27)) (justify left) hide)
     )
-    (property "Digi-Key PN" "PN" (at 93.98 41.91 0)
+    (property "Digi-Key PN" "" (at 93.98 41.91 0)
       (effects (font (size 1.524 1.524)) hide)
     )
@@
       (effects (font (size 1.27 1.27)) (justify left) hide)
     )
-    (property "Digi-Key PN" "PN" (at 78.74 41.91 0)
+    (property "Digi-Key PN" "" (at 78.74 41.91 0)
       (effects (font (size 1.524 1.524)) hide)
     )
@@
       (effects (font (size 1.27 1.27)) hide)
     )
-    (property "display_footprint" "0402" (at 185.42 54.61 90)
+    (property "display_footprint" "0603" (at 185.42 54.61 90)
       (effects (font (size 1.27 1.27)) hide)
     )
@@
       (effects (font (size 1.27 1.27)) hide)
     )
-    (property "Wattage" "1/16W" (at 180.34 54.61 90)
-      (effects (font (size 1.27 1.27)) hide)
-    )
-    (property "Digi-Key PN" "RMCF0402FT10R0CT-ND" (at 187.96 54.61 0)
+    (property "Wattage" "1/10W" (at 180.34 54.61 90)
+      (effects (font (size 1.27 1.27)) hide)
+    )
+    (property "Digi-Key PN" "" (at 187.96 54.61 0)
       (effects (font (size 1.27 1.27)) hide)
     )
@@
       (effects (font (size 1.27 1.27)) hide)
     )
-    (property "display_footprint" "0402" (at 173.99 118.11 90)
+    (property "display_footprint" "0603" (at 173.99 118.11 90)
       (effects (font (size 1.27 1.27)) hide)
     )
@@
       (effects (font (size 1.27 1.27)) hide)
     )
-    (property "Wattage" "1/16W" (at 168.91 118.11 90)
-      (effects (font (size 1.27 1.27)) hide)
-    )
-    (property "Digi-Key PN" "RMCF0402FT10R0CT-ND" (at 176.53 118.11 0)
+    (property "Wattage" "1/10W" (at 168.91 118.11 90)
+      (effects (font (size 1.27 1.27)) hide)
+    )
+    (property "Digi-Key PN" "" (at 176.53 118.11 0)
       (effects (font (size 1.27 1.27)) hide)
     )
@@
       (effects (font (size 1.27 1.27)) hide)
     )
-    (property "display_footprint" "0402" (at 173.99 54.61 90)
+    (property "display_footprint" "0603" (at 173.99 54.61 90)
       (effects (font (size 1.27 1.27)) hide)
     )
@@
       (effects (font (size 1.27 1.27)) hide)
     )
-    (property "Wattage" "1/16W" (at 168.91 54.61 90)
-      (effects (font (size 1.27 1.27)) hide)
-    )
-    (property "Digi-Key PN" "RMCF0402FT10R0CT-ND" (at 176.53 54.61 0)
+    (property "Wattage" "1/10W" (at 168.91 54.61 90)
+      (effects (font (size 1.27 1.27)) hide)
+    )
+    (property "Digi-Key PN" "" (at 176.53 54.61 0)
       (effects (font (size 1.27 1.27)) hide)
     )
@@
       (effects (font (size 1.27 1.27)) (justify left) hide)
     )
-    (property "Digi-Key PN" "PN" (at 71.12 105.41 0)
+    (property "Digi-Key PN" "" (at 71.12 105.41 0)
       (effects (font (size 1.524 1.524)) hide)
     )
@@
       (effects (font (size 1.27 1.27)) hide)
     )
-    (property "display_footprint" "0402" (at 185.42 118.11 90)
+    (property "display_footprint" "0603" (at 185.42 118.11 90)
       (effects (font (size 1.27 1.27)) hide)
     )
@@
       (effects (font (size 1.27 1.27)) hide)
     )
-    (property "Wattage" "1/16W" (at 180.34 118.11 90)
-      (effects (font (size 1.27 1.27)) hide)
-    )
-    (property "Digi-Key PN" "RMCF0402FT10R0CT-ND" (at 187.96 118.11 0)
+    (property "Wattage" "1/10W" (at 180.34 118.11 90)
+      (effects (font (size 1.27 1.27)) hide)
+    )
+    (property "Digi-Key PN" "" (at 187.96 118.11 0)
       (effects (font (size 1.27 1.27)) hide)
     )
@@
       (effects (font (size 1.27 1.27)) hide)
     )
-    (property "display_footprint" "0402" (at 149.86 118.11 90)
+    (property "display_footprint" "0603" (at 149.86 118.11 90)
       (effects (font (size 1.27 1.27)) hide)
     )
@@
       (effects (font (size 1.27 1.27)) hide)
     )
-    (property "Wattage" "1/16W" (at 144.78 118.11 90)
-      (effects (font (size 1.27 1.27)) hide)
-    )
-    (property "Digi-Key PN" "RMCF0402FT10R0CT-ND" (at 152.4 118.11 0)
+    (property "Wattage" "1/10W" (at 144.78 118.11 90)
+      (effects (font (size 1.27 1.27)) hide)
+    )
+    (property "Digi-Key PN" "" (at 152.4 118.11 0)
       (effects (font (size 1.27 1.27)) hide)
     )
@@
       (effects (font (size 1.27 1.27)) hide)
     )
-    (property "display_footprint" "0402" (at 161.29 54.61 90)
+    (property "display_footprint" "0603" (at 161.29 54.61 90)
       (effects (font (size 1.27 1.27)) hide)
     )
@@
       (effects (font (size 1.27 1.27)) hide)
     )
-    (property "Wattage" "1/16W" (at 156.21 54.61 90)
-      (effects (font (size 1.27 1.27)) hide)
-    )
-    (property "Digi-Key PN" "RMCF0402FT10R0CT-ND" (at 163.83 54.61 0)
+    (property "Wattage" "1/10W" (at 156.21 54.61 90)
+      (effects (font (size 1.27 1.27)) hide)
+    )
+    (property "Digi-Key PN" "" (at 163.83 54.61 0)
       (effects (font (size 1.27 1.27)) hide)
     )
@@
       (effects (font (size 1.27 1.27)) (justify right))
     )
-    (property "Digi-Key PN" "399-7845-1-ND" (at 135.255 24.13 0)
+    (property "Digi-Key PN" "1276-1935-1-ND" (at 135.255 24.13 0)
       (effects (font (size 1.524 1.524)) hide)
     )
@@
       (effects (font (size 1.27 1.27)) (justify left) hide)
     )
-    (property "Digi-Key PN" "PN" (at 71.12 41.91 0)
+    (property "Digi-Key PN" "" (at 71.12 41.91 0)
       (effects (font (size 1.524 1.524)) hide)
     )
@@
       (effects (font (size 1.27 1.27)) (justify left) hide)
     )
-    (property "Digi-Key PN" "PN" (at 86.36 41.91 0)
+    (property "Digi-Key PN" "" (at 86.36 41.91 0)
       (effects (font (size 1.524 1.524)) hide)
     )
@@
       (effects (font (size 1.27 1.27)) hide)
     )
-    (property "display_footprint" "0402" (at 149.86 54.61 90)
+    (property "display_footprint" "0603" (at 149.86 54.61 90)
       (effects (font (size 1.27 1.27)) hide)
     )
@@
       (effects (font (size 1.27 1.27)) hide)
     )
-    (property "Wattage" "1/16W" (at 144.78 54.61 90)
-      (effects (font (size 1.27 1.27)) hide)
-    )
-    (property "Digi-Key PN" "RMCF0402FT10R0CT-ND" (at 152.4 54.61 0)
-      (effects (font (size 1.27 1.27)) hide)
-    )
+    (property "Wattage" "1/10W" (at 144.78 54.61 90)
+      (effects (font (size 1.27 1.27)) hide)
+    )
+    (property "Digi-Key PN" "" (at 152.4 54.61 0)
+      (effects (font (size 1.27 1.27)) hide)
+    )
