File: hdw/USB_Hub/USB_Hub.kicad_pcb (KiCad board)
At the start: 4 copper layers, 356 parts, among them J1101 USB_B_Mini, J1801 USB_A, J1901 USB_A, J2001 USB_A, J201 +12V IN, J2101 USB_A, J2201 USB_B_Mini, J2401 I2C, J2402 USB UART, J901 PICKIT4, Q401 BSS214NW, Q402 ZXMS6004FFTA, Q601 BSS214NW, Q602 ZXMS6004FFTA, Q901 BSS214NW, SW1601 Cap_Touch, SW1602 Cap_Touch, SW1603 Cap_Touch, SW901 MRST, U1001 PIC18(L)F47K40T-I_PT, U1101 TLV6700, U1102 FT234XD, U1103 TXB0102DCU, U1104 TPD3S014DBVR, U1201 74LVC1G97, U1202 74LVC1G97, U1203 74LVC1G97, U1204 74LVC1G97, U1205 74LVC1G97, U1301 74LVC1G97, U1302 74LVC1G97, U1303 74LVC1G97, U1401 74LVC1G97, U1402 74LVC1G97, U1403 74LVC1G97, U1404 74LVC1G97, U1405 74LVC1G97, U1406 74LVC1G97, U1407 74LVC1G97, U1408 74LVC1G97, U1409 74LVC1G97, U1501 SSD1306, U1502 DS1683, U1601 AT42QT1010-TSHR, U1602 AT42QT1010-TSHR, U1603 AT42QT1010-TSHR, U1701 74LVC1G97, U1702 TPS3808G33, U1703 M93C46-WMN6TP, U1704 74LVC1G97, U1705 TUSB2046BIRHBT, U201 TPS26600RHFT, U2201 TPD3S044DBVR, U2301 TPS2044D, U2401 INA219BxDCN, U2402 INA219BxDCN, U2403 MCP9804, U2404 INA219BxDCN, U2405 INA219BxDCN, U301 INA219BxDCN, U302 MCP9804, U401 74LVC1G97, U402 TPS62133, U501 INA219BxDCN, U502 MCP9804, U601 74LVC1G97, U602 TPS62132, U701 INA219BxDCN, U702 MCP9804, U801 TPS2121RUXR, X1701 ASE-48.000MHz

Commit message: random stuff
Parts:
- C1201, C1202, C1203, C1204, C1205, C1301, C1401, C1402, C1403, C1404, C1405, C1406, C1407, C1408, C1409, D201, R1001, R1401, R1402, R201, R202, R203, R205, R209, R210: moved to B.Cu
- moved C1302 241.9 mm to (444.3, 133.2)
- moved C1303 241.9 mm to (444.3, 135.6)
- moved D1302 241.9 mm to (444.4, 140.3)
- moved D1303 241.9 mm to (444.4, 142.6)
- moved R1301 241.9 mm to (436.4, 131.0)
- moved R1302 241.9 mm to (436.4, 133.4)
- moved R1304 241.9 mm to (436.4, 138.4)
- moved R1305 241.9 mm to (436.4, 140.9)
- moved R1306 241.9 mm to (436.4, 143.4)
- moved U1302 241.9 mm to (440.3, 135.5)
- moved U1303 241.9 mm to (440.3, 139.3)
- moved R1303 233.1 mm to (427.6, 134.2)
- moved U1301 226.1 mm to (424.2, 134.9)
- moved D1301 225.0 mm to (427.6, 135.6)
- moved C1301 222.1 mm to (424.2, 134.9), turned to 180 degrees
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Other:
- board text added: "+12V"
- board text added: "+12Vin"

Commit message: big restructuring, removed microcontroller and all telemtry
Parts:
- removed C1001, C1002, C1101, C1102, C1104, C1105, C1106, C1108, C1110, C1201, C1202, C1203, C1204, C1205, C1301, C1302, C1303, C1401, C1402, C1403, C1404, C1405, C1406, C1407, C1408, C1409, C1504, C1505, C1601, C1602, C1603, C1607, C1608, C1609, C1701, C1702, C1703, C1704, C1705, C1707, C1708, C1709, C202, C2203, C2301, C2302, C2401, C2402, C2403, C2404, C2405, C2406, C2407, C2408, C2409, C301, C302, C303, C401, C405, C501, C502, C503, C601, C605, C701, C702, C703, C801, C802, C803, C804, C901, C902: 0.1uF, Capacitors_SMD:C_0603
- removed C1103, C1501, C1502, C1503, C1506, C1706, C1710, C403, C603: 10uF, Capacitors_SMD:C_0603
- removed C1107, C1109: 47pF, Capacitors_SMD:C_0603
- removed C1604, C1605, C1606, C201, C404, C604: 10nF, Capacitors_SMD:C_0603
- removed C1801, C1802, C1901, C1902, C2001, C2002, C2101, C2102, C2201, C2202: 22pF, Capacitors_SMD:C_0603
- removed C1803, C1903, C2003, C203, C2103: 100uF, Capacitor_Tantalum_SMD:CP_EIA-7343-43_Kemet-X
- removed C402, C406, C407, C602, C606, C607: 10uF, Capacitors_SMD:C_1206
- removed D1101: Yellow, LEDs:LED_0603
- removed D1201, D1202, D1203, D1204, D1205, D1301, D1401, D1402, D1403, D1404: Green, LEDs:LED_0603
- removed D1302, D1303, D1405, D1406, D1407, D1408: Red, LEDs:LED_0603
- removed D1501, D401, D601: BAT48JFILM, Diode_SMD:D_SOD-323
- removed D1801, D1901, D2001, D2101, D901: SP0503BAHT, Package_TO_SOT_SMD:SOT-143
- removed D201: 24V, Diodes_SMD:D_SMA
- removed H2501, H2502, H2503, H2504: 3mm Mounting Hole, MountingHole:MountingHole_3mm
- removed J1101, J2201: USB_B_Mini, Connectors:USB_Mini-B
- removed J1801, J1901, J2001, J2101: USB_A, Connector_USB:USB_A_Molex_67643_Horizontal
- removed J201: +12V IN, Connectors:BARREL_JACK
- removed J2401: I2C, Connector_PinHeader_2.54mm:PinHeader_1x03_P2.54mm_Vertical
- removed J2402: USB UART, Connector_PinHeader_2.54mm:PinHeader_1x03_P2.54mm_Vertical
- removed J901: PICKIT4, Custom Footprints Library:PICKIT4_Header
- removed L1101, L901, L902: 600R 0.5A, Inductors_SMD:L_0603
- removed L1701: 600R 0.5A, Inductors_SMD:L_0402
- removed L401, L601: 2.2uH, Inductors_SMD:L_Vishay_IHLP-2020
- removed Q401, Q601, Q901: BSS214NW, Package_TO_SOT_SMD:SOT-323_SC-70
- removed Q402, Q602: ZXMS6004FFTA, Package_TO_SOT_SMD:SOT-23
- removed R1001, R1002, R1003, R1105, R1301, R1302, R1305, R1401, R1402, R204, R207, R211, R2301, R2302, R2303, R2304, R2305, R2306, R2307, R2308, R2401, R2403, R801, R810, R902, R904: 10k, Resistors_SMD:R_0603
- removed R1101, R1201, R1202, R1203, R1204, R1205, R1303, R1304, R1306, R1403, R1404, R1405, R1406, R1407, R1408, R1409, R1410, R1702, R905: 1k, Resistors_SMD:R_0603
- removed R1102: 487k, Resistors_SMD:R_0603
- removed R1103: 6.04k, Resistors_SMD:R_0603
- removed R1104: 40.2k, Resistors_SMD:R_0603
- removed R1106, R1107, R1110, R1111: 100k, Resistors_SMD:R_0603
- removed R1108, R1109, R1801, R1802, R1901, R1902, R2001, R2002, R2101, R2102, R2201, R2202: 27, Resistors_SMD:R_0603
- removed R1601, R1602, R1603: 499, Resistors_SMD:R_0603
- removed R1604, R1605, R1606, R1703, R1704, R1705, R1706, R1707, R404, R405, R601, R602, R603, R604: 10k, Resistors_SMD:R_0402
- removed R1701, R2309, R2310, R2313, R2314, R2315, R2316, R2319, R2320, R606, R608, R809, R812: 10, Resistors_SMD:R_0402
- removed R201: 51.1k, Resistors_SMD:R_0603
- removed R202: 1.15k, Resistors_SMD:R_0603
- removed R203, R209: 5.11k, Resistors_SMD:R_0603
- removed R205, R210, R2402, R2404, R901, R903: 10, Resistors_SMD:R_0603
- removed R206, R2311, R2312, R2317, R2318, R607, R811: 0.02, Resistors_SMD:R_0612
- removed R208: 13k, Resistors_SMD:R_0603
- removed R401: 2.67k, Resistors_SMD:R_0603
- removed R402, R406, R605: 0, Resistors_SMD:R_0402
- removed R403: 1.37k, Resistors_SMD:R_0603
- removed R407: 953k, Resistors_SMD:R_0402
- removed R408: 180k, Resistors_SMD:R_0402
- removed R609: 1.21M, Resistors_SMD:R_0603
- removed R610: 383k, Resistors_SMD:R_0603
- removed R802, R804, R806, R808: 4.99k, Resistors_SMD:R_0603
- removed R803, R813: 18.7k, Resistors_SMD:R_0603
- removed R805, R807: 23.7k, Resistors_SMD:R_0603
- removed SW1601, SW1602, SW1603: Cap_Touch, Custom Footprints Library:Capacitive_Touch_Pad
- removed SW901: MRST, Button_Switch_THT:SW_PUSH_6mm
- removed TP1001, TP1101, TP202, TP203, TP2201, TP401, TP601: TP, Custom Footprints Library:Test_Point
- removed TP201: TP, Connector_PinHeader_2.54mm:PinHeader_1x01_P2.54mm_Horizontal
- removed U1001: PIC18(L)F47K40T-I_PT, Housings_QFP:TQFP-44_10x10mm_Pitch0.8mm
- removed U1101: TLV6700, Package_TO_SOT_SMD:SOT-23-6
- removed U1102: FT234XD, Housings_DFN_QFN:DFN-12-1EP_3x3mm_Pitch0.45mm
- removed U1103: TXB0102DCU, Package_SO:VSSOP-8_2.4x2.1mm_P0.5mm
- removed U1104: TPD3S014DBVR, TO_SOT_Packages_SMD:SOT-23-6
- removed U1201, U1202, U1203, U1204, U1205, U1301, U1302, U1303, U1401, U1402, U1403, U1404, U1405, U1406, U1407, U1408, U1409, U1701, U1704, U401, U601: 74LVC1G97, Package_TO_SOT_SMD:SOT-363_SC-70-6
- removed U1501: SSD1306, Connector_PinSocket_2.54mm:PinSocket_1x04_P2.54mm_Vertical
- removed U1502: DS1683, Housings_SOIC:SOIC-8_3.9x4.9mm_Pitch1.27mm
- removed U1601, U1602, U1603: AT42QT1010-TSHR, TO_SOT_Packages_SMD:SOT-23-6
- removed U1702: TPS3808G33, Package_TO_SOT_SMD:SOT-23-6
- removed U1703: M93C46-WMN6TP, Package_SO:SOIC-8_3.9x4.9mm_P1.27mm
- removed U1705: TUSB2046BIRHBT, Package_DFN_QFN:VQFN-32-1EP_5x5mm_P0.5mm_EP3.5x3.5mm
- removed U201: TPS26600RHFT, Housings_DFN_QFN:QFN-24-1EP_4x5mm_Pitch0.5mm
- removed U2201: TPD3S044DBVR, TO_SOT_Packages_SMD:SOT-23-6
- removed U2301: TPS2044D, Package_SO:SOIC-16_3.9x9.9mm_P1.27mm
- removed U2401, U2402, U2404, U2405, U301, U501, U701: INA219BxDCN, Package_TO_SOT_SMD:SOT-23-8
- removed U2403, U302, U502, U702: MCP9804, Package_DFN_QFN:DFN-8-1EP_3x2mm_P0.5mm_EP1.3x1.5mm
- removed U402: TPS62133, Package_DFN_QFN:QFN-16-1EP_3x3mm_P0.5mm_EP1.75x1.75mm
- removed U602: TPS62132, Package_DFN_QFN:QFN-16-1EP_3x3mm_P0.5mm_EP1.75x1.75mm
- removed U801: TPS2121RUXR, Custom Footprints Library:12-VQFN-HR_2x2p5
- removed X1701: ASE-48.000MHz, Oscillator:Oscillator_SMD_Abracon_ASE-4Pin_3.2x2.5mm
Other:
- board text removed: "+12V"
- board text removed: "+12Vin"

Commit message: pulled in fotprints into layout
Parts:
- added C1001: 22pF, Capacitors_SMD:C_0603, F.Cu at (428.0, 110.0)
- added C1002: 22pF, Capacitors_SMD:C_0603, F.Cu at (428.0, 112.3)
- added C1003: 100uF, Capacitor_Tantalum_SMD:CP_EIA-7343-43_Kemet-X, F.Cu at (417.6, 111.7)
- added C1101: 22pF, Capacitors_SMD:C_0603, F.Cu at (428.0, 127.5)
- added C1102: 22pF, Capacitors_SMD:C_0603, F.Cu at (428.0, 129.8)
- added C1103: 100uF, Capacitor_Tantalum_SMD:CP_EIA-7343-43_Kemet-X, F.Cu at (417.6, 129.2)
- added C1201: 22pF, Capacitors_SMD:C_0603, F.Cu at (451.7, 110.0)
- added C1202: 22pF, Capacitors_SMD:C_0603, F.Cu at (451.7, 112.3)
- added C1203: 100uF, Capacitor_Tantalum_SMD:CP_EIA-7343-43_Kemet-X, F.Cu at (441.3, 111.7)
- added C1301: 22pF, Capacitors_SMD:C_0603, F.Cu at (451.7, 127.5)
- added C1302: 22pF, Capacitors_SMD:C_0603, F.Cu at (451.7, 129.8)
- added C1303: 100uF, Capacitor_Tantalum_SMD:CP_EIA-7343-43_Kemet-X, F.Cu at (441.3, 129.2)
- added C1401: 22pF, Capacitors_SMD:C_0603, F.Cu at (420.6, 49.2)
- added C1402: 22pF, Capacitors_SMD:C_0603, F.Cu at (420.6, 51.5)
- added C1403: 0.1uF, Capacitors_SMD:C_0603, F.Cu at (420.6, 53.9)
- added C1501: 0.1uF, Capacitors_SMD:C_0603, F.Cu at (431.0, 58.5)
- added C1502: 0.1uF, Capacitors_SMD:C_0603, F.Cu at (431.0, 60.8)
- added C201: 10nF, Capacitors_SMD:C_0603, F.Cu at (403.4, 49.2)
- added C202: 0.1uF, Capacitors_SMD:C_0603, F.Cu at (403.4, 51.5)
- added C203: 100uF, Capacitor_Tantalum_SMD:CP_EIA-7343-43_Kemet-X, F.Cu at (389.4, 68.1)
- added C301: 0.1uF, Capacitors_SMD:C_0603, F.Cu at (438.8, 75.3)
- added C302: 10uF, Capacitors_SMD:C_1206, F.Cu at (434.1, 75.7)
- added C303: 10uF, Capacitors_SMD:C_0603, F.Cu at (438.8, 77.7)
- added C304: 10nF, Capacitors_SMD:C_0603, F.Cu at (438.8, 80.0)
- added C305: 0.1uF, Capacitors_SMD:C_0603, F.Cu at (438.8, 82.4)
- added C306: 10uF, Capacitors_SMD:C_1206, F.Cu at (434.1, 78.9)
- added C307: 10uF, Capacitors_SMD:C_1206, F.Cu at (434.1, 82.0)
- added C401: 10uF, Capacitors_SMD:C_0603, F.Cu at (449.0, 79.4)
- added C402: 0.1uF, Capacitors_SMD:C_0603, F.Cu at (449.0, 81.7)
- added C403: 10uF, Capacitors_SMD:C_0603, F.Cu at (449.0, 84.1)
- added C404: 10uF, Capacitors_SMD:C_0603, F.Cu at (449.0, 86.4)
- added C501: 0.1uF, Capacitors_SMD:C_0603, F.Cu at (446.7, 49.2)
- added C502: 0.1uF, Capacitors_SMD:C_0603, F.Cu at (446.7, 51.5)
- added C503: 0.1uF, Capacitors_SMD:C_0603, F.Cu at (446.7, 53.9)
- added C504: 0.1uF, Capacitors_SMD:C_0603, F.Cu at (446.7, 56.2)
- added C601: 0.1uF, Capacitors_SMD:C_0603, F.Cu at (390.6, 103.8)
- added C602: 0.1uF, Capacitors_SMD:C_0603, F.Cu at (390.6, 106.2)
- added C603: 0.1uF, Capacitors_SMD:C_0603, F.Cu at (390.6, 108.5)
- added C604: 0.1uF, Capacitors_SMD:C_0603, F.Cu at (390.6, 110.9)
- added C605: 0.1uF, Capacitors_SMD:C_0603, F.Cu at (390.6, 113.2)
- added C701: 0.1uF, Capacitors_SMD:C_0603, F.Cu at (395.3, 75.3)
- added C702: 0.1uF, Capacitors_SMD:C_0603, F.Cu at (395.3, 77.7)
- added C703: 0.1uF, Capacitors_SMD:C_0603, F.Cu at (395.3, 80.0)
- added C704: 0.1uF, Capacitors_SMD:C_0603, F.Cu at (395.3, 82.4)
- added C705: 0.1uF, Capacitors_SMD:C_0603, F.Cu at (395.3, 84.7)
- added C706: 0.1uF, Capacitors_SMD:C_0603, F.Cu at (395.3, 87.1)
- added C707: 0.1uF, Capacitors_SMD:C_0603, F.Cu at (399.1, 75.3)
- added C708: 0.1uF, Capacitors_SMD:C_0603, F.Cu at (399.1, 77.7)
- added C709: 0.1uF, Capacitors_SMD:C_0603, F.Cu at (399.1, 80.0)
- added C710: 0.1uF, Capacitors_SMD:C_0603, F.Cu at (399.1, 82.4)
- added C901: 0.1uF, Capacitors_SMD:C_0603, F.Cu at (408.5, 75.3)
- added C902: 0.1uF, Capacitors_SMD:C_0603, F.Cu at (408.5, 77.7)
- added C903: 0.1uF, Capacitors_SMD:C_0603, F.Cu at (408.5, 80.0)
- added C904: 0.1uF, Capacitors_SMD:C_0603, F.Cu at (408.5, 82.4)
- added C905: 0.1uF, Capacitors_SMD:C_0603, F.Cu at (408.5, 84.7)
- added C906: 10uF, Capacitors_SMD:C_0603, F.Cu at (408.5, 87.1)
- added C907: 0.1uF, Capacitors_SMD:C_0603, F.Cu at (412.4, 75.3)
- added C908: 0.1uF, Capacitors_SMD:C_0603, F.Cu at (412.4, 77.7)
- added C909: 0.1uF, Capacitors_SMD:C_0603, F.Cu at (412.4, 80.0)
- added C910: 10uF, Capacitors_SMD:C_0603, F.Cu at (412.4, 82.4)
- added D1001: SP0503BAHT, Package_TO_SOT_SMD:SOT-143, F.Cu at (432.0, 111.0)
- added D1101: SP0503BAHT, Package_TO_SOT_SMD:SOT-143, F.Cu at (432.0, 128.5)
- added D1201: SP0503BAHT, Package_TO_SOT_SMD:SOT-143, F.Cu at (455.7, 111.0)
- added D1301: SP0503BAHT, Package_TO_SOT_SMD:SOT-143, F.Cu at (455.7, 128.5)
- added D201: 24V, Diodes_SMD:D_SMA, F.Cu at (401.9, 62.8)
- added D301: BAT48JFILM, Diode_SMD:D_SOD-323, F.Cu at (442.9, 75.6)
- added D601: Green, LEDs:LED_0603, F.Cu at (394.5, 103.8)
- added D602: Green, LEDs:LED_0603, F.Cu at (394.5, 106.2)
- added D603: Green, LEDs:LED_0603, F.Cu at (394.5, 108.5)
- added D604: Green, LEDs:LED_0603, F.Cu at (394.5, 110.9)
- added D605: Green, LEDs:LED_0603, F.Cu at (394.5, 113.2)
- added D701: Green, LEDs:LED_0603, F.Cu at (382.9, 75.3)
- added D702: Green, LEDs:LED_0603, F.Cu at (382.9, 77.7)
- added D703: Green, LEDs:LED_0603, F.Cu at (382.9, 80.0)
- added D704: Green, LEDs:LED_0603, F.Cu at (382.9, 82.4)
- added D705: Red, LEDs:LED_0603, F.Cu at (382.9, 84.7)
- added D706: Red, LEDs:LED_0603, F.Cu at (382.9, 87.1)
- added D707: Red, LEDs:LED_0603, F.Cu at (382.9, 89.4)
- added D708: Red, LEDs:LED_0603, F.Cu at (382.9, 91.8)
- added D709: Red, LEDs:LED_0603, F.Cu at (382.9, 94.1)
- added D710: Green, LEDs:LED_0603, F.Cu at (382.9, 96.5)
- added H801: 3mm Mounting Hole, MountingHole:MountingHole_3mm, F.Cu at (406.8, 102.9)
- added H802: 3mm Mounting Hole, MountingHole:MountingHole_3mm, F.Cu at (406.8, 110.5)
- added H803: 3mm Mounting Hole, MountingHole:MountingHole_3mm, F.Cu at (406.8, 118.0)
- added H804: 3mm Mounting Hole, MountingHole:MountingHole_3mm, F.Cu at (406.8, 125.6)
- added J1001: USB_A, Connector_USB:USB_A_Wuerth_614004134726_Horizontal, F.Cu at (426.0, 104.0)
- added J1101: USB_A, Connector_USB:USB_A_Wuerth_614004134726_Horizontal, F.Cu at (426.0, 121.5)
- added J1201: USB_A, Connector_USB:USB_A_Wuerth_614004134726_Horizontal, F.Cu at (449.7, 104.0)
- added J1301: USB_A, Connector_USB:USB_A_Wuerth_614004134726_Horizontal, F.Cu at (449.7, 121.5)
- added J1401: USB_B_Mini, Connectors:USB_Mini-B, F.Cu at (413.9, 54.2)
- added J201: +12V IN, Connectors:BARREL_JACK, F.Cu at (399.0, 53.3)
- added L301: 2.2uH, Inductors_SMD:L_Vishay_IHLP-2020, F.Cu at (435.5, 86.9)
- added L901: 600R 0.5A, Inductors_SMD:L_0402, F.Cu at (424.2, 83.9)
- added Q301: BSS214NW, Package_TO_SOT_SMD:SOT-323_SC-70, F.Cu at (433.6, 92.1)
- added Q302: ZXMS6004FFTA, Package_TO_SOT_SMD:SOT-23, F.Cu at (442.1, 91.1)
- added R1001: 27, Resistors_SMD:R_0603, F.Cu at (424.3, 110.0)
- added R1002: 27, Resistors_SMD:R_0603, F.Cu at (424.3, 112.5)
- added R1101: 27, Resistors_SMD:R_0603, F.Cu at (424.3, 127.5)
- added R1102: 27, Resistors_SMD:R_0603, F.Cu at (424.3, 130.0)
- added R1201: 27, Resistors_SMD:R_0603, F.Cu at (448.0, 110.0)
- added R1202: 27, Resistors_SMD:R_0603, F.Cu at (448.0, 112.5)
- added R1301: 27, Resistors_SMD:R_0603, F.Cu at (448.0, 127.5)
- added R1302: 27, Resistors_SMD:R_0603, F.Cu at (448.0, 130.0)
- added R1401: 27, Resistors_SMD:R_0603, F.Cu at (420.4, 56.3)
- added R1402: 27, Resistors_SMD:R_0603, F.Cu at (420.4, 58.8)
- added R1501: 10k, Resistors_SMD:R_0603, F.Cu at (427.3, 49.2)
- added R1502: 10k, Resistors_SMD:R_0603, F.Cu at (427.3, 51.7)
- added R1503: 10k, Resistors_SMD:R_0603, F.Cu at (427.3, 54.2)
- added R1504: 10k, Resistors_SMD:R_0603, F.Cu at (427.3, 56.7)
- added R1505: 10k, Resistors_SMD:R_0603, F.Cu at (427.3, 59.1)
- added R1506: 10k, Resistors_SMD:R_0603, F.Cu at (427.3, 61.6)
- added R1507: 10k, Resistors_SMD:R_0603, F.Cu at (427.3, 64.1)
- added R1508: 10k, Resistors_SMD:R_0603, F.Cu at (427.3, 66.6)
- added R201: 51.1k, Resistors_SMD:R_0603, F.Cu at (382.7, 49.2)
- added R202: 1.15k, Resistors_SMD:R_0603, F.Cu at (382.7, 51.7)
- added R203: 5.11k, Resistors_SMD:R_0603, F.Cu at (382.7, 54.2)
- added R204: 10k, Resistors_SMD:R_0603, F.Cu at (382.7, 56.7)
- added R205: 10k, Resistors_SMD:R_0603, F.Cu at (382.7, 59.1)
- added R206: 13k, Resistors_SMD:R_0603, F.Cu at (382.7, 61.6)
- added R207: 5.11k, Resistors_SMD:R_0603, F.Cu at (382.7, 64.1)
- added R208: 10k, Resistors_SMD:R_0603, F.Cu at (382.7, 66.6)
- added R301: 2.67k, Resistors_SMD:R_0603, F.Cu at (429.6, 75.4)
- added R302: 10, Resistors_SMD:R_0603, F.Cu at (429.6, 77.9)
- added R303: 1.37k, Resistors_SMD:R_0603, F.Cu at (429.6, 80.3)
- added R304: 10k, Resistors_SMD:R_0603, F.Cu at (429.6, 82.8)
- added R305: 10k, Resistors_SMD:R_0603, F.Cu at (429.6, 85.3)
- added R306: 10, Resistors_SMD:R_0603, F.Cu at (429.6, 87.8)
- added R307: 953k, Resistors_SMD:R_0603, F.Cu at (429.6, 90.3)
- added R308: 180k, Resistors_SMD:R_0603, F.Cu at (429.6, 92.7)
- added R401: 10k, Resistors_SMD:R_0603, F.Cu at (452.7, 79.4)
- added R402: 10k, Resistors_SMD:R_0603, F.Cu at (452.7, 81.9)
- added R403: 3.57k, Resistors_SMD:R_0603, F.Cu at (452.7, 84.4)
- added R404: 1.15k, Resistors_SMD:R_0603, F.Cu at (452.7, 86.9)
- added R501: 10k, Resistors_SMD:R_0603, F.Cu at (439.5, 49.2)
- added R502: 4.99k, Resistors_SMD:R_0603, F.Cu at (439.5, 51.7)
- added R503: 18.7k, Resistors_SMD:R_0603, F.Cu at (439.5, 54.2)
- added R504: 4.99k, Resistors_SMD:R_0603, F.Cu at (439.5, 56.7)
- added R505: 23.7k, Resistors_SMD:R_0603, F.Cu at (439.5, 59.1)
- added R506: 4.99k, Resistors_SMD:R_0603, F.Cu at (443.0, 49.2)
- added R507: 23.7k, Resistors_SMD:R_0603, F.Cu at (443.0, 51.7)
- added R508: 4.99k, Resistors_SMD:R_0603, F.Cu at (443.0, 54.2)
- added R509: 10k, Resistors_SMD:R_0603, F.Cu at (443.0, 56.7)
- added R510: 18.7k, Resistors_SMD:R_0603, F.Cu at (443.0, 59.1)
- added R601: 1k, Resistors_SMD:R_0603, F.Cu at (386.9, 103.9)
- added R602: 1k, Resistors_SMD:R_0603, F.Cu at (386.9, 106.4)
- added R603: 1k, Resistors_SMD:R_0603, F.Cu at (386.9, 108.8)
- added R604: 1k, Resistors_SMD:R_0603, F.Cu at (386.9, 111.3)
- added R605: 10k, Resistors_SMD:R_0603, F.Cu at (386.9, 113.8)
- added R606: 1k, Resistors_SMD:R_0603, F.Cu at (386.9, 116.3)
- added R701: 1k, Resistors_SMD:R_0603, F.Cu at (395.1, 89.5)
- added R702: 1k, Resistors_SMD:R_0603, F.Cu at (395.1, 92.0)
- added R703: 1k, Resistors_SMD:R_0603, F.Cu at (395.1, 94.4)
- added R704: 1k, Resistors_SMD:R_0603, F.Cu at (395.1, 96.9)
- added R705: 1k, Resistors_SMD:R_0603, F.Cu at (395.1, 99.4)
- added R706: 1k, Resistors_SMD:R_0603, F.Cu at (398.7, 89.5)
- added R707: 1k, Resistors_SMD:R_0603, F.Cu at (398.7, 92.0)
- added R708: 1k, Resistors_SMD:R_0603, F.Cu at (398.7, 94.4)
- added R709: 1k, Resistors_SMD:R_0603, F.Cu at (398.7, 96.9)
- added R710: 1k, Resistors_SMD:R_0603, F.Cu at (398.7, 99.4)
- added R901: 10, Resistors_SMD:R_0603, F.Cu at (404.8, 75.4)
- added R902: 1k, Resistors_SMD:R_0603, F.Cu at (404.8, 77.9)
- added R903: 10k, Resistors_SMD:R_0603, F.Cu at (404.8, 80.3)
- added R904: 10k, Resistors_SMD:R_0603, F.Cu at (404.8, 82.8)
- added R905: 10k, Resistors_SMD:R_0603, F.Cu at (404.8, 85.3)
- added R906: 10k, Resistors_SMD:R_0603, F.Cu at (404.8, 87.8)
- added R907: 10k, Resistors_SMD:R_0603, F.Cu at (404.8, 90.3)
- added SW901: RESET, Button_Switch_THT:SW_PUSH_6mm, F.Cu at (416.3, 76.2)
- added TP1401: TP, Custom Footprints Library:Test_Point, F.Cu at (409.5, 62.0)
- added TP201: TP, Connector_PinHeader_2.54mm:PinHeader_1x01_P2.54mm_Horizontal, F.Cu at (386.8, 62.9)
- added TP202: TP, Custom Footprints Library:Test_Point, F.Cu at (395.9, 66.8)
- added TP203: TP, Custom Footprints Library:Test_Point, F.Cu at (395.9, 70.0)
- added TP301: TP, Custom Footprints Library:Test_Point, F.Cu at (437.4, 91.9)
- added TP401: TP, Custom Footprints Library:Test_Point, F.Cu at (453.4, 75.7)
- added U1401: TPD3S044DBVR, TO_SOT_Packages_SMD:SOT-23-6, F.Cu at (421.1, 62.3)
- added U1501: TPS2042BDGN, Housings_SSOP:MSOP-8-1EP_3x3mm_Pitch0.65mm, F.Cu at (432.4, 50.3)
- added U1502: TPS2042BDGN, Housings_SSOP:MSOP-8-1EP_3x3mm_Pitch0.65mm, F.Cu at (432.4, 55.0)
- added U201: TPS26600RHFT, Housings_DFN_QFN:QFN-24-1EP_4x5mm_Pitch0.5mm, F.Cu at (400.9, 68.6)
- added U301: 74LVC1G97, Package_TO_SOT_SMD:SOT-363_SC-70-6, F.Cu at (442.9, 79.0)
- added U302: TPS62133, Package_DFN_QFN:QFN-16-1EP_3x3mm_P0.5mm_EP1.75x1.75mm, F.Cu at (442.3, 86.2)
- added U401: TPS7A92, Package_DFN_QFN:Texas_S-PDSO-N10_EP1.2x2mm, F.Cu at (449.4, 76.2)
- added U501: TPS2121RUXR, Custom Footprints Library:12-VQFN-HR_2x2p5, F.Cu at (446.5, 59.3)
- added U601: 74LVC1G97, Package_TO_SOT_SMD:SOT-363_SC-70-6, F.Cu at (383.0, 104.6)
- added U602: 74LVC1G97, Package_TO_SOT_SMD:SOT-363_SC-70-6, F.Cu at (383.0, 108.4)
- added U603: 74LVC1G97, Package_TO_SOT_SMD:SOT-363_SC-70-6, F.Cu at (383.0, 112.3)
- added U604: 74LVC1G97, Package_TO_SOT_SMD:SOT-363_SC-70-6, F.Cu at (383.0, 116.1)
- added U605: 74LVC1G97, Package_TO_SOT_SMD:SOT-363_SC-70-6, F.Cu at (383.0, 120.0)
- added U701: 74LVC1G97, Package_TO_SOT_SMD:SOT-363_SC-70-6, F.Cu at (387.0, 76.1)
- added U702: 74LVC1G97, Package_TO_SOT_SMD:SOT-363_SC-70-6, F.Cu at (387.0, 79.9)
- added U703: 74LVC1G97, Package_TO_SOT_SMD:SOT-363_SC-70-6, F.Cu at (387.0, 83.8)
- added U704: 74LVC1G97, Package_TO_SOT_SMD:SOT-363_SC-70-6, F.Cu at (387.0, 87.6)
- added U705: 74LVC1G97, Package_TO_SOT_SMD:SOT-363_SC-70-6, F.Cu at (387.0, 91.5)
- added U706: 74LVC1G97, Package_TO_SOT_SMD:SOT-363_SC-70-6, F.Cu at (391.2, 76.1)
- added U707: 74LVC1G97, Package_TO_SOT_SMD:SOT-363_SC-70-6, F.Cu at (391.2, 79.9)
- added U708: 74LVC1G97, Package_TO_SOT_SMD:SOT-363_SC-70-6, F.Cu at (391.2, 83.8)
- added U709: 74LVC1G97, Package_TO_SOT_SMD:SOT-363_SC-70-6, F.Cu at (391.2, 87.6)
- added U710: 74LVC1G97, Package_TO_SOT_SMD:SOT-363_SC-70-6, F.Cu at (391.2, 91.5)
- added U901: 74LVC1G97, Package_TO_SOT_SMD:SOT-363_SC-70-6, F.Cu at (416.4, 91.1)
- added U902: TPS3808G33, Package_TO_SOT_SMD:SOT-23-6, F.Cu at (409.2, 90.5)
- added U903: M93C46-WMN6TP, Package_SO:SOIC-8_3.9x4.9mm_P1.27mm, F.Cu at (418.5, 85.9)
- added U904: 74LVC1G373, Package_TO_SOT_SMD:SOT-363_SC-70-6, F.Cu at (416.4, 94.9)
- added U905: TUSB2046BIRHBT, Package_DFN_QFN:VQFN-32-1EP_5x5mm_P0.5mm_EP3.5x3.5mm, F.Cu at (422.2, 92.8)
- added X901: ASE-48.000MHz, Oscillator:Oscillator_SMD_Abracon_ASE-4Pin_3.2x2.5mm, F.Cu at (409.1, 94.9)

Commit message: pulled in design rules
Parts:
- D201, R201, R202, R203, R207: moved to B.Cu
- moved C1001 105.1 mm to (332.0, 67.0)
- moved C1002 105.1 mm to (332.0, 69.4)
- moved C1101 105.1 mm to (332.0, 84.5)
- moved C1102 105.1 mm to (332.0, 86.9)
- moved C1501 105.1 mm to (335.1, 15.5)
- moved C1502 105.1 mm to (335.1, 17.9)
- moved C401 105.1 mm to (353.0, 36.4)
- moved C402 105.1 mm to (353.0, 38.8)
- moved C403 105.1 mm to (353.0, 41.1)
- moved C404 105.1 mm to (353.0, 43.5)
- moved C501 105.1 mm to (350.8, 6.21)
- moved C502 105.1 mm to (350.8, 8.56)
- moved C503 105.1 mm to (350.8, 10.9)
- moved C504 105.1 mm to (350.8, 13.3)
- moved C701 105.1 mm to (299.4, 32.4)
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
Commit message: some component placement
Parts:
- added C308: 10uF, Capacitors_SMD:C_1206, F.Cu at (324.0, 151.8)
- C301, C303, C501, C502, C503, D301, R301, R302, R305, R502, R504, R506, R508: moved to B.Cu
- moved C501 134.6 mm to (359.4, 140.5)
- moved R501 134.5 mm to (357.1, 140.1), turned to 90 degrees
- moved R506 134.1 mm to (355.6, 140.1), turned to -90 degrees
- moved R502 132.1 mm to (357.1, 140.1), turned to -90 degrees
- moved R507 128.2 mm to (355.6, 136.7), turned to -90 degrees
- moved C502 127.3 mm to (358.7, 135.6), turned to 90 degrees
- moved R509 126.8 mm to (362.9, 139.5), turned to 180 degrees
- moved R503 126.2 mm to (357.1, 136.7), turned to -90 degrees
- moved R508 125.7 mm to (355.6, 136.7), turned to 90 degrees
- moved C503 125.1 mm to (360.1, 135.6), turned to 90 degrees
- moved R505 124.5 mm to (355.6, 140.1), turned to 90 degrees
- moved C504 124.5 mm to (362.2, 137.2), turned to 90 degrees
- moved R504 123.7 mm to (357.1, 136.7), turned to 90 degrees
- moved U501 122.4 mm to (359.5, 138.5), turned to -90 degrees
- moved R510 122.1 mm to (363.7, 137.2), turned to 90 degrees
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Other:
- board text added: "+12V"
- board text added: "+12VIN"
- board text added: "+3.3V"
- board text added: "+5V"

Commit message: VBUS power switch placement
Parts:
- R1501, R1502, R1503, R1504: moved to B.Cu
- moved R1502 182.6 mm to (439.1, 156.2), turned to 180 degrees
- moved R1504 180.3 mm to (439.1, 158.3), turned to 180 degrees
- moved R1501 179.3 mm to (439.1, 149.7), turned to 180 degrees
- moved R1503 177.1 mm to (439.1, 151.8), turned to 180 degrees
- moved U1502 175.4 mm to (434.9, 157.2)
- moved U1501 173.9 mm to (434.9, 150.7)
- moved R1506 170.4 mm to (430.6, 157.2)
- moved C1502 167.8 mm to (430.6, 155.8), turned to 180 degrees
- moved R1508 167.7 mm to (430.6, 158.8)
- moved R1505 167.2 mm to (430.6, 150.7)
- moved R1507 164.4 mm to (430.6, 152.2)
- moved C1501 164.4 mm to (430.6, 149.3), turned to 180 degrees
- moved C201 27.4 mm to (315.6, 167.2)
- moved C202 27.4 mm to (309.4, 161.6)
- moved C203 27.4 mm to (321.5, 162.6)
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Connections:
- U1501 pad 9: (no net) -> GND
- U1502 pad 9: (no net) -> GND

Commit message: fixed some netlist connectivity issues, finished grouping parts in PCB
Parts:
- C1003, C1103, C1203, C1303, C1401, C1402, C1403, C601, C602, C603, C604, C605, C701, C702, C703, C704, C705, C706, C707, C708, C709, C710, C901, C902, C903, C904, C907, C908, C909, C910, D1001, D1101, D1201, D1301, R1401, R1402, R601, R602, R603, R604, R605, R606, R701, R702, R703, R704, R705, R706, R707, R708, R709, R710, R904, R905, R906, R907, U903: moved to B.Cu
- L901: footprint Inductors_SMD:L_0402 -> Inductors_SMD:L_0603
- moved TP1401 152.5 mm to (465.8, 27.8)
- moved D710 141.3 mm to (425.9, 79.4), turned to 90 degrees
- moved D709 141.0 mm to (425.9, 75.0), turned to 90 degrees
- moved D708 140.7 mm to (425.9, 70.7), turned to 90 degrees
- moved D707 140.4 mm to (425.9, 66.4), turned to 90 degrees
- moved D706 140.1 mm to (425.9, 62.1), turned to 90 degrees
- moved D705 139.9 mm to (425.9, 57.8), turned to 90 degrees
- moved D704 139.6 mm to (425.9, 53.5), turned to 90 degrees
- moved D703 139.5 mm to (425.9, 49.1), turned to 90 degrees
- moved D702 139.3 mm to (425.9, 44.8), turned to 90 degrees
- moved D701 139.2 mm to (425.9, 40.5), turned to 90 degrees
- moved C1401 136.4 mm to (458.5, 32.3), turned to -90 degrees
- moved C1402 135.4 mm to (458.5, 29.2), turned to 90 degrees
- moved J1401 133.9 mm to (450.4, 30.6)
- moved U1401 133.5 mm to (458.4, 27.8), turned to -90 degrees
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Connections:
- C1401 pad 1: /Upstream Port/UFP_USB_CONN_USB- -> UFP_USB_D+
- C1402 pad 1: /Upstream Port/UFP_USB_CONN_USB+ -> UFP_USB_D-
- D1001 pad 3: /Downstream Port 0/DFP0_USB_CONN_D+ -> /Downstream Port 0/DFP0_USB_CONN_D-
- D1001 pad 4: /Downstream Port 0/DFP0_USB_CONN_D- -> /Downstream Port 0/DFP0_USB_CONN_D+
- D1101 pad 3: /Downstream Port 1/DFP1_USB_CONN_D+ -> /Downstream Port 1/DFP1_USB_CONN_D-
- D1101 pad 4: /Downstream Port 1/DFP1_USB_CONN_D- -> /Downstream Port 1/DFP1_USB_CONN_D+
- D1301 pad 3: /Downstream Port 3/DFP3_USB_CONN_D+ -> /Downstream Port 3/DFP3_USB_CONN_D-
- D1301 pad 4: /Downstream Port 3/DFP3_USB_CONN_D- -> /Downstream Port 3/DFP3_USB_CONN_D+
- U1401 pad 5: /Upstream Port/UFP_USB_CONN_USB- -> UFP_USB_D-
- U1401 pad 6: /Upstream Port/UFP_USB_CONN_USB+ -> UFP_USB_D+
- U1501 pad 9: GND -> (no net)
- U1502 pad 9: GND -> (no net)
Other:
- board text added: "VBUS"

Commit message: created board outline
Parts:
- C203: moved to B.Cu
- moved J1001 348.9 mm to (109.8, 98.7), turned to 90 degrees
- moved D1001 348.3 mm to (112.5, 95.7), turned to 180 degrees
- moved C1003 343.6 mm to (109.8, 105.2), turned to -90 degrees
- moved J1101 337.3 mm to (119.9, 98.7), turned to 90 degrees
- moved D1101 336.9 mm to (122.6, 95.7), turned to 180 degrees
- moved C1103 331.8 mm to (119.9, 105.2), turned to -90 degrees
- moved J1201 326.0 mm to (130.1, 98.7), turned to 90 degrees
- moved D1201 325.8 mm to (132.8, 95.7), turned to 180 degrees
- moved C1401 324.5 mm to (136.5, 72.6), turned to 180 degrees
- moved C1402 321.9 mm to (139.6, 72.6), turned to 0 degrees
- moved R1401 321.6 mm to (137.3, 70.5), turned to -90 degrees
- moved TP1401 320.8 mm to (148.0, 71.7), turned to 90 degrees
- moved C1203 320.3 mm to (130.1, 105.2), turned to -90 degrees
- moved R1402 320.2 mm to (138.8, 70.5), turned to -90 degrees
- moved U1401 319.6 mm to (141.8, 70.8)
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Other:
- board outline added: 50 x 50 mm
- board text added: "0"
- board text added: "0 mm"
- board text added: "0.01 mm"
- board text added: "0.0152 mm"
- board text added: "0.02"
- board text added: "0.035 mm"
- board text added: "0.1 mm"
- board text added: "1"
- board text added: "1.254 mm"
- board text added: "3.3"
- board text added: "4.6"
- board text added: "B.Cu"
- board text added: "B.Mask"
- board text added: "B.Paste"
- board text added: "B.Silkscreen"
- board text added: "Bottom Silk Screen"
- board text added: "Bottom Solder Mask"
- board text added: "Bottom Solder Paste"
- board text added: "Color"
- board text added: "Dielectric 1"
- board text added: "Dielectric 2"
- board text added: "Dielectric 3"
- board text added: "Epsilon R"
- board text added: "F.Cu"
- board text added: "F.Mask"
- board text added: "F.Paste"
- board text added: "F.Silkscreen"
- board text added: "FR4"
- board text added: "GND"
- board text added: "In1.Cu"
- board text added: "In2.Cu"
- board text added: "JLC04161H-3313 Stackup"
- board text added: "Layer Name"
- board text added: "Loss Tangent"
- board text added: "Material"
- board text added: "Not specified"
- board text added: "Thickness (mm)"
- board text added: "Top Silk Screen"
- board text added: "Top Solder Mask"
- board text added: "Top Solder Paste"
- board text added: "Type"
- board text added: "copper"
- board text added: "core"
- board text added: "prepreg"
