File: hdw/USB_Hub/USB_Hub.kicad_pcb (KiCad board)
At the start: 4 copper layers, 50 x 50 mm, 203 parts, among them J1001 USB_A, J1101 USB_A, J1201 USB_A, J1301 USB_A, J1401 USB_B_Mini, J201 +12V IN, Q301 BSS214NW, Q302 ZXMS6004FFTA, SW901 RESET, U1401 TPD3S044DBVR, U1501 TPS2042BDGN, U1502 TPS2042BDGN, U201 TPS26600RHFT, U301 74LVC1G97, U302 TPS62133, U401 TPS7A92, U501 TPS2121RUXR, U601 74LVC1G97, U602 74LVC1G97, U603 74LVC1G97, U604 74LVC1G97, U605 74LVC1G97, U701 74LVC1G97, U702 74LVC1G97, U703 74LVC1G97, U704 74LVC1G97, U705 74LVC1G97, U706 74LVC1G97, U707 74LVC1G97, U708 74LVC1G97, U709 74LVC1G97, U710 74LVC1G97, U901 74LVC1G97, U902 TPS3808G33, U903 M93C46-WMN6TP, U904 74LVC1G373, U905 TUSB2046BIRHBT, X901 ASE-48.000MHz

Commit message: finished placing parts in baoard outline
Parts:
- added TP501: TP, Custom Footprints Library:Test_Point, F.Cu at (124.9, 62.9)
- C402, Q301, Q302, R401, R402, R404: moved to B.Cu
- moved D701 165.7 mm to (111.1, 91.3), turned to 180 degrees
- moved R701 165.7 mm to (111.1, 91.3), turned to 180 degrees
- moved C701 163.9 mm to (111.1, 93.8), turned to -90 degrees
- moved U701 163.9 mm to (111.1, 93.8), turned to 90 degrees
- moved D705 162.2 mm to (111.1, 86.3), turned to 180 degrees
- moved R705 162.2 mm to (111.1, 86.3), turned to 180 degrees
- moved D702 160.6 mm to (115.4, 91.3), turned to 180 degrees
- moved R702 160.6 mm to (115.4, 91.3), turned to 180 degrees
- moved C705 160.0 mm to (111.1, 88.8), turned to -90 degrees
- moved U705 160.0 mm to (111.1, 88.8), turned to 90 degrees
- moved C702 158.7 mm to (115.4, 93.8), turned to -90 degrees
- moved U702 158.7 mm to (115.4, 93.8), turned to 90 degrees
- moved D706 157.6 mm to (115.4, 86.3), turned to 180 degrees
- moved R706 157.6 mm to (115.4, 86.3), turned to 180 degrees
- moved D703 155.5 mm to (119.7, 91.3), turned to 180 degrees
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Other:
- board text added: "RESET"

Commit message: added GND plane
Routing:
- added copper zone on In1.Cu, net GND
Changed lines of the file:
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@@
     (effects (font (size 1.5 1.5) (thickness 0.1)) (justify left top))
+  )
+  (zone (net 3) (net_name "GND") (layer "In1.Cu") (hatch edge 0.5)
+    (connect_pads yes (clearance 0.254))
+    (min_thickness 0.254) (filled_areas_thickness no)
+    (fill yes (thermal_gap 0.5) (thermal_bridge_width 0.5))
+    (polygon
+      (pts
+        (xy 99.9998 59.9948)
+        (xy 150.0124 59.9948)
+        (xy 150.0124 110.0074)
+        (xy 99.9998 110.0074)
+      )
+    )
   )
   (group "group-boardStackUp" (id 2f1f8c82-7c76-448a-94ff-7ee9920bd810)

Commit message: lots of PCB progress, fixed some netlist issues
Parts:
- moved C404 0.40 mm to (120.3, 67.9)
- moved C403 0.40 mm to (120.3, 66.6)
Connections:
- D1201 pad 3: /Downstream Port 2/DFP2_USB_CONN_D+ -> /Downstream Port 2/DFP2_USB_CONN_D-
- D1201 pad 4: /Downstream Port 2/DFP2_USB_CONN_D- -> /Downstream Port 2/DFP2_USB_CONN_D+
Routing:
- net GND: track 0.00 -> 76.4 mm, vias 0 -> 19
- net +5V: track 0.00 -> 45.3 mm, vias 0 -> 12
- net +3.3V: track 0.00 -> 13.6 mm, vias 0 -> 4
- net ~{HUB_RESET}: track 0.00 -> 10.0 mm, vias 0 -> 1
- net +5VP: track 0.00 -> 6.48 mm, vias 0 -> 2
- net VBUS: track 0.00 -> 6.08 mm, vias 0 -> 2
- net HUB_CLK_EN: track 0.00 -> 5.93 mm, vias 0 -> 1
- net Net-(#FLG0901-pwr): track 0.00 -> 5.75 mm
- net POS12_PGOOD: track 0.00 -> 5.45 mm, vias 0 -> 1
- net DFP3_VBUS: track 0.00 -> 4.54 mm
- net DFP2_VBUS: track 0.00 -> 4.54 mm
- net DFP0_VBUS: track 0.00 -> 4.54 mm
- net DFP1_VBUS: track 0.00 -> 4.54 mm
- net Net-(U501-OV1): track 0.00 -> 4.44 mm, vias 0 -> 1
- net Net-(U501-OV2): track 0.00 -> 4.37 mm, vias 0 -> 1
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
Commit message: routed diff pairs
Parts:
- moved C1301 1.96 mm to (138.0, 85.7)
- moved R1301 1.96 mm to (137.3, 87.7)
- moved C1302 1.96 mm to (135.0, 85.7)
- moved R1302 1.96 mm to (135.8, 87.7)
- moved R1101 0.69 mm to (125.2, 82.9)
- moved R1102 0.69 mm to (125.2, 81.4)
- moved R1001 0.65 mm to (125.2, 77.0)
- moved R1002 0.65 mm to (125.2, 75.5)
- moved C1001 0.65 mm to (127.3, 77.8)
- moved C1002 0.65 mm to (127.3, 74.8)
- moved C1101 0.63 mm to (127.3, 83.6)
- moved C1102 0.63 mm to (127.3, 80.7)
- moved C705 0.29 mm to (110.8, 88.8)
- moved C706 0.29 mm to (115.1, 88.8)
- moved D701 0.29 mm to (110.8, 91.2)
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Routing:
- net /Downstream Port 0/DFP0_USB_CONN_D-: track 1.71 -> 50.4 mm
- net /Downstream Port 0/DFP0_USB_CONN_D+: track 1.71 -> 47.9 mm
- net /Downstream Port 1/DFP1_USB_CONN_D-: track 1.71 -> 26.2 mm
- net /Downstream Port 1/DFP1_USB_CONN_D+: track 1.71 -> 23.7 mm
- net /Downstream Port 2/DFP2_USB_CONN_D-: track 1.71 -> 22.5 mm
- net /Downstream Port 2/DFP2_USB_CONN_D+: track 1.71 -> 21.7 mm
- net /Downstream Port 3/DFP3_USB_CONN_D-: track 1.71 -> 18.1 mm
- net /Downstream Port 3/DFP3_USB_CONN_D+: track 1.71 -> 17.4 mm
- net UFP_USB_D-: track 0.00 -> 14.1 mm, vias 0 -> 1
- net UFP_USB_D+: track 0.00 -> 13.2 mm, vias 0 -> 1
- net /Upstream Port/UFP_USB_CONN_USB+: track 0.00 -> 8.56 mm, vias 0 -> 1
- net /Upstream Port/UFP_USB_CONN_USB-: track 0.00 -> 8.56 mm, vias 0 -> 1
- net DFP3_USB_D-: track 0.00 -> 7.35 mm
- net DFP3_USB_D+: track 0.00 -> 7.35 mm
- net DFP0_USB_D+: track 0.00 -> 7.18 mm
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
Commit message: random routing, via placement
Routing:
- net GND: track 76.4 -> 83.3 mm, vias 19 -> 147
- net HUB_CLK_EN: track 0.00 -> 5.87 mm, vias 0 -> 1
- net Net-(U302-PG): track 0.00 -> 4.55 mm
- net HUB_48MHCLK: track 0.00 -> 3.67 mm
- net UFP_USB_D+: track 13.2 -> 15.9 mm, vias 1 -> 2
- net +12V: track 0.00 -> 2.10 mm
- net Net-(X901-OUT): track 0.00 -> 1.83 mm
- net UFP_USB_D-: track 14.1 -> 15.4 mm, vias 1 -> 2
- added copper zone on F.Cu, net Net-(L301-Pad1)

Commit message: random power and signal routing
Parts:
- R1505, R1506, R1507, R1508: moved to B.Cu
- moved R1506 2.27 mm to (147.5, 96.0), turned to 90 degrees
- moved R1508 2.27 mm to (146.0, 96.0), turned to 90 degrees
- moved R1505 2.27 mm to (102.5, 96.0), turned to 90 degrees
- moved R1507 2.27 mm to (101.0, 96.0), turned to 90 degrees
- moved R1501 2.15 mm to (103.2, 100.1), turned to -90 degrees
- moved R1503 2.15 mm to (101.0, 100.1), turned to -90 degrees
- moved R1502 2.13 mm to (149.0, 100.1), turned to -90 degrees
- moved R1504 2.11 mm to (146.9, 100.1), turned to -90 degrees
- moved C1501 0.92 mm to (103.4, 94.5), turned to 0 degrees
- moved R906 0.14 mm to (135.6, 78.2)
- moved C1502 0.06 mm to (149.0, 93.8)
Routing:
- net VBUS: track 6.08 -> 34.5 mm, vias 2 -> 5
- net +3.3V: track 13.6 -> 28.1 mm, vias 4 -> 8
- net GND: track 83.3 -> 95.1 mm, vias 147 -> 166
- net Net-(J1401-VBUS): track 0.00 -> 8.53 mm
- net Net-(U201-RTN): track 0.00 -> 2.95 mm
- net +5V: track 45.3 -> 48.2 mm, vias 12 -> 13
- net ~{DFP0_OC}: track 2.57 -> 0.75 mm
- net ~{DFP1_OC}: track 2.57 -> 0.75 mm
- net ~{DFP3_OC}: track 2.45 -> 0.75 mm
- net ~{DFP2_OC}: track 2.42 -> 0.78 mm
- net +5VP: track 6.48 -> 7.98 mm
- net ~{DFP2_EN}: track 1.45 -> 0.67 mm, vias 0 -> 1
- net ~{DFP1_EN}: track 1.47 -> 0.69 mm, vias 0 -> 1
- net ~{DFP3_EN}: track 2.15 -> 1.53 mm, vias 0 -> 1
- net ~{DFP0_EN}: track 1.88 -> 1.38 mm, vias 0 -> 1
- added copper zone on F.Cu, net +12Vin
- added copper zone on In2.Cu, net +5V
- added copper zone on B.Cu, net DFP0_VBUS
- added copper zone on B.Cu, net DFP1_VBUS
- added copper zone on B.Cu, net DFP2_VBUS
- added copper zone on B.Cu, net DFP3_VBUS
- added copper zone on F.Cu, net GND

Commit message: lots of misc routing
Parts:
- moved C308 0.25 mm to (113.0, 71.7)
- moved C306 0.13 mm to (109.7, 77.6)
- moved C302 0.10 mm to (113.0, 74.1)
- moved C307 0.09 mm to (112.0, 77.6)
- turned R302 to 180 degrees
Routing:
- net POS12_PGOOD: track 5.45 -> 44.7 mm, vias 1 -> 2
- net POS5P_PGOOD: track 0.00 -> 34.1 mm, vias 0 -> 1
- net GND: track 95.1 -> 125.5 mm, vias 166 -> 175
- net POS5P_RUN: track 0.00 -> 16.9 mm, vias 0 -> 2
- net POS3P3_PGOOD: track 1.63 -> 8.05 mm
- net +5VP: track 7.98 -> 14.2 mm, vias 2 -> 5
- net Net-(U201-RTN): track 2.95 -> 9.11 mm, vias 0 -> 1
- net HUB_BUSPWR: track 1.55 -> 7.64 mm
- net POS5_SOURCE_STATUS: track 1.25 -> 5.50 mm
- net +3.3V: track 28.1 -> 32.0 mm
- net HUB_EECLK: track 0.00 -> 3.71 mm, vias 0 -> 1
- net HUB_EEDATA: track 0.00 -> 3.58 mm, vias 0 -> 1
- net VBUS: track 34.5 -> 38.0 mm
- net +12V: track 2.10 -> 3.75 mm, vias 0 -> 18
- net Net-(U903-Q): track 0.00 -> 0.13 mm, vias 0 -> 1
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- added copper zone on B.Cu, net +12V
- added copper zone on F.Cu, net +12V
- added copper zone on F.Cu, net +5VP
- added copper zone on F.Cu, net DFP0_VBUS
- added copper zone on F.Cu, net DFP1_VBUS
- added copper zone on F.Cu, net DFP2_VBUS
- added copper zone on F.Cu, net DFP3_VBUS

Commit message: much more routing
Parts:
- moved C709 4.49 mm to (138.3, 92.9)
- moved D709 4.49 mm to (138.3, 90.4)
- moved R709 4.49 mm to (138.3, 90.4)
- moved U709 4.49 mm to (138.3, 92.9)
- moved C710 4.38 mm to (133.8, 92.9)
- moved D710 4.38 mm to (133.8, 90.4)
- moved R710 4.38 mm to (133.8, 90.4)
- moved U710 4.38 mm to (133.8, 92.9)
- moved R1503 0.11 mm to (101.1, 100.1)
Routing:
- net +3.3V: track 32.0 -> 139.9 mm, vias 8 -> 22
- net CHASSIS: track 0.00 -> 54.8 mm, vias 0 -> 3
- net Net-(U902-~{MR}): track 0.00 -> 31.5 mm, vias 0 -> 3
- net +5VP: track 14.2 -> 40.5 mm, vias 5 -> 19
- net HUB_BUSPWR: track 7.64 -> 33.7 mm
- net POS3P3_PGOOD: track 8.05 -> 28.0 mm
- net Net-(U302-PG): track 4.55 -> 23.4 mm, vias 0 -> 2
- net HUB_SUSPND: track 2.27 -> 19.8 mm
- net GND: track 125.5 -> 142.3 mm, vias 175 -> 187
- net HUB_CLK_EN: track 5.87 -> 19.4 mm, vias 1 -> 4
- net POS5_SOURCE_STATUS: track 5.50 -> 15.7 mm, vias 0 -> 2
- net +5V: track 48.2 -> 52.0 mm, vias 14 -> 31
- net Net-(U902-CT): track 2.16 -> 0.25 mm
- net ~{DFP0_OC}: track 0.75 -> 2.56 mm, vias 1 -> 2
- net ~{DFP2_OC}: track 0.78 -> 2.39 mm, vias 1 -> 2
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- added copper zone on B.Cu, net +3.3V
- added copper zone on F.Cu, net +3.3V
- added copper zone on F.Cu, net +5V
- added copper zone on In2.Cu, net +5VP
- added copper zone on In2.Cu, net CHASSIS
- added copper zone on B.Cu, net Net-(U201-RTN)
