File: hdw/USB_Hub/USB_Hub.kicad_pcb (KiCad board)
At the start: 4 copper layers, 50 x 50 mm, 204 parts, among them J1001 USB_A, J1101 USB_A, J1201 USB_A, J1301 USB_A, J1401 USB_B_Mini, J201 +12V IN, Q301 BSS214NW, Q302 ZXMS6004FFTA, SW901 RESET, U1401 TPD3S044DBVR, U1501 TPS2042BDGN, U1502 TPS2042BDGN, U201 TPS26600RHFT, U301 74LVC1G97, U302 TPS62133, U401 TPS7A92, U501 TPS2121RUXR, U601 74LVC1G97, U602 74LVC1G97, U603 74LVC1G97, U604 74LVC1G97, U605 74LVC1G97, U701 74LVC1G97, U702 74LVC1G97, U703 74LVC1G97, U704 74LVC1G97, U705 74LVC1G97, U706 74LVC1G97, U707 74LVC1G97, U708 74LVC1G97, U709 74LVC1G97, U710 74LVC1G97, U901 74LVC1G97, U902 TPS3808G33, U903 M93C46-WMN6TP, U904 74LVC1G373, U905 TUSB2046BIRHBT, X901 ASE-48.000MHz

Commit message: got unconnects to 0
Parts:
- added G***: Owl_1_Logo, Custom Footprints Library:Owl_1_Logo, B.Cu at (124.9, 79.6)
Routing:
- net ~{DFP2_EN}: track 1.55 -> 52.4 mm, vias 2 -> 8
- net ~{DFP2_OC}: track 2.39 -> 52.9 mm, vias 2 -> 7
- net ~{DFP1_OC}: track 1.70 -> 49.7 mm, vias 2 -> 6
- net ~{DFP0_OC}: track 2.56 -> 48.4 mm, vias 2 -> 4
- net ~{DFP1_EN}: track 2.01 -> 47.7 mm, vias 2 -> 5
- net ~{DFP0_EN}: track 1.90 -> 46.5 mm, vias 2 -> 7
- net ~{DFP3_OC}: track 1.92 -> 43.3 mm, vias 2 -> 5
- net ~{DFP3_EN}: track 2.43 -> 41.4 mm, vias 2 -> 4
Other:
- board text added: "DFP0"
- board text added: "DFP1"
- board text added: "DFP2"
- board text added: "DFP3"
- board text added: "October 2023"
- board text added: "UFP"
- board text added: "USB Hub Rev A"

Commit message: added some random PCB silkscreen/misc things
Parts:
- added REF**: Symbol_Barrel_Polarity_Small, Custom Footprints Library:Symbol_Barrel_Polarity_Small, F.Cu at (103.2, 66.8)
Other:
- board text added: "+"
- board text added: "+5VP"
- board text added: "-"
- board text added: "2"
- board text added: "3"
- board text added: "4"
- board text added: "Drew Maatman"
- board text added: "JLCJLCJLCJLC"
