File: hdw/USB_Hub/power_oring.kicad_sch (KiCad schematic)
At the start: 18 parts

Commit message: lots and lots of sch progress
Parts:
- gave numbers to parts that had none: 1
Other:
- note added: "ST High when wall wart powering output, low when upstream VBUS powering output. This should not change during operation"

Commit message: pulled footprints into layout
Parts:
- R? (x2): Digi-Key PN RMCF0402FT10R0CT-ND -> (none); Wattage 1/16W -> 1/10W; display_footprint 0402 -> 0603
- R? (x2): Digi-Key PN 311-1.00KHRCT-ND -> (none)
Changed lines of the file:
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@@
       (effects (font (size 1.27 1.27)) hide)
     )
-    (property "display_footprint" "0402" (at 143.51 53.34 90)
+    (property "display_footprint" "0603" (at 143.51 53.34 90)
       (effects (font (size 1.27 1.27)) hide)
     )
@@
       (effects (font (size 1.27 1.27)) hide)
     )
-    (property "Wattage" "1/16W" (at 138.43 53.34 90)
-      (effects (font (size 1.27 1.27)) hide)
-    )
-    (property "Digi-Key PN" "RMCF0402FT10R0CT-ND" (at 146.05 53.34 0)
+    (property "Wattage" "1/10W" (at 138.43 53.34 90)
+      (effects (font (size 1.27 1.27)) hide)
+    )
+    (property "Digi-Key PN" "" (at 146.05 53.34 0)
       (effects (font (size 1.27 1.27)) hide)
     )
@@
       (effects (font (size 1.27 1.27)) (justify left) hide)
     )
-    (property "Digi-Key PN" "311-1.00KHRCT-ND" (at 149.86 102.87 0)
+    (property "Digi-Key PN" "" (at 149.86 102.87 0)
       (effects (font (size 1.524 1.524)) hide)
     )
@@
       (effects (font (size 1.27 1.27)) hide)
     )
-    (property "display_footprint" "0402" (at 154.94 53.34 90)
+    (property "display_footprint" "0603" (at 154.94 53.34 90)
       (effects (font (size 1.27 1.27)) hide)
     )
@@
       (effects (font (size 1.27 1.27)) hide)
     )
-    (property "Wattage" "1/16W" (at 149.86 53.34 90)
-      (effects (font (size 1.27 1.27)) hide)
-    )
-    (property "Digi-Key PN" "RMCF0402FT10R0CT-ND" (at 157.48 53.34 0)
+    (property "Wattage" "1/10W" (at 149.86 53.34 90)
+      (effects (font (size 1.27 1.27)) hide)
+    )
+    (property "Digi-Key PN" "" (at 157.48 53.34 0)
       (effects (font (size 1.27 1.27)) hide)
     )
@@
       (effects (font (size 1.27 1.27)) (justify left) hide)
     )
-    (property "Digi-Key PN" "311-1.00KHRCT-ND" (at 77.47 88.9 0)
+    (property "Digi-Key PN" "" (at 77.47 88.9 0)
       (effects (font (size 1.524 1.524)) hide)
     )

Commit message: big restructuring, removed microcontroller and all telemtry
Parts:
- removed R? (x2): 10, Resistors_SMD:R_0402, symbol Custom_Library:R_Custom
- removed R?: 0.02, Resistors_SMD:R_0612, symbol Custom_Library:R_Custom
- gave numbers to parts that had none: 10
- renumbered U801 to U501
Connections:
- net +5V: now also U501.1 (OUT), U501.8 (OUT)

Commit message: fixed footprints, assigned digikey pns
Parts:
- R501, R509: Digi-Key PN (none) -> 541-10.0KHCT-ND
- R502, R504, R506, R508: Digi-Key PN (none) -> 541-4.99KHCT-ND
- R503, R510: Digi-Key PN (none) -> 541-18.7KHCT-ND
- R505, R507: Digi-Key PN (none) -> 541-23.7KHCT-ND
Changed lines of the file:
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@@
       (effects (font (size 1.27 1.27)) (justify left) hide)
     )
-    (property "Digi-Key PN" "" (at 77.47 58.42 0)
+    (property "Digi-Key PN" "541-10.0KHCT-ND" (at 77.47 58.42 0)
       (effects (font (size 1.524 1.524)) hide)
     )
@@
       (effects (font (size 1.27 1.27)) (justify left) hide)
     )
-    (property "Digi-Key PN" "" (at 138.43 77.47 0)
+    (property "Digi-Key PN" "541-10.0KHCT-ND" (at 138.43 77.47 0)
       (effects (font (size 1.524 1.524)) hide)
     )
@@
       (effects (font (size 1.27 1.27)) (justify left) hide)
     )
-    (property "Digi-Key PN" "" (at 77.47 102.87 0)
+    (property "Digi-Key PN" "541-4.99KHCT-ND" (at 77.47 102.87 0)
       (effects (font (size 1.524 1.524)) hide)
     )
@@
       (effects (font (size 1.27 1.27)) (justify left) hide)
     )
-    (property "Digi-Key PN" "" (at 149.86 102.87 0)
+    (property "Digi-Key PN" "541-18.7KHCT-ND" (at 149.86 102.87 0)
       (effects (font (size 1.524 1.524)) hide)
     )
@@
       (effects (font (size 1.27 1.27)) (justify left) hide)
     )
-    (property "Digi-Key PN" "" (at 90.17 58.42 0)
+    (property "Digi-Key PN" "541-23.7KHCT-ND" (at 90.17 58.42 0)
       (effects (font (size 1.524 1.524)) hide)
     )
@@
       (effects (font (size 1.27 1.27)) (justify left) hide)
     )
-    (property "Digi-Key PN" "" (at 77.47 72.39 0)
+    (property "Digi-Key PN" "541-4.99KHCT-ND" (at 77.47 72.39 0)
       (effects (font (size 1.524 1.524)) hide)
     )
@@
       (effects (font (size 1.27 1.27)) (justify left) hide)
     )
-    (property "Digi-Key PN" "" (at 90.17 72.39 0)
+    (property "Digi-Key PN" "541-4.99KHCT-ND" (at 90.17 72.39 0)
       (effects (font (size 1.524 1.524)) hide)
     )
@@
       (effects (font (size 1.27 1.27)) (justify left) hide)
     )
-    (property "Digi-Key PN" "" (at 90.17 102.87 0)
+    (property "Digi-Key PN" "541-4.99KHCT-ND" (at 90.17 102.87 0)
       (effects (font (size 1.524 1.524)) hide)
     )
@@
       (effects (font (size 1.27 1.27)) (justify left) hide)
     )
-    (property "Digi-Key PN" "" (at 77.47 88.9 0)
+    (property "Digi-Key PN" "541-18.7KHCT-ND" (at 77.47 88.9 0)
       (effects (font (size 1.524 1.524)) hide)
     )
@@
       (effects (font (size 1.27 1.27)) (justify left) hide)
     )
-    (property "Digi-Key PN" "" (at 90.17 88.9 0)
+    (property "Digi-Key PN" "541-23.7KHCT-ND" (at 90.17 88.9 0)
       (effects (font (size 1.524 1.524)) hide)
     )

Commit message: finished placing parts in baoard outline
Parts:
- added TP401: TP, Custom Footprints Library:Test_Point, symbol Custom_Library:TP
Connections:
- net +5V: now also TP401.1 (TP)
Changed lines of the file:
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@@
   (junction (at 146.05 92.71) (diameter 0) (color 0 0 0 0)
   )
+  (junction (at 163.195 62.23) (diameter 0) (color 0 0 0 0)
+  )
   (junction (at 138.43 62.23) (diameter 0) (color 0 0 0 0)
   )
@@
     (stroke (width 0) (type default))
   )
+  (wire (pts (xy 163.195 60.96) (xy 163.195 62.23))
+    (stroke (width 0) (type default))
+  )
   (wire (pts (xy 157.48 109.22) (xy 157.48 105.41))
     (stroke (width 0) (type default))
@@
     (stroke (width 0) (type default))
   )
-  (wire (pts (xy 138.43 62.23) (xy 176.53 62.23))
+  (wire (pts (xy 138.43 62.23) (xy 163.195 62.23))
     (stroke (width 0) (type default))
   )
@@
   )
   (wire (pts (xy 146.05 91.44) (xy 146.05 92.71))
+    (stroke (width 0) (type default))
+  )
+  (wire (pts (xy 163.195 62.23) (xy 176.53 62.23))
     (stroke (width 0) (type default))
   )
@@
         )
       )
+    )
+  )
+  (symbol (lib_id "Custom_Library:TP") (at 163.195 60.96 0) (unit 1)
+    (in_bom yes) (on_board yes) (dnp no)
+    (property "Reference" "TP401" (at 163.195 57.15 0)
+      (effects (font (size 1.27 1.27)))
+    )
+    (property "Value" "TP" (at 163.195 57.15 0)
+      (effects (font (size 1.27 1.27)) hide)
+    )
+    (property "Footprint" "Custom Footprints Library:Test_Point" (at 163.195 60.96 0)
+      (effects (font (size 1.524 1.524)) hide)
+    )
+    (property "Datasheet" "" (at 163.195 60.96 0)
+      (effects (font (size 1.524 1.524)))
+    )
+    (pin "1")
+    (instances
+      (project "USB_Hub"
+        (path "/e85aac8c-404c-45dd-bda3-1057cae83baf/203423c4-94fc-4748-bda0-ab8f2e301358"
+          (reference "TP401") (unit 1)
+        )
+        (path "/e85aac8c-404c-45dd-bda3-1057cae83baf/5b35e0c1-9928-450a-ba6b-f2a701eceaac"
+          (reference "TP501") (unit 1)
+        )
+      )
+      (project "Pulse_Oximeter"
+        (path "/fc908724-b650-4421-b3fb-90738df6e526/00000000-0000-0000-0000-00005c1d5c9e"
+          (reference "TP?") (unit 1)
+        )
+        (path "/fc908724-b650-4421-b3fb-90738df6e526/00000000-0000-0000-0000-00005e939cff"
+          (reference "TP?") (unit 1)
+        )
+        (path "/fc908724-b650-4421-b3fb-90738df6e526/00000000-0000-0000-0000-00005eae2d66"
+          (reference "TP?") (unit 1)
+        )
+        (path "/fc908724-b650-4421-b3fb-90738df6e526/00000000-0000-0000-0000-00005c1d5cd8"
+          (reference "TP?") (unit 1)
+        )
+        (path "/fc908724-b650-4421-b3fb-90738df6e526/00000000-0000-0000-0000-00005e9e0e87"
+          (reference "TP?") (unit 1)
+        )
+        (path "/fc908724-b650-4421-b3fb-90738df6e526/00000000-0000-0000-0000-00005cb6f1ed"
+          (reference "TP?") (unit 1)
+        )
+        (path "/fc908724-b650-4421-b3fb-90738df6e526/00000000-0000-0000-0000-00005eae2e5f"
+          (reference "TP?") (unit 1)
+        )
+      )
